File: bornhack2026-hardware.kicad_pcb (KiCad board)
At the start: 2 copper layers, 40 parts, among them J3 USB device, U1 NRF52840-QIAA-R, X1 S201632M10PF10PPM, Y3 32.768KHz

Commit message: Fixed mistake in NRF52 footprint, add NAND FLASH, add NFC antenna schematic.
Parts:
- removed J3: USB device, Connector_USB:USB_C_Receptacle_HRO_TYPE-C-31-M-12
- removed Y3: 32.768KHz, Crystal:Crystal_SMD_3215-2Pin_3.2x1.5mm
- added C19: 2.2uF, Capacitor_SMD:C_0402_1005Metric, F.Cu at (-178.9, 124.3)
- added C20: 2.2uF, Capacitor_SMD:C_0402_1005Metric, F.Cu at (-178.9, 126.3)
- added C21: 10pF, Capacitor_SMD:C_0402_1005Metric, F.Cu at (-190.8, 121.8)
- added C23: 10pF, Capacitor_SMD:C_0402_1005Metric, F.Cu at (-190.8, 123.8)
- added C24: 100nF, Capacitor_SMD:C_0402_1005Metric, F.Cu at (-190.8, 125.8)
- added C32: 4.7u, Capacitor_SMD:C_0603_1608Metric, F.Cu at (-197.0, 107.6)
- added C33: 1u, Capacitor_SMD:C_0603_1608Metric, F.Cu at (-197.0, 110.1)
- added C34: 1u, Capacitor_SMD:C_0603_1608Metric, F.Cu at (-197.0, 112.6)
- added C35: 1u, Capacitor_SMD:C_0603_1608Metric, F.Cu at (-197.0, 115.1)
- added C36: 1u, Capacitor_SMD:C_0603_1608Metric, F.Cu at (-197.0, 117.6)
- added C37: 1u, Capacitor_SMD:C_0603_1608Metric, F.Cu at (-193.0, 107.6)
- added C38: 1u, Capacitor_SMD:C_0603_1608Metric, F.Cu at (-193.0, 110.1)
- added C39: 1u, Capacitor_SMD:C_0603_1608Metric, F.Cu at (-193.0, 112.6)
- added C40: 1u, Capacitor_SMD:C_0603_1608Metric, F.Cu at (-193.0, 115.1)
- added C41: 470n, Capacitor_SMD:C_0603_1608Metric, F.Cu at (-193.0, 117.6)
- added D2: D, Diode_SMD:D_SMA, F.Cu at (-180.5, 121.1)
- added J1: USB device, Connector_USB:USB_C_Receptacle_HRO_TYPE-C-31-M-12, F.Cu at (-178.7, 112.1)
- added L7: 0900FM15D0039001E, lcsc:FILTER-SMD_10P-L2.0-W1.3-BL, F.Cu at (-191.7, 128.5)
- added Q1: JSM2301S, lcsc:SOT-23-3_L2.9-W1.3-P1.90-LS2.4-BR, F.Cu at (-182.4, 125.4)
- added R11: 2.2, Resistor_SMD:R_0805_2012Metric, F.Cu at (-188.8, 107.8)
- added R12: 100k, Resistor_SMD:R_0402_1005Metric, F.Cu at (-189.5, 110.3)
- added R13: 0, Resistor_SMD:R_0402_1005Metric, F.Cu at (-189.5, 112.2)
- added R8: 1k, Resistor_SMD:R_0402_1005Metric, F.Cu at (-176.0, 130.5)
- added U2: SGM2040-3.3YUDH4G/TR_C5152920, lcsc:UTDFN-4AL_L1.0-W1.0-P0.65-BL, F.Cu at (-176.1, 124.6)
- added U3: SX1262IMLTRT, lcsc:QFN-24_L4.0-W4.0-P0.50-BL-EP2.6, F.Cu at (-196.2, 129.9)
- added U4: BGS12SN6E6327XTSA1, lcsc:TSNP-6_L1.1-W0.7-P0.40-BL, F.Cu at (-192.2, 130.8)
- added U5: ZD25WQ16CTIGT, lcsc:SOIC-8_L4.9-W3.9-P1.27-LS6.0-BL, F.Cu at (-128.6, 143.3)
- added X2: S201632M10PF10PPM, lcsc:CRYSTAL-SMD_4P-L2.0-W1.6-BL, F.Cu at (-195.6, 124.0)
- added Y1: 32.768KHz, Crystal:Crystal_SMD_3215-2Pin_3.2x1.5mm, F.Cu at (-145.5, 160.2)
- C1: value 2.2uF -> 1nF
- C10: value .5pF -> 100nF
- C11: value .8pF -> 100pF
- C12: value 1nF -> 100pF
- C13: value 2.2uF -> 820pF
- C14: value 2.2uF -> 100nF
- C16, C17: value 10nF -> 2.2uF
- C18: value 820pF -> 2.2uF
- C2: value 2.2uF -> 10pF
- C3, C4: value 10pF -> 10nF
- C5: value 100pF -> .5pF
- C6: value 100pF -> 10pF
- C7: value 100nF -> .8pF
- C9: value 100nF -> 2.2uF
- L1: value 10uH -> RFECA3216060A1T; footprint Inductor_SMD:L_0805_2012Metric -> lcsc:ANT-SMD_L3.1-W1.6
- L3: value RFECA3216060A1T -> 10uH; footprint lcsc:ANT-SMD_L3.1-W1.6 -> Inductor_SMD:L_0805_2012Metric
- R1, R2: value 33 -> 5k1
- R3, R4: value 5k1 -> 33
- R5: value 1k -> 100k
- moved C3 28.9 mm to (-149.0, 159.8)
- moved C4 28.6 mm to (-142.2, 160.9), turned to 180 degrees
- moved X1 5.00 mm to (-152.7, 138.1)
Connections:
- net /NRF52840_MCU/P0.04 renamed EXTERNAL_I2C_SDA
- net /NRF52840_MCU/P0.05 renamed EXTERNAL_I2C_SCL
- net /NRF52840_MCU/P0.07 renamed INTERNAL_I2C_SDA
- net /NRF52840_MCU/P0.09_NFC1 renamed /NFC Antenna/NFC1
- net /NRF52840_MCU/P0.10_NFC2 renamed /NFC Antenna/NFC2
- net /NRF52840_MCU/P0.27 renamed INTERNAL_I2C_SCL
- net /NRF52840_MCU/P0.31 renamed P0.31/VBAT
- C1 pad 1: +3V3 -> Net-(C1-Pad1)
- C10 pad 1: Net-(C10-Pad1) -> +3V3
- C10 pad 2: +3V3 -> Net-(U1-DEC1)
- C11 pad 1: /NRF52840_MCU/ANT -> +3V3
- C11 pad 2: +3V3 -> Net-(U1-DEC6)
- C12 pad 1: Net-(C12-Pad1) -> +3V3
- C12 pad 2: +3V3 -> Net-(U1-DEC3)
- C13 pad 1: VBUS -> +3V3
- C13 pad 2: +3V3 -> Net-(U1-DEC5)
- C14 pad 1: Net-(U1-VDDH) -> +3V3
- C14 pad 2: +3V3 -> Net-(U1-DEC2)
- C15 pad 1: Net-(U1-DECUSB) -> +3V3
- C16 pad 1: +3V3 -> VBUS
- C16 pad 2: /NRF52840_MCU/XL1 -> +3V3
- C17 pad 1: +3V3 -> Net-(U1-DECUSB)
- C17 pad 2: /NRF52840_MCU/XL2 -> +3V3
- C18 pad 1: +3V3 -> Net-(U1-VDDH)
- C18 pad 2: Net-(U1-DEC5) -> +3V3
- C2 pad 1: +3V3 -> /NRF52840_MCU/XC2
- C2 pad 2: DEC4-6 -> +3V3
- C3 pad 1: /NRF52840_MCU/XC1 -> +3V3
- C3 pad 2: +3V3 -> /NRF52840_MCU/XL1
- C4 pad 1: /NRF52840_MCU/XC2 -> +3V3
- C4 pad 2: +3V3 -> /NRF52840_MCU/XL2
- C5 pad 1: +3V3 -> Net-(C5-Pad1)
- C5 pad 2: Net-(U1-DEC3) -> +3V3
- C6 pad 1: +3V3 -> /NRF52840_MCU/XC1
- C6 pad 2: Net-(U1-DEC6) -> +3V3
- C7 pad 1: +3V3 -> /NRF52840_MCU/ANT
- C7 pad 2: Net-(U1-DEC1) -> +3V3
- C9 pad 2: Net-(U1-DEC2) -> DEC4-6
- L1 pad 1: DEC4-6 -> Net-(C1-Pad1)
- L1 pad 2: Net-(U1-DCC) -> Net-(C5-Pad1)
- L2 pad 1: Net-(C10-Pad1) -> Net-(C5-Pad1)
- L3 pad 1: Net-(C12-Pad1) -> DEC4-6
- L3 pad 2: Net-(C10-Pad1) -> Net-(U1-DCC)
- R1 pad 1: Net-(U1-D-) -> +3V3
- R1 pad 2: /USB_D- -> /CC1
- R2 pad 1: Net-(U1-D+) -> +3V3
- R2 pad 2: /USB_D+ -> /CC2
- R3 pad 1: +3V3 -> Net-(U1-D+)
- R3 pad 2: /CC1 -> /USB_D+
- R4 pad 1: +3V3 -> Net-(U1-D-)
- R4 pad 2: /CC2 -> /USB_D-
- R5 pad 1: P0.26 -> /POWER/VBUS
- R5 pad 2: Net-(LED1-R-) -> +3V3
- R6 pad 1: Net-(LED1-G-) -> P0.26/RED
- R6 pad 2: P0.30 -> Net-(LED1-R-)
- R7 pad 1: Net-(LED1-B-) -> Net-(LED1-G-)
- R7 pad 2: P0.06 -> P0.30/GREEN
- U1 pad AC17: (no net) -> /NRF52840_MCU/P0.21
- U1 pad B9: P0.30 -> P0.30/GREEN
- U1 pad D2: /NRF52840_MCU/P0.21 -> /NRF52840_MCU/XL1
- U1 pad G1: P0.26 -> P0.26/RED
- U1 pad L1: P0.06 -> P0.06/BLUE
Other:
- copper layers 2 -> 4

Commit message: Add original tamagotchi buttons to schematic.
Parts:
- added R14: 10k, Resistor_SMD:R_0402_1005Metric, F.Cu at (-129.9, 99.7)
- added R15: 10k, Resistor_SMD:R_0402_1005Metric, F.Cu at (-121.4, 117.0)
- added R16: 10k, Resistor_SMD:R_0402_1005Metric, F.Cu at (-129.9, 108.3)
- added R18: 10k, Resistor_SMD:R_0402_1005Metric, F.Cu at (-138.4, 117.0)
- added R19: 10k, Resistor_SMD:R_0402_1005Metric, F.Cu at (-129.9, 117.0)
- added R20: 10k, Resistor_SMD:R_0402_1005Metric, F.Cu at (-121.4, 99.7)
- added R21: 10k, Resistor_SMD:R_0402_1005Metric, F.Cu at (-138.4, 99.7)
- added R22: 10k, Resistor_SMD:R_0402_1005Metric, F.Cu at (-121.4, 108.3)
- added R23: 10k, Resistor_SMD:R_0402_1005Metric, F.Cu at (-138.4, 108.3)
- added SW1: TS3425PA 160GF 098, lcsc:SW-SMD_4P-L4.2-W3.4-P2.15-LS5.2, F.Cu at (-128.1, 96.3)
- added SW10: TS3425PA 160GF 098, lcsc:SW-SMD_4P-L4.2-W3.4-P2.15-LS5.2, F.Cu at (-136.6, 105.0)
- added SW2: TS3425PA 160GF 098, lcsc:SW-SMD_4P-L4.2-W3.4-P2.15-LS5.2, F.Cu at (-119.6, 113.6)
- added SW3: TS3425PA 160GF 098, lcsc:SW-SMD_4P-L4.2-W3.4-P2.15-LS5.2, F.Cu at (-128.1, 105.0)
- added SW5: TS3425PA 160GF 098, lcsc:SW-SMD_4P-L4.2-W3.4-P2.15-LS5.2, F.Cu at (-136.6, 113.6)
- added SW6: TS3425PA 160GF 098, lcsc:SW-SMD_4P-L4.2-W3.4-P2.15-LS5.2, F.Cu at (-128.1, 113.6)
- added SW7: TS3425PA 160GF 098, lcsc:SW-SMD_4P-L4.2-W3.4-P2.15-LS5.2, F.Cu at (-119.6, 96.3)
- added SW8: TS3425PA 160GF 098, lcsc:SW-SMD_4P-L4.2-W3.4-P2.15-LS5.2, F.Cu at (-136.6, 96.3)
- added SW9: TS3425PA 160GF 098, lcsc:SW-SMD_4P-L4.2-W3.4-P2.15-LS5.2, F.Cu at (-119.6, 105.0)
Connections:
- C32 pad 2: +3V3 -> /DISPLAY/3V3
- R13 pad 1: +3V3 -> /DISPLAY/3V3

Commit message: PCB layout egg shape, for reference.
Parts:
- added C22: 470nF, Capacitor_SMD:C_0603_1608Metric, F.Cu at (-75.1, -4.31)
- added C25: 47nF, Capacitor_SMD:C_0603_1608Metric, F.Cu at (-75.1, -1.80)
- added C26: 47pF, Capacitor_SMD:C_0402_1005Metric, F.Cu at (-88.0, -5.37)
- added C27: 1nF, Capacitor_SMD:C_0402_1005Metric, F.Cu at (-88.0, -3.40)
- added C28: 1nF, Capacitor_SMD:C_0402_1005Metric, F.Cu at (-85.1, -13.2)
- added C29: 47pF, Capacitor_SMD:C_0402_1005Metric, F.Cu at (-85.1, -11.3)
- added C30: 3.6pF, Capacitor_SMD:C_0402_1005Metric, F.Cu at (-85.1, -9.31)
- added C31: 3.6pF, Capacitor_SMD:C_0402_1005Metric, B.Cu at (-85.1, -7.34)
- added C44: 2.2uF, Capacitor_SMD:C_0402_1005Metric, B.Cu at (-85.1, -5.37)
- added J2: E-Paper, lcsc:FPC-SMD_FH12-24S-0.5SH-55, B.Cu at (0.00, 15.0)
- added TP7: VBAT+, TestPoint:TestPoint_Pad_D1.0mm, F.Cu at (-118.8, 83.7)
- C1, C10, C11, C12, C13, C14, C15, C16, C17, C18, C2, C3, C4, C5, C6, C7, C8, C9, L1, L2, L3, R14, R3, R4, SW1, TP1, TP2, TP3, TP4, TP5, TP6, U1, U5, X1, Y1: moved to B.Cu
- moved R18 207.7 mm to (15.0, -23.0)
- moved SW5 206.1 mm to (14.8, -26.1)
- moved U1 198.7 mm to (-0.75, 3.50)
- moved C7 192.4 mm to (-90.8, -13.2)
- moved C13 190.7 mm to (-88.0, -13.2)
- moved C14 190.7 mm to (-88.0, -11.3)
- moved R16 184.6 mm to (0.00, -22.9)
- moved SW3 183.3 mm to (0.00, -26.1)
- moved R3 181.1 mm to (-75.5, 6.01)
- moved R4 181.1 mm to (-75.5, 8.00)
- moved C5 180.9 mm to (-93.7, -5.37)
- moved C6 180.9 mm to (-93.7, -3.40)
- moved C1 180.9 mm to (-93.7, -13.2)
- moved C18 180.9 mm to (-88.0, -7.34)
- moved C2 180.9 mm to (-93.7, -11.3)
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Connections:
- net /NRF52840_MCU/P0.20 renamed /NRF52840_MCU/P0.20_QSPI_SIO_0
- net /NRF52840_MCU/P0.21 renamed /NRF52840_MCU/P0.21_QSPI_SCK
- net /NRF52840_MCU/P0.22 renamed /NRF52840_MCU/P0.22_QSPI_SIO_2
- net /NRF52840_MCU/P0.23 renamed /NRF52840_MCU/P0.23_QSPI_SIO_3
- net /NRF52840_MCU/P0.24 renamed /NRF52840_MCU/P0.24_QSPI_SIO_1
- net /NRF52840_MCU/P0.25 renamed /NRF52840_MCU/P0.25_QSPI_CSN
- net /NRF52840_MCU/P1.13 renamed /P1.13_SCK
- net /NRF52840_MCU/P1.14 renamed /P1.14_MISO
- net /NRF52840_MCU/P1.15 renamed /P1.15_MOSI
- C1 pad 2: +3V3 -> GND
- C10 pad 1: +3V3 -> GND
- C11 pad 1: +3V3 -> GND
- C12 pad 1: +3V3 -> GND
- C13 pad 1: +3V3 -> GND
- C14 pad 1: +3V3 -> GND
- C15 pad 2: +3V3 -> GND
- C16 pad 2: +3V3 -> GND
- C17 pad 2: +3V3 -> GND
- C18 pad 2: +3V3 -> GND
- C19 pad 2: +3V3 -> GND
- C2 pad 2: +3V3 -> GND
- C20 pad 1: /POWER/+3V3_OUT -> +3V3
- C20 pad 2: +3V3 -> GND
- C21 pad 2: +3V3 -> GND
- C23 pad 2: +3V3 -> GND
- C24 pad 1: +3V3 -> GND
- C3 pad 1: +3V3 -> GND
- C32 pad 1: +3V3 -> GND
- C32 pad 2: /DISPLAY/3V3 -> +3V3
- C34 pad 2: +3V3 -> GND
- C35 pad 1: +3V3 -> GND
- C36 pad 1: +3V3 -> GND
- C37 pad 1: +3V3 -> GND
- C38 pad 1: +3V3 -> GND
- C39 pad 1: +3V3 -> GND
- C4 pad 1: +3V3 -> GND
- C40 pad 1: +3V3 -> GND
- C41 pad 1: +3V3 -> GND
- C5 pad 2: +3V3 -> GND
- C6 pad 2: +3V3 -> GND
- C7 pad 2: +3V3 -> GND
- C8 pad 2: +3V3 -> GND
- C9 pad 1: +3V3 -> GND
- D1 pad 2: +3V3 -> GND
- D2 pad 2: /POWER/VBUS -> VBUS
- J1 pad A1: +3V3 -> GND
- J1 pad A12: +3V3 -> GND
- J1 pad B1: +3V3 -> GND
- J1 pad B12: +3V3 -> GND
- J1 pad S1: +3V3 -> GND
- L7 pad 10: +3V3 -> GND
- L7 pad 2: +3V3 -> GND
- L7 pad 5: +3V3 -> GND
- L7 pad 7: +3V3 -> GND
- L7 pad 9: +3V3 -> GND
- Q1 pad 1: /POWER/VBUS -> VBUS
- R1 pad 1: +3V3 -> GND
- R11 pad 1: +3V3 -> GND
- R12 pad 1: +3V3 -> GND
- R13 pad 1: /DISPLAY/3V3 -> +3V3
- R14 pad 1: /INPUT/3V3 -> +3V3
- R15 pad 1: /INPUT/3V3 -> +3V3
- R16 pad 1: /INPUT/3V3 -> +3V3
- R18 pad 1: /INPUT/3V3 -> +3V3
- R19 pad 1: /INPUT/3V3 -> +3V3
- R2 pad 1: +3V3 -> GND
- R20 pad 1: /INPUT/3V3 -> +3V3
- R21 pad 1: /INPUT/3V3 -> +3V3
- R22 pad 1: /INPUT/3V3 -> +3V3
- R23 pad 1: /INPUT/3V3 -> +3V3
- R5 pad 1: /POWER/VBUS -> VBUS
- R5 pad 2: +3V3 -> GND
- SW1 pad 3: +3V3 -> GND
- SW10 pad 3: +3V3 -> GND
- SW2 pad 3: +3V3 -> GND
- SW3 pad 3: +3V3 -> GND
- SW5 pad 3: +3V3 -> GND
- SW6 pad 3: +3V3 -> GND
- SW7 pad 3: +3V3 -> GND
- SW8 pad 3: +3V3 -> GND
- SW9 pad 3: +3V3 -> GND
- TP1 pad 1: +3V3 -> GND
- U1 pad 0: +3V3 -> GND
- U1 pad B7: +3V3 -> GND
- U1 pad F23: +3V3 -> GND
- U2 pad 1: /POWER/+3V3_OUT -> +3V3
- U2 pad 2: +3V3 -> GND
- U3 pad 2: +3V3 -> GND
- U3 pad 20: +3V3 -> GND
- U3 pad 25: +3V3 -> GND
- U3 pad 5: +3V3 -> GND
- U3 pad 8: +3V3 -> GND
- U4 pad 2: +3V3 -> GND
- U5 pad 4: +3V3 -> GND
- X1 pad 2: +3V3 -> GND
- X1 pad 4: +3V3 -> GND
- X2 pad 2: +3V3 -> GND
- X2 pad 4: +3V3 -> GND
Routing:
- added copper zone on In2.Cu, net +3V3
- added copper zone on B.Cu, net GND
- added copper zone on F.Cu, net GND
- added copper zone on In1.Cu, net GND
Other:
- board outline added: 67.5 x 90.1 mm

Commit message: Switched the LC filters from ceramic LoRa filter.
Parts:
- removed U4: BGS12SN6E6327XTSA1, lcsc:TSNP-6_L1.1-W0.7-P0.40-BL
- added C45: 3pF, Capacitor_SMD:C_0402_1005Metric, F.Cu at (14.0, -67.8)
- added C46: C_Small, Capacitor_SMD:C_0402_1005Metric, F.Cu at (14.0, -65.9)
- added C47: 5.6pF, Capacitor_SMD:C_0402_1005Metric, F.Cu at (14.0, -63.9)
- added C48: 39pF, Capacitor_SMD:C_0402_1005Metric, F.Cu at (14.0, -61.9)
- added C49: 1.8pF, Capacitor_SMD:C_0402_1005Metric, F.Cu at (14.0, -59.9)
- added C50: 1.8pF, Capacitor_SMD:C_0402_1005Metric, F.Cu at (14.0, -58.0)
- added C51: 2.4pF, Capacitor_SMD:C_0402_1005Metric, F.Cu at (16.8, -67.8)
- added L10: 4.7nH, Inductor_SMD:L_0402_1005Metric, F.Cu at (19.7, -63.8)
- added L11: 0, Inductor_SMD:L_0402_1005Metric, F.Cu at (19.7, -61.8)
- added L12: 15nH, Capacitor_SMD:C_0402_1005Metric, F.Cu at (16.8, -63.9)
- added L5: 15uH, Inductor_SMD:L_0603_1608Metric, F.Cu at (35.8, -31.0)
- added L6: 47nH, Inductor_SMD:L_0402_1005Metric, F.Cu at (19.7, -67.8)
- added L8: 8.2nH, Inductor_SMD:L_0402_1005Metric, F.Cu at (19.7, -65.8)
- added RF1: A-IPEX1-1.25A, lcsc:IPEX-SMD_3P-L2.6-W2.6-LS3.0_RF1200001R, B.Cu at (11.2, -34.4)
- added U6: SGM2040-3.3YN5G/TR, lcsc:SOT-23-5_L2.9-W1.6-P0.95-LS2.8-BL, F.Cu at (35.9, -25.6)
- C21, C23, J1, U3, X2: moved to B.Cu
- C31: moved to F.Cu
- L7: value 0900FM15D0039001E -> 2.5nH; footprint lcsc:FILTER-SMD_10P-L2.0-W1.3-BL -> Capacitor_SMD:C_0402_1005Metric
- U2: value SGM2040-3.3YUDH4G/TR_C5152920 -> TPE4259-63; footprint lcsc:UTDFN-4AL_L1.0-W1.0-P0.65-BL -> lcsc:SOT-363-6_L2.0-W1.3-P0.65-LS2.1-BL
- moved L7 191.2 mm to (16.8, -65.9)
- moved C24 183.7 mm to (28.7, -46.3)
- moved U2 169.2 mm to (20.1, -59.1)
- moved X2 158.4 mm to (22.3, -5.85)
- moved U3 155.7 mm to (15.1, -5.90), turned to -90 degrees
- moved C21 154.3 mm to (22.5, -7.90)
- moved C23 153.3 mm to (22.5, -3.90), turned to 180 degrees
- moved C22 121.8 mm to (37.8, -50.0)
- moved C26 117.1 mm to (11.1, -67.8)
- moved C27 117.1 mm to (11.1, -65.9)
- moved C28 108.7 mm to (11.1, -63.9)
- moved C29 108.7 mm to (11.1, -61.9)
- moved C30 108.7 mm to (11.1, -59.9)
- moved C31 108.7 mm to (11.1, -58.0)
- moved C6 105.7 mm to (9.98, -24.1)
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Connections:
- net /NRF52840_MCU/P0.15 renamed /NRF52840_MCU/P1.12
- net /SX1262 LoRA/LORA_SPI_MOSI renamed /P1.15_LORA_MOSI
- net EXTERNAL_I2C_SCL renamed /NRF52840_MCU/P0.05
- net EXTERNAL_I2C_SDA renamed /P0.04_LORA_RF_SW1
- C24 pad 2: +3V3 -> /SX1262 LoRA/3V3
- C27 pad 1: Net-(U4-CTRL) -> Net-(U2-VC2)
- C28 pad 1: Net-(U4-VDD) -> Net-(U2-VC1)
- C29 pad 1: Net-(U4-RFIN) -> Net-(U2-RFC)
- L7 pad 1: Net-(L7-RFO) -> Net-(C45-Pad1)
- L7 pad 2: GND -> Net-(C45-Pad2)
- U1 pad A10: /NRF52840_MCU/P0.29 -> /P0.29_LORA_SPI_NSS
- U1 pad A12: /NRF52840_MCU/P0.02 -> /P0.02_LORA_DIO1
- U1 pad AC9: /NRF52840_MCU/P0.14_READ_BAT -> /P1.14_LORA_MISO
- U1 pad AD6: (no net) -> Net-(U1-D+)
- U1 pad AD8: /NRF52840_MCU/P0.13 -> /P0.13_LORA_SCK
- U1 pad B11: /NRF52840_MCU/P0.28 -> /P0.28_LORA_RST
- U1 pad B13: /NRF52840_MCU/P0.03 -> /P0.03_LORA_BUSY
- U2 pad 1: +3V3 -> Net-(U2-RF2)
- U2 pad 3: /POWER/VIN -> Net-(U2-RF1)
- U2 pad 4: /POWER/VIN -> Net-(U2-VC1)
- U3 pad 1: Net-(U3-VDD_IN) -> /SX1262 LoRA/3V3
- U3 pad 10: +3V3 -> /SX1262 LoRA/3V3
- U3 pad 11: +3V3 -> /SX1262 LoRA/3V3
- U3 pad 13: /SX1262 LoRA/LORA_DIO1 -> /P0.02_LORA_DIO1
- U3 pad 14: /SX1262 LoRA/LORA_BUSY -> /P0.03_LORA_BUSY
- U3 pad 15: /SX1262 LoRA/LORA_RST -> /P0.28_LORA_RST
- U3 pad 16: /SX1262 LoRA/LORA_SPI_MISO -> /P1.14_LORA_MISO
- U3 pad 18: /SX1262 LoRA/LORA_SPI_SCK -> /P0.13_LORA_SCK
- U3 pad 19: /SX1262 LoRA/LORA_SPI_NSS -> /P0.29_LORA_SPI_NSS
- U3 pad 21: Net-(L7-RFI_P) -> Net-(U3-RFI_P)
- U3 pad 22: Net-(L7-RFI_N) -> Net-(U3-RFI_N)
- U3 pad 23: Net-(L7-RFO) -> Net-(U3-RFO)
Routing:
- net /SX1262 LoRA/XTB: track 0.00 -> 8.64 mm, vias 0 -> 2
- net /SX1262 LoRA/XTA: track 0.00 -> 6.37 mm, vias 0 -> 2
- net Net-(U1-DECUSB): track 0.00 -> 3.59 mm, vias 0 -> 1
- net Net-(U1-VDDH): track 0.00 -> 2.94 mm
- net P0.30/GREEN: vias 0 -> 1
- net Net-(U1-DEC3): vias 0 -> 1
- net INTERNAL_I2C_SDA: vias 0 -> 1
- net INTERNAL_I2C_SCL: vias 0 -> 1
- net GND: vias 0 -> 8
- net /P1.14_MISO: vias 0 -> 1
- net /P1.14_LORA_MISO: vias 0 -> 1
- net /P0.28_LORA_RST: vias 0 -> 1
- net /P0.03_LORA_BUSY: vias 0 -> 1
- net /NRF52840_MCU/RESET: vias 0 -> 1
- net /NRF52840_MCU/P1.12: vias 0 -> 1
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
Commit message: Progress, routed more stuff.
Parts:
- removed R18, R22, R23: 10k, Resistor_SMD:R_0402_1005Metric
- removed SW10, SW3, SW5, SW9: TS3425PA 160GF 098, lcsc:SW-SMD_4P-L4.2-W3.4-P2.15-LS5.2
- removed TP7: VBAT+, TestPoint:TestPoint_Pad_D1.0mm
- removed U1: NRF52840-QIAA-R, lcsc:AQFN-73_L7.0-W7.0-P0.50-BL-EP4.8
- added AE1: Antenna_Dipole, lcsc:NFC_4uH_COIL, F.Cu at (0.07, -40.1)
- added C42: 15pF, Capacitor_SMD:C_0402_1005Metric, B.Cu at (-7.77, -29.4)
- added C43: 15pF, Capacitor_SMD:C_0402_1005Metric, B.Cu at (-9.77, -29.4)
- added C52: C_Small, Capacitor_SMD:C_0402_1005Metric, B.Cu at (26.8, 2.90)
- added C53: 1uF, Capacitor_SMD:C_0603_1608Metric, B.Cu at (21.4, -8.80)
- added C54: 10uF, Capacitor_SMD:C_0603_1608Metric, B.Cu at (-18.0, 9.08)
- added C55: 100nF, Capacitor_SMD:C_0402_1005Metric, B.Cu at (-16.6, 8.47)
- added C56: 10uF, Capacitor_SMD:C_0603_1608Metric, B.Cu at (-15.2, 9.08)
- added C57: 100nF, Capacitor_SMD:C_0402_1005Metric, B.Cu at (-14.4, -11.7)
- added C58: 22uF, Capacitor_SMD:C_0805_2012Metric, B.Cu at (-11.3, -7.09)
- added C59: ~, Capacitor_SMD:C_0402_1005Metric, B.Cu at (-7.77, -28.4)
- added C60: 10uF, Capacitor_SMD:C_0603_1608Metric, B.Cu at (-20.1, -8.13)
- added C61: 10uF, Capacitor_SMD:C_0603_1608Metric, B.Cu at (-21.6, -8.13)
- added C62: 22uF, Capacitor_SMD:C_0805_2012Metric, B.Cu at (-9.27, -7.09)
- added C63: 22uF, Capacitor_SMD:C_0805_2012Metric, B.Cu at (-7.24, -7.09)
- added C64: 100nF, Capacitor_SMD:C_0402_1005Metric, B.Cu at (-12.8, -7.08)
- added D23: NSR0320MW2T1G, Diode_SMD:D_SOD-323, B.Cu at (-20.4, 8.50)
- added D3: NSR0320MW2T1G, Diode_SMD:D_SOD-323, B.Cu at (12.0, 1.50)
- added D4: NSR0320MW2T1G, Diode_SMD:D_SOD-323, B.Cu at (8.50, 1.50)
- added D5: NSR0320MW2T1G, Diode_SMD:D_SOD-323, B.Cu at (8.50, -1.00)
- added J9: Battery, lcsc:CONN-SMD_S2B-ZR-SM4A, B.Cu at (-26.5, 15.1)
- added L4: CMLW6028S1R5MST, lcsc:IND-SMD_L6.0-W6.0, B.Cu at (-15.9, -0.76)
- added L9: 47uH, Inductor_SMD:L_1210_3225Metric, B.Cu at (-9.00, -0.40)
- added Q2: AP2302B, lcsc:SOT-23-3_L2.9-W1.3-P1.90-LS2.4-BR, B.Cu at (-10.0, 6.50)
- added R10: 100, Resistor_SMD:R_0402_1005Metric, B.Cu at (27.2, 5.60)
- added R17: 1M, Resistor_SMD:R_0402_1005Metric_Pad0.72x0.64mm_HandSolder, B.Cu at (-11.1, -10.4)
- added R24: 180k, Resistor_SMD:R_0402_1005Metric_Pad0.72x0.64mm_HandSolder, B.Cu at (-12.8, -11.0)
- added R25: 2k, Resistor_SMD:R_0402_1005Metric, B.Cu at (-17.5, 3.17)
- added R26: 10k, Resistor_SMD:R_0402_1005Metric, B.Cu at (-15.2, 3.17)
- added R9: 100, Resistor_SMD:R_0402_1005Metric, B.Cu at (23.6, 5.60)
- added U4: XT4054K421MR-G, lcsc:SOT-23-5_L2.9-W1.6-P0.95-LS2.8-BL, B.Cu at (-16.8, 5.59)
- added U7: TPS63020DSJR, lcsc:VSON-14_L4.0-W3.0-P0.50-BL-EP_TI_DSJ, B.Cu at (-15.9, -7.87)
- C19, C22, C24, C25, C26, C27, C28, C29, C30, C31, C41, C45, C46, C47, C48, C49, C50, C51, D1, L10, L11, L12, L5, L6, L8, Q1, R11, R12, R13, R15, R5, R6, R7, R8, U2: moved to B.Cu
- C20: value 2.2uF -> ~; moved to B.Cu
- C32: value 4.7u -> 4.7uF; moved to B.Cu
- C33, C34, C35, C36, C37, C38, C39, C40: value 1u -> 1uF; moved to B.Cu
- D2: value D -> B160_13F; moved to B.Cu
- L7: footprint Capacitor_SMD:C_0402_1005Metric -> Inductor_SMD:L_0402_1005Metric; moved to B.Cu
- R14: value 10k -> 1k
- R16: value 10k -> 1k; moved to B.Cu
- SW1: value TS3425PA 160GF 098 -> TS-1187A-B-A-B; footprint lcsc:SW-SMD_4P-L4.2-W3.4-P2.15-LS5.2 -> lcsc:SW-SMD_4P-L5.1-W5.1-P3.70-LS6.5-TL_H1.5
- SW2: value TS3425PA 160GF 098 -> SK-3296S-01-L1; footprint lcsc:SW-SMD_4P-L4.2-W3.4-P2.15-LS5.2 -> lcsc:SW-SMD_3P-P1.50_L2.7-W6.6; moved to B.Cu
- SW6, SW7, SW8: footprint lcsc:SW-SMD_4P-L4.2-W3.4-P2.15-LS5.2 -> lcsc:KEY-SMD_2P-L6.0-W6.0-P6.00
- U6: value SGM2040-3.3YN5G/TR -> NRF52840-QIAA-R; footprint lcsc:SOT-23-5_L2.9-W1.6-P0.95-LS2.8-BL -> lcsc:XCVR_NRF52840-QIAA-R; moved to B.Cu
- moved R7 152.9 mm to (19.5, -20.8)
- moved R6 152.2 mm to (19.5, -21.9), turned to 180 degrees
- moved R8 147.3 mm to (19.5, -23.0)
- moved LED1 145.9 mm to (19.5, -21.7)
- moved C33 135.7 mm to (12.0, -1.00), turned to 180 degrees
- moved C41 129.8 mm to (9.50, 6.50), turned to -90 degrees
- moved C20 129.5 mm to (-9.77, -28.4)
- moved C34 129.4 mm to (7.25, 6.50), turned to 90 degrees
- moved C35 126.7 mm to (3.25, 6.50), turned to -90 degrees
- moved C40 124.9 mm to (5.25, 6.50), turned to -90 degrees
- moved C32 123.3 mm to (-0.23, -0.50)
- moved C36 120.6 mm to (-4.75, 6.50), turned to -90 degrees
- moved C39 120.2 mm to (1.25, 6.50), turned to -90 degrees
- moved R13 117.8 mm to (0.00, 2.00), turned to 180 degrees
- moved C38 117.4 mm to (-0.75, 6.50), turned to -90 degrees
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Connections:
- net /INPUT/BTN_LIGHTS renamed /INPUT/BTN_CONFIRM
- C10 pad 2: Net-(U1-DEC1) -> Net-(U6-DEC1)
- C11 pad 2: Net-(U1-DEC6) -> Net-(U6-DEC6)
- C12 pad 2: Net-(U1-DEC3) -> Net-(U6-DEC3)
- C13 pad 2: Net-(U1-DEC5) -> Net-(U6-DEC5)
- C14 pad 2: Net-(U1-DEC2) -> Net-(U6-DEC2)
- C17 pad 1: Net-(U1-DECUSB) -> Net-(U6-DECUSB)
- C18 pad 1: Net-(U1-VDDH) -> +3V3
- C19 pad 1: /POWER/VIN -> VIN
- C20 pad 1: +3V3 -> GND
- C20 pad 2: GND -> /NFC Antenna/NFC1
- C24 pad 2: /SX1262 LoRA/3V3 -> +3V3
- D1 pad 1: +3.3V -> VBUS
- D2 pad 1: /POWER/VIN -> VIN
- L3 pad 2: Net-(U1-DCC) -> /NRF52840_MCU/DCC
- Q1 pad 2: /POWER/VIN -> VIN
- R14 pad 1: +3V3 -> Net-(U7-PS/SYNC)
- R14 pad 2: /INPUT/BTN_RESET -> Net-(R14-Pad2)
- R15 pad 2: /INPUT/BTN_MEAL -> /INPUT/BTN_RESET
- R16 pad 1: +3V3 -> GND
- R16 pad 2: /INPUT/BTN_SNACKS -> Net-(R16-Pad2)
- R19 pad 2: /INPUT/BTN_TOILET -> /INPUT/BTN_SELECT
- R21 pad 2: /INPUT/BTN_STATS -> /INPUT/BTN_CANCEL
- R3 pad 1: Net-(U1-D+) -> /NRF52840_MCU/NRF_USB_D+
- R4 pad 1: Net-(U1-D-) -> /NRF52840_MCU/NRF_USB_D-
- SW2 pad 1: unconnected-(SW2-Pad1) -> Net-(R14-Pad2)
- SW2 pad 2: /INPUT/BTN_MEAL -> Net-(U7-EN)
- SW2 pad 3: GND -> Net-(R16-Pad2)
- SW6 pad 1: unconnected-(SW6-Pad1) -> GND
- SW6 pad 2: /INPUT/BTN_TOILET -> /INPUT/BTN_SELECT
- SW7 pad 1: unconnected-(SW7-Pad1) -> GND
- SW8 pad 1: unconnected-(SW8-Pad1) -> GND
- SW8 pad 2: /INPUT/BTN_STATS -> /INPUT/BTN_CANCEL
- U3 pad 1: /SX1262 LoRA/3V3 -> +3V3
- U3 pad 10: /SX1262 LoRA/3V3 -> +3V3
- U3 pad 11: /SX1262 LoRA/3V3 -> +3V3
- U3 pad 6: /SX1262 LoRA/DIO3 -> unconnected-(U3-DIO3-Pad6)
Routing:
- net VBUS: track 0.00 -> 58.0 mm, vias 0 -> 2
- net Net-(U7-PS/SYNC): track 0.00 -> 49.7 mm, vias 0 -> 2
- net /P1.15_LORA_MOSI: track 0.00 -> 46.7 mm, vias 0 -> 2
- net /P1.14_LORA_MISO: track 0.00 -> 43.8 mm, vias 1 -> 2
- net /P0.13_LORA_SCK: track 0.00 -> 43.5 mm, vias 0 -> 2
- net /POWER/VBAT: track 0.00 -> 42.5 mm, vias 0 -> 2
- net /P0.04_LORA_RF_SW1: track 0.00 -> 41.9 mm, vias 0 -> 2
- net Net-(U7-EN): track 0.00 -> 39.4 mm, vias 0 -> 2
- net /USB_D-: track 0.00 -> 38.6 mm, vias 0 -> 2
- net /USB_D+: track 0.00 -> 38.5 mm, vias 0 -> 2
- net +3V3: track 0.00 -> 31.7 mm, vias 3 -> 23
- net P0.06/BLUE: track 0.00 -> 31.0 mm, vias 0 -> 2
- net /P0.29_LORA_SPI_NSS: track 0.00 -> 31.0 mm, vias 0 -> 2
- net /P0.03_LORA_BUSY: track 0.00 -> 29.8 mm, vias 1 -> 2
- net /P0.28_LORA_RST: track 0.00 -> 29.6 mm, vias 1 -> 2
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- added copper zone on B.Cu, net +3V3
- added copper zone on In1.Cu, net +3V3
- added copper zone on In2.Cu, net GND
- added copper zone on B.Cu, net Net-(L4-Pad1)
- added copper zone on B.Cu, net Net-(L4-Pad2)
- added copper zone on B.Cu, net VIN
- removed copper zone on In2.Cu, net +3V3
- removed copper zone on In1.Cu, net GND
Other:
- outline, holes or cut-outs redrawn
