File: bornhack2026-hardware.kicad_pcb (KiCad board)
At the start: 4 copper layers, 67.5 x 90.1 mm, 133 parts, among them J1 USB device, J2 E-Paper, J9 Battery, Q1 JSM2301S, Q2 AP2302B, SW1 TS-1187A-B-A-B, SW2 SK-3296S-01-L1, SW6 TS3425PA 160GF 098, SW7 TS3425PA 160GF 098, SW8 TS3425PA 160GF 098, U2 TPE4259-63, U3 SX1262IMLTRT, U4 XT4054K421MR-G, U5 ZD25WQ16CTIGT, U6 NRF52840-QIAA-R, U7 TPS63020DSJR, X1 S201632M10PF10PPM, X2 S201632M10PF10PPM, Y1 32.768KHz

Commit message: Bluetooth antenna should work better, NFC has IPEX for tuning.
Parts:
- added NT1: NetTie_2 (Feed to ground), lcsc:NetTie-2_SMD_SQ_Pad0.8mm, B.Cu at (10.5, -31.8)
- added R18: 10k, Resistor_SMD:R_0402_1005Metric, B.Cu at (19.5, 12.8)
- added R22: 10k, Resistor_SMD:R_0402_1005Metric, B.Cu at (20.5, 12.8)
- added R23: 10k, Resistor_SMD:R_0402_1005Metric, B.Cu at (14.8, 12.8)
- added R27: 10k, Resistor_SMD:R_0402_1005Metric, B.Cu at (16.0, 12.8)
- added R28: 10k, Resistor_SMD:R_0402_1005Metric, B.Cu at (13.5, 12.8)
- added R29: 0, Resistor_SMD:R_0402_1005Metric, B.Cu at (-5.49, -23.1)
- added R30: 0, Resistor_SMD:R_0402_1005Metric, B.Cu at (-5.49, -24.1)
- added RF2: A-IPEX1-1.25A, lcsc:IPEX-SMD_3P-L2.6-W2.6-LS3.0_RF1200001R, B.Cu at (-9.60, -25.8)
- added SW3: SKRHABE010, lcsc:SW-SMD_SKRHABE010, F.Cu at (16.8, 13.5)
- C42, C43: value 15pF -> 12pF
- R1, R19, R2, R20, R21: moved to B.Cu
- moved R2 11.4 mm to (-28.5, -1.26), turned to -90 degrees
- moved R1 9.80 mm to (-29.5, -1.26), turned to -90 degrees
- moved C5 5.08 mm to (4.75, -26.9), turned to 90 degrees
- moved R19 4.32 mm to (-15.0, 27.1)
- moved R20 4.32 mm to (0.01, 27.1)
- moved R21 4.32 mm to (15.0, 27.1)
- moved L1 3.78 mm to (12.4, -33.1), turned to 45 degrees
- moved C1 3.74 mm to (14.9, -35.5), turned to 45 degrees
- moved TP5 2.87 mm to (-2.29, -27.9), turned to -90 degrees
- moved TP6 2.83 mm to (-2.29, -25.2), turned to -90 degrees
- moved TP3 2.75 mm to (-27.2, -15.9)
- moved TP4 2.75 mm to (-24.5, -15.9)
- moved C7 2.55 mm to (1.70, -26.9), turned to 90 degrees
- moved L2 2.10 mm to (3.20, -26.4), turned to 180 degrees
- moved C12 1.20 mm to (4.30, -23.0)
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Connections:
- AE1 pad 1: /NFC Antenna/NFC2 -> Net-(AE1-Pad1)
- AE1 pad 2: /NFC Antenna/NFC1 -> Net-(AE1-Pad2)
- C20 pad 2: /NFC Antenna/NFC1 -> Net-(AE1-Pad2)
- C42 pad 1: /NFC Antenna/NFC2 -> Net-(AE1-Pad1)
- C43 pad 2: /NFC Antenna/NFC1 -> Net-(AE1-Pad2)
- C59 pad 2: /NFC Antenna/NFC2 -> Net-(AE1-Pad1)
- L1 pad 1: Net-(C1-Pad1) -> Net-(L1-Pad1)
- L1 pad 2: Net-(C5-Pad1) -> Net-(C1-Pad1)
- R15 pad 2: /INPUT/BTN_RESET -> /MCU_RESET
- SW1 pad 2: /INPUT/BTN_RESET -> /MCU_RESET
- TP2 pad 1: /NRF52840_MCU/RESET -> /MCU_RESET
- U6 pad AC13: /NRF52840_MCU/RESET -> /MCU_RESET
Routing:
- net /MCU_RESET: track 0.00 -> 86.7 mm, vias 0 -> 3
- net SWDCLK: track 0.00 -> 27.0 mm
- net SWDIO: track 0.00 -> 23.4 mm
- net Net-(AE1-Pad2): track 0.00 -> 15.1 mm
- net Net-(C5-Pad1): track 17.8 -> 4.22 mm
- net /NFC Antenna/NFC1: track 21.1 -> 9.53 mm
- net Net-(AE1-Pad1): track 0.00 -> 11.4 mm, vias 0 -> 1
- net /CC1: track 0.00 -> 10.7 mm
- net +3V3: track 31.7 -> 41.0 mm, vias 23 -> 28
- net /CC2: track 0.00 -> 7.53 mm
- net /INPUT/BTN_JOY_DOWN: track 0.00 -> 6.22 mm, vias 0 -> 2
- net /INPUT/BTN_JOY_UP: track 0.00 -> 5.31 mm, vias 0 -> 1
- net /NFC Antenna/NFC2: track 18.9 -> 14.0 mm, vias 1 -> 0
- net /INPUT/BTN_JOY_RIGHT: track 0.00 -> 4.44 mm, vias 0 -> 1
- net /INPUT/BTN_JOY_FIRE: track 0.00 -> 4.20 mm, vias 0 -> 1
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
Commit message: Wired in display
Parts:
- moved R18 25.0 mm to (40.1, 27.0)
- moved R22 25.0 mm to (41.1, 27.0)
- moved R23 25.0 mm to (35.4, 27.0)
- moved R27 25.0 mm to (36.6, 27.0)
- moved R28 25.0 mm to (34.1, 27.0)
- moved SW3 25.0 mm to (37.4, 27.7)
- moved C33 17.7 mm to (-5.60, -2.40), turned to -90 degrees
- moved D3 15.6 mm to (-3.10, -2.40), turned to -90 degrees
- moved D5 14.3 mm to (-5.60, 1.10), turned to 90 degrees
- moved D4 11.6 mm to (-3.10, 1.10), turned to -90 degrees
- moved R13 7.10 mm to (-0.80, 9.05), turned to 90 degrees
- moved C32 2.59 mm to (2.00, -1.82), turned to -90 degrees
- moved C4 0.60 mm to (0.00, -11.1)
- moved C3 0.60 mm to (1.90, -11.1)
- moved C18 0.58 mm to (-3.60, -10.6)
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Connections:
- net INTERNAL_I2C_SCL renamed /NRF52840_MCU/P0.27
- J2 pad 11: /DISPLAY/MOSI -> /P0.05_DSP_MOSI
- J2 pad 12: /DISPLAY/SCK -> /P0.07_DSP_SCK
- J2 pad 13: /DISPLAY/CS -> /P0.08_DSP_CSN
- J2 pad 15: /DISPLAY/RESET -> /P0.11_DSP_RESET
- J2 pad 16: /DISPLAY/BUSY -> /P0.12_DSP_BUSY
- U6 pad K2: /NRF52840_MCU/P0.05 -> /P0.05_DSP_MOSI
- U6 pad M2: INTERNAL_I2C_SDA -> /P0.07_DSP_SCK
- U6 pad N1: /NRF52840_MCU/P0.08 -> /P0.08_DSP_CSN
- U6 pad T2: /NRF52840_MCU/P0.11/6D_INT1 -> /P0.11_DSP_RESET
- U6 pad U1: /NRF52840_MCU/P0.12 -> /P0.12_DSP_BUSY
Routing:
- net /P0.05_DSP_MOSI: track 0.00 -> 28.7 mm, vias 0 -> 2
- net /P0.11_DSP_RESET: track 0.00 -> 27.8 mm, vias 0 -> 2
- net /P0.07_DSP_SCK: track 0.00 -> 27.3 mm, vias 0 -> 2
- net /P0.12_DSP_BUSY: track 0.00 -> 27.0 mm
- net /P0.08_DSP_CSN: track 0.00 -> 26.1 mm
- net /DISPLAY/PREVGH: track 0.00 -> 20.8 mm, vias 0 -> 2
- net /DISPLAY/PREVGL: track 0.00 -> 19.7 mm, vias 0 -> 2
- net Net-(D5-A): track 0.00 -> 12.7 mm
- net /DISPLAY/GDR: track 0.00 -> 12.5 mm
- net /DISPLAY/RESE: track 0.00 -> 8.64 mm
- net /DISPLAY/VCOM: track 0.00 -> 7.13 mm
- net Net-(J2-Pin_7): track 0.00 -> 7.07 mm, vias 0 -> 2
- net /DISPLAY/VSH: track 0.00 -> 5.54 mm, vias 0 -> 2
- net Net-(D3-A): track 0.00 -> 4.92 mm
- net /DISPLAY/VGH: track 0.00 -> 4.92 mm
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
Commit message: Redid the sx1268 RF circuit for the layout to comply with the datasheet.
Parts:
- C25: footprint Capacitor_SMD:C_0603_1608Metric -> Capacitor_SMD:C_0402_1005Metric
- moved R15 31.2 mm to (2.04, -4.94), turned to 90 degrees
- moved SW1 23.1 mm to (8.00, -3.50), turned to 180 degrees
- moved C52 7.89 mm to (25.1, -4.80)
- moved C51 7.79 mm to (24.6, -6.20)
- moved L12 7.68 mm to (25.1, -7.60)
- moved C50 5.54 mm to (25.6, -6.20), turned to 90 degrees
- moved C22 3.48 mm to (22.9, -15.2)
- moved C53 2.73 mm to (19.4, -7.00), turned to 180 degrees
- moved C46 2.56 mm to (23.1, -4.80), turned to 0 degrees
- moved R9 2.55 mm to (21.3, 4.50), turned to 0 degrees
- moved C26 1.60 mm to (22.1, -6.80)
- moved C25 1.30 mm to (22.1, -7.80)
- moved L11 1.30 mm to (23.6, -7.30)
- moved L6 1.29 mm to (23.1, -5.80)
- moved U2 1.24 mm to (24.5, 4.80)
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Routing:
- net /MCU_RESET: track 86.9 -> 42.7 mm
- net Net-(U3-RFI_N): track 11.7 -> 3.11 mm
- net Net-(U3-RFI_P): track 10.4 -> 3.18 mm
- net Net-(U2-RF1): track 3.01 -> 10.1 mm
- net GND: track 11.8 -> 18.2 mm, vias 161 -> 291
- net /P0.04_LORA_RF_SW1: track 40.7 -> 36.1 mm
- net /P0.02_LORA_DIO1: track 29.4 -> 31.6 mm
- net /P0.28_LORA_RST: track 29.6 -> 31.5 mm
- net +3V3: track 41.0 -> 42.8 mm, vias 28 -> 29
- net /P0.03_LORA_BUSY: track 29.8 -> 31.6 mm
- net Net-(U3-VR_PA): track 6.17 -> 4.44 mm
- net /P1.15_LORA_MOSI: track 47.0 -> 48.2 mm
- net /P1.14_LORA_MISO: track 44.0 -> 45.3 mm
- net Net-(U2-VC2): track 2.37 -> 3.18 mm
- net /P0.13_LORA_SCK: track 43.8 -> 44.5 mm
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