File: bornhack2026-hardware.kicad_pcb (KiCad board)
At the start: 4 copper layers, 67.5 x 90.1 mm, 143 parts, among them J1 USB device, J2 E-Paper, J9 Battery, Q1 JSM2301S, Q2 AP2302B, SW1 TS-1187A-B-A-B, SW2 SK-3296S-01-L1, SW3 SKRHABE010, SW6 TS3425PA 160GF 098, SW7 TS3425PA 160GF 098, SW8 TS3425PA 160GF 098, U2 TPE4259-63, U3 SX1262IMLTRT, U4 XT4054K421MR-G, U5 ZD25WQ16CTIGT, U6 NRF52840-QIAA-R, U7 TPS63020DSJR, X1 S201632M10PF10PPM, X2 S201632M10PF10PPM, Y1 32.768KHz

Commit message: small fixes.
Parts:
- removed R20: 10k, Resistor_SMD:R_0402_1005Metric
- removed SW7: TS3425PA 160GF 098, lcsc:KEY-SMD_2P-L6.0-W6.0-P6.00
- moved R18 37.4 mm to (2.69, 27.0)
- moved R22 37.4 mm to (3.69, 27.0)
- moved R23 37.4 mm to (-2.06, 27.0)
- moved R27 37.4 mm to (-0.81, 27.0)
- moved R28 37.4 mm to (-3.31, 27.0)
- moved SW3 37.4 mm to (-0.06, 27.7)
- moved LED1 4.12 mm to (15.9, -23.7)
- moved R7 4.12 mm to (15.9, -22.8)
- moved R6 4.12 mm to (15.9, -23.9)
- moved R8 4.12 mm to (15.9, -25.0)
Routing:
- net /INPUT/BTN_CONFIRM: track 2.40 -> 0.00 mm, vias 1 -> 0
- net (no net): track 0.00 -> 1.43 mm
- net P0.30/GREEN: track 22.4 -> 21.1 mm
- net P0.26/RED: track 28.1 -> 26.9 mm
- net +3V3: track 42.8 -> 41.8 mm, vias 29 -> 28
- net P0.06/BLUE: track 32.7 -> 32.2 mm
- net GND: vias 291 -> 290

Commit message: Routed buttons to MCU.
Parts:
- removed TP2: RESET, TestPoint:TestPoint_Pad_D1.5mm
- added C65: ~, Capacitor_SMD:C_0402_1005Metric, B.Cu at (-8.83, -30.1)
- added H1: MountingHole_Pad, MountingHole:MountingHole_2.2mm_M2_DIN965_Pad, F.Cu at (27.0, -9.00)
- added H2: MountingHole_Pad, MountingHole:MountingHole_2.2mm_M2_DIN965_Pad, F.Cu at (-27.0, -9.00)
- added H3: MountingHole_Pad, MountingHole:MountingHole_2.2mm_M2_DIN965_Pad, F.Cu at (0.00, 36.0)
- added L13: 400-1000MHZ-CHIP(B&T-1503), lcsc:ANT-SMD_L15.0-W3.0, B.Cu at (22.1, -23.2)
- added R31: 0, Resistor_SMD:R_0402_1005Metric, B.Cu at (18.8, -9.02)
- added R32: 0, Resistor_SMD:R_0402_1005Metric, B.Cu at (19.5, -9.01)
- R6, R8: value 1k -> 2k
- R7: value 1k -> 10k
- TP5, TP6: footprint TestPoint:TestPoint_Pad_D1.5mm -> TestPoint:TestPoint_Pad_D1.0mm
- moved L5 37.7 mm to (20.3, 20.9), turned to 180 degrees
- moved C24 36.1 mm to (17.6, 19.7), turned to 0 degrees
- moved C22 34.7 mm to (20.8, 19.5), turned to 180 degrees
- moved C23 33.4 mm to (26.2, 18.3), turned to 0 degrees
- moved X2 29.4 mm to (26.1, 16.2), turned to -90 degrees
- moved U3 28.2 mm to (18.7, 15.9), turned to -90 degrees
- moved RF1 26.1 mm to (18.4, -11.5), turned to 0 degrees
- moved C21 25.4 mm to (26.2, 14.1), turned to 180 degrees
- moved TP1 21.6 mm to (-18.4, -33.0), turned to -90 degrees
- moved TP3 20.6 mm to (-15.7, -33.0), turned to -90 degrees
- moved L12 20.5 mm to (18.6, 11.9), turned to 0 degrees
- moved C31 20.4 mm to (18.7, -7.53), turned to 180 degrees
- moved C25 19.9 mm to (21.6, 12.1), turned to 0 degrees
- moved L11 19.2 mm to (20.1, 11.6), turned to 90 degrees
- moved C53 18.9 mm to (24.4, 11.3), turned to 0 degrees
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Connections:
- R18 pad 2: /INPUT/BTN_JOY_DOWN -> /BTN_JOY_DOWN
- R19 pad 2: /INPUT/BTN_SELECT -> /BTN_SELECT
- R21 pad 2: /INPUT/BTN_CANCEL -> /BTN_CANCEL
- R22 pad 2: /INPUT/BTN_JOY_RIGHT -> /BTN_JOY_RIGHT
- R23 pad 2: /INPUT/BTN_JOY_FIRE -> /BTN_JOY_FIRE
- R27 pad 2: /INPUT/BTN_JOY_UP -> /BTN_JOY_UP
- R28 pad 2: /INPUT/BTN_JOY_LEFT -> /BTN_JOY_LEFT
- RF1 pad 1: /SX1262 LoRA/LORA_ANT -> Net-(R31-Pad1)
- SW3 pad 1: /INPUT/BTN_JOY_UP -> /BTN_JOY_UP
- SW3 pad 2: /INPUT/BTN_JOY_FIRE -> /BTN_JOY_FIRE
- SW3 pad 3: /INPUT/BTN_JOY_LEFT -> /BTN_JOY_LEFT
- SW3 pad 4: /INPUT/BTN_JOY_RIGHT -> /BTN_JOY_RIGHT
- SW3 pad 6: /INPUT/BTN_JOY_DOWN -> /BTN_JOY_DOWN
- SW6 pad 2: /INPUT/BTN_SELECT -> /BTN_SELECT
- SW8 pad 2: /INPUT/BTN_CANCEL -> /BTN_CANCEL
- U6 pad P23: /NRF52840_MCU/P1.07 -> /BTN_SELECT
- U6 pad R1: /NRF52840_MCU/P1.09 -> /BTN_CANCEL
- U6 pad T23: /NRF52840_MCU/P1.05 -> /BTN_JOY_FIRE
- U6 pad U24: /NRF52840_MCU/P1.04 -> /BTN_JOY_LEFT
- U6 pad V23: /NRF52840_MCU/P1.03 -> /BTN_JOY_DOWN
- U6 pad W24: /NRF52840_MCU/P1.02 -> /BTN_JOY_UP
- U6 pad Y23: /NRF52840_MCU/P1.01 -> /BTN_JOY_RIGHT
Routing:
- net /BTN_JOY_DOWN: track 0.00 -> 91.7 mm, vias 0 -> 2
- net /BTN_JOY_RIGHT: track 0.00 -> 87.4 mm, vias 0 -> 2
- net /BTN_JOY_UP: track 0.00 -> 80.8 mm, vias 0 -> 2
- net /BTN_JOY_FIRE: track 0.00 -> 79.3 mm, vias 0 -> 2
- net /BTN_JOY_LEFT: track 0.00 -> 78.4 mm, vias 0 -> 2
- net /BTN_SELECT: track 0.00 -> 75.6 mm, vias 0 -> 2
- net /BTN_CANCEL: track 0.00 -> 59.0 mm, vias 0 -> 3
- net /MCU_RESET: track 42.7 -> 22.1 mm, vias 3 -> 2
- net /P0.03_LORA_BUSY: track 31.6 -> 45.4 mm, vias 2 -> 4
- net /P0.02_LORA_DIO1: track 31.6 -> 43.6 mm, vias 2 -> 4
- net /P0.28_LORA_RST: track 31.5 -> 42.4 mm, vias 2 -> 4
- net Net-(L13-ANT): track 0.00 -> 9.63 mm
- net /P0.29_LORA_SPI_NSS: track 31.4 -> 40.8 mm, vias 2 -> 3
- net VBUS: track 58.0 -> 67.1 mm
- net P0.06/BLUE: track 32.2 -> 25.7 mm
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
Commit message: Fixed DRC errors, added bunch of stitch through vias.
Parts:
- moved SW2 0.94 mm to (-21.7, 29.3)
- moved J1 0.13 mm to (-29.8, 6.03)
- moved C25 0.06 mm to (21.6, 12.1)
- moved C26 0.06 mm to (21.6, 11.1)
- moved C46 0.06 mm to (20.6, 9.13)
- moved C47 0.06 mm to (20.6, 6.33)
- moved C51 0.06 mm to (19.1, 10.5)
- moved C52 0.06 mm to (18.7, 9.13)
- moved C53 0.06 mm to (24.4, 11.3)
- moved L11 0.06 mm to (20.1, 11.6)
- moved L12 0.06 mm to (18.6, 11.9)
- moved L6 0.06 mm to (20.6, 10.1)
- moved L7 0.06 mm to (21.1, 7.73)
- moved C45 0.06 mm to (20.1, 7.73)
- moved C48 0.06 mm to (20.1, 4.93)
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Routing:
- net Net-(R14-Pad2): track 2.33 -> 1.43 mm
- net /USB_D+: track 39.5 -> 40.0 mm
- net /BTN_JOY_RIGHT: track 87.4 -> 88.0 mm
- net Net-(R16-Pad2): track 2.71 -> 2.18 mm
- net /P0.29_LORA_SPI_NSS: track 40.8 -> 40.5 mm, vias 3 -> 2
- net GND: vias 364 -> 598
Other:
- outline, holes or cut-outs redrawn

Commit message: Fix tiny issues, add more vias.
Parts:
- added C66: 2.2uF, Capacitor_SMD:C_0402_1005Metric, B.Cu at (-19.5, 26.4)
- added C67: 2.2uF, Capacitor_SMD:C_0402_1005Metric, B.Cu at (-20.2, 24.3)
- added C68: 100nF, Capacitor_SMD:C_0402_1005Metric, B.Cu at (-18.3, -20.5)
- added R33: 1M, Resistor_SMD:R_0402_1005Metric_Pad0.72x0.64mm_HandSolder, B.Cu at (-21.0, -11.2)
- moved R14 2.89 mm to (-18.8, 25.7), turned to -45 degrees
- moved R16 0.87 mm to (-20.9, 25.0)
- moved TP5 0.40 mm to (-2.29, -26.3)
- moved TP6 0.40 mm to (-2.45, -24.2)
Connections:
- C57 pad 1: Net-(U7-PS/SYNC) -> Net-(U7-VINA)
- R14 pad 1: Net-(U7-PS/SYNC) -> Net-(U7-VINA)
- U6 pad AD12: /NRF52840_MCU/P0.17 -> /P0.17_PS_SYNC
- U7 pad 1: Net-(U7-PS/SYNC) -> Net-(U7-VINA)
- U7 pad 13: Net-(U7-PS/SYNC) -> /P0.17_PS_SYNC
Routing:
- net Net-(U7-VINA): track 0.00 -> 51.3 mm, vias 0 -> 2
- net Net-(U7-PS/SYNC): track 48.9 -> 0.00 mm, vias 2 -> 0
- net /P0.17_PS_SYNC: track 0.00 -> 29.6 mm, vias 0 -> 2
- net Net-(R14-Pad2): track 1.43 -> 4.78 mm
- net +3V3: track 44.4 -> 47.1 mm
- net /BTN_JOY_UP: track 80.8 -> 82.4 mm
- net Net-(C67-Pad2): track 2.18 -> 3.60 mm
- net P0.06/BLUE: track 25.7 -> 26.9 mm
- net VBUS: track 67.1 -> 66.4 mm
- net GND: vias 598 -> 649

Commit message: Moved SMA-connector Lora for VNA testing.
Parts:
- moved R32 6.43 mm to (24.7, -12.8)
- moved RF1 4.06 mm to (22.3, -10.5), turned to -45 degrees
- moved R31 1.74 mm to (20.5, -8.78), turned to -135 degrees
- moved L13 1.38 mm to (22.6, -24.5)
Connections:
- R32 pad 2: /SX1262 LoRA/LORA_ANT -> Net-(R31-Pad1)
Routing:
- net Net-(R31-Pad1): track 1.20 -> 4.82 mm
- net Net-(L13-ANT): track 9.63 -> 7.52 mm
- net GND: vias 649 -> 667
