File: bornhack2026-hardware.kicad_pcb (KiCad board)
At the start: 4 copper layers, 67.4 x 89.9 mm, 159 parts, among them J1 USB device, J2 E-Paper, J3 Conn_01x05, J9 Battery, Q1 JSM2301S, Q2 AP2302B, SW1 TS-1187A-B-A-B, SW2 SK-3296S-01-L1, SW3 SKRHABE010, SW6 TS3425PA 160GF 098, SW8 TS3425PA 160GF 098, U2 TPE4259-63, U3 SX1262IMLTRT, U4 XT4054K421MR-G, U5 ZD25WQ16CTIGT, U6 NRF52840-QIAA-R, U7 TPS63020DSJR, X1 S201632M10PF10PPM, X2 S201632M10PF10PPM, X3 32.768KHz

Commit message: Badge.Team
Parts:
- N2: value Ranzbak -> Badge.Team; footprint defeest:goatse_01 -> symbols:stamp

Commit message: Fix screen outline (that I broke), add epaper 3D model back in, move flat cable hole down a bit.
Routing:
- net GND: vias 611 -> 602

Commit message: Squashed in new battery connector, made NFC coil and Bluetooth fit as good and bad as possible.
Parts:
- removed J9: Battery, lcsc:CONN-SMD_S2B-ZR-SM4A
- removed TP5: NFC2, TestPoint:TestPoint_Pad_D1.0mm
- removed TP6: NFC1, TestPoint:TestPoint_Pad_D1.0mm
- added N3: Bornhack, lcsc:bornhack-logo-10mm, B.Cu at (20.4, -17.2)
- added U1: PH-2AWB, lcsc:CONN-SMD_PH-2AWB, B.Cu at (-27.2, 12.1)
- moved RF2 7.61 mm to (-1.60, -25.7), turned to 180 degrees
- moved C20 7.11 mm to (-2.68, -27.5)
- moved C42 7.11 mm to (-0.68, -28.6)
- moved C43 7.11 mm to (-2.68, -28.6)
- moved C59 7.11 mm to (-0.68, -27.5)
- moved C65 7.11 mm to (-1.74, -29.5)
- moved R30 5.75 mm to (-0.40, -22.6), turned to -90 degrees
- moved R2 5.50 mm to (-27.2, -5.66), turned to -90 degrees
- moved R1 4.73 mm to (-28.2, -5.66), turned to -90 degrees
- moved J1 4.27 mm to (-29.1, 1.80)
- moved R29 4.24 mm to (-1.40, -22.6), turned to -90 degrees
- moved AE2 3.68 mm to (8.88, -29.0), turned to 176 degrees
- moved AE1 1.80 mm to (-1.80, -40.0), turned to -90 degrees
- moved Q1 1.02 mm to (-22.6, -4.70)
Routing:
- net Net-(U7-EN): track 29.8 -> 13.9 mm, vias 2 -> 1
- net Net-(AE1-Pad2): track 14.0 -> 3.71 mm
- net /NFC Antenna/NFC2: track 10.0 -> 0.00 mm
- net /NFC Antenna/NFC1: track 7.71 -> 0.00 mm
- net Net-(AE1-Pad1): track 9.88 -> 3.82 mm
- net /USB_D+: track 39.6 -> 35.0 mm
- net VBUS: track 67.2 -> 62.7 mm
- net /USB_D-: track 39.8 -> 35.4 mm
- net Net-(AE2-Pad1): track 5.61 -> 3.17 mm
- net GND: track 15.0 -> 13.5 mm, vias 602 -> 566
- net VIN: track 12.6 -> 11.6 mm
- net /CC1: track 11.9 -> 11.2 mm
- net /POWER/VBAT: track 37.7 -> 38.2 mm, vias 0 -> 2
Other:
- board text removed: "-"

Commit message: Clean up NFC connection.
Parts:
- moved C20 0.34 mm to (-2.34, -27.5)
- moved C43 0.34 mm to (-2.34, -28.6)
- moved C42 0.34 mm to (-0.34, -28.6)
- moved C59 0.34 mm to (-0.34, -27.5)
- moved C65 0.34 mm to (-1.40, -29.5)
Routing:
- net Net-(AE1-Pad2): track 3.71 -> 8.96 mm
- net Net-(AE1-Pad1): track 3.82 -> 8.47 mm
- net /NFC Antenna/NFC1: track 0.00 -> 2.55 mm
- net /NFC Antenna/NFC2: track 0.00 -> 2.34 mm
