File: nrf52840_mcu.kicad_sch (KiCad schematic)
At the start: 32 parts, among them U1 NRF52840-QIAA-R, X1 S201632M10PF10PPM, Y3 32.768KHz

Commit message: Fixed mistake in NRF52 footprint, add NAND FLASH, add NFC antenna schematic.
Parts:
- added U5: ZD25WQ16CTIGT, lcsc:SOIC-8_L4.9-W3.9-P1.27-LS6.0-BL, symbol lcsc:ZD25WQ16CTIGT
- renumbered C12 to C1, C7 to C10, C6 to C11, C5 to C12, C18 to C13, C9 to C14, C8 to C15, C13 to C16, C15 to C17, C14 to C18, C4 to C2, C16 to C3, C17 to C4, C10 to C5, C3 to C6, C11 to C7, C1 to C8, C2 to C9, L3 to L1, L1 to L3, R2 to R3, R1 to R4, Y3 to Y1
Connections:
- net +3V3: now also U5.4 (VSS), U5.8 (VCC)
- net P0.20: now also U5.5 (SI/IO0)
- net P0.21: now also U5.6 (SCLK)
- net P0.22: now also U5.3 (~{WP}/IO2)
- net P0.23: now also U5.7 (~{HOLD}/IO3)
- net P0.24: now also U5.2 (SO/IO1)
- net P0.25: now also U5.1 (~{CS})
Other:
- note added: "TODO: ADD POWER LED"
- note added: "TODO: ADD QSPI pin functions to label names"
- note added: "TODO: ADD SWD connector"
- company: (none) -> Badge.Team
- title: (none) -> Bornhack 2026

Commit message: Add original tamagotchi buttons to schematic.
Connections:
- net P0.21: now also U1.AC17 (P0.21); no longer U1.D2 (P0.21)
Changed lines of the file:
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@@
 			)
 		)
-		(property "Datasheet" "https://jlcpcb.com/partdetail/NordicSemicon-NRF52840_QIAAR/C190794"
+		(property "Datasheet" "https://lcsc.com/product-detail/Others_Nordic-Semicon_NRF52840-QIAA-R_Nordic-Semicon-NRF52840-QIAA-R_C190794.html"
 			(at 157.48 144.78 0)
 			(effects
@@
 		(pin "AD12"
 		)
-		(pin "D2"
+		(pin "AC17"
 		)
 		(pin "L24"

Commit message: PCB layout egg shape, for reference.
Parts:
- added C44: 2.2uF, Capacitor_SMD:C_0402_1005Metric, symbol Device:C_Small
Connections:
- net +3V3: now also C44.1; no longer C1.2, C10.1, C11.1, C12.1, C13.1, C14.1, C15.2, C16.2, C17.2, C18.2, C2.2, C3.1, C4.1, C5.2, C6.2, C7.2, C8.2, C9.1, TP1.1, U1.0 (EP), U1.B7 (VSS), U1.F23 (VSS_PA), U5.4 (VSS), X1.2 (GND), X1.4 (GND)
- net P0.20 renamed P0.20_QSPI_SIO_0
- net P0.21 renamed P0.21_QSPI_SCK
- net P0.22 renamed P0.22_QSPI_SIO_2
- net P0.23 renamed P0.23_QSPI_SIO_3
- net P0.24 renamed P0.24_QSPI_SIO_1
- net P0.25 renamed P0.25_QSPI_CSN
- new net GND: C1.2, C10.1, C11.1, C12.1, C13.1, C14.1, C15.2, C16.2, C17.2, C18.2, C2.2, C3.1, C4.1, C44.2, C5.2, C6.2, C7.2, C8.2, C9.1, TP1.1, U1.0 (EP), U1.B7 (VSS), U1.F23 (VSS_PA), U5.4 (VSS), X1.2 (GND), X1.4 (GND)
Changed lines of the file:
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@@
 	)
 	(junction
-		(at 24.13 31.75)
-		(diameter 0)
-		(color 0 0 0 0)
-	)
-	(junction
 		(at 31.75 62.23)
 		(diameter 0)
@@
 	)
 	(junction
+		(at 63.5 60.96)
+		(diameter 0)
+		(color 0 0 0 0)
+	)
+	(junction
 		(at 57.15 173.99)
 		(diameter 0)
@@
 	)
 	(junction
-		(at 66.04 60.96)
-		(diameter 0)
-		(color 0 0 0 0)
-	)
-	(junction
-		(at 50.8 26.67)
-		(diameter 0)
-		(color 0 0 0 0)
-	)
-	(junction
 		(at 92.71 71.12)
 		(diameter 0)
@@
 	(wire
 		(pts
-			(xy 50.8 26.67) (xy 45.72 26.67)
+			(xy 45.72 26.67) (xy 50.8 26.67)
 		)
 		(stroke
@@
 	(wire
 		(pts
-			(xy 66.04 60.96) (xy 66.04 63.5)
-		)
-		(stroke
-			(width 0)
-			(type default)
-		)
-	)
-	(wire
-		(pts
 			(xy 190.5 96.52) (xy 228.6 96.52)
 		)
@@
 	(wire
 		(pts
-			(xy 53.34 26.67) (xy 50.8 26.67)
-		)
-		(stroke
-			(width 0)
-			(type default)
-		)
-	)
-	(wire
-		(pts
 			(xy 228.6 72.39) (xy 228.6 73.66)
 		)
@@
 	(wire
 		(pts
-			(xy 21.59 31.75) (xy 24.13 31.75)
-		)
-		(stroke
-			(width 0)
-			(type default)
-		)
-	)
-	(wire
-		(pts
 			(xy 100.33 134.62) (xy 100.33 135.89)
 		)
@@
 	(wire
 		(pts
-			(xy 66.04 60.96) (xy 124.46 60.96)
+			(xy 63.5 60.96) (xy 124.46 60.96)
 		)
 		(stroke
@@
 	)
 	(label "XC1"
-		(at 53.34 26.67 0)
+		(at 46.99 26.67 0)
 		(effects
 			(font
@@
 	)
 	(label "XC2"
-		(at 21.59 31.75 0)
+		(at 24.13 31.75 0)
 		(effects
 			(font
@@
 		)
 	)
-	(hierarchical_label "P0.23"
-		(shape input)
-		(at 190.5 81.28 0)
-		(effects
-			(font
-				(size 1.27 1.27)
-			)
-			(justify left)
-		)
-	)
 	(hierarchical_label "P0.17"
 		(shape input)
@@
 		)
 	)
-	(hierarchical_label "P0.20"
-		(shape input)
-		(at 190.5 55.88 0)
-		(effects
-			(font
-				(size 1.27 1.27)
-			)
-			(justify left)
-		)
-	)
 	(hierarchical_label "P0.16"
 		(shape input)
@@
 		)
 	)
+	(hierarchical_label "P0.23_QSPI_SIO_3"
+		(shape input)
+		(at 190.5 81.28 0)
+		(effects
+			(font
+				(size 1.27 1.27)
+			)
+			(justify left)
+		)
+	)
 	(hierarchical_label "P0.26"
 		(shape input)
@@
 		)
 	)
+	(hierarchical_label "P0.21_QSPI_SCK"
+		(shape input)
+		(at 190.5 83.82 0)
+		(effects
+			(font
+				(size 1.27 1.27)
+			)
+			(justify left)
+		)
+	)
 	(hierarchical_label "P1.13"
 		(shape input)
@@
 		)
 	)
-	(hierarchical_label "P0.20"
+	(hierarchical_label "P0.22_QSPI_SIO_2"
+		(shape input)
+		(at 190.5 53.34 0)
+		(effects
+			(font
+				(size 1.27 1.27)
+			)
+			(justify left)
+		)
+	)
+	(hierarchical_label "P0.20_QSPI_SIO_0"
 		(shape input)
 		(at 147.32 177.8 0)
@@
 		)
 	)
-	(hierarchical_label "P0.23"
+	(hierarchical_label "P0.23_QSPI_SIO_3"
 		(shape input)
 		(at 147.32 172.72 0)
@@
 		)
 	)
-	(hierarchical_label "P0.22"
-		(shape input)
-		(at 190.5 53.34 0)
-		(effects
-			(font
-				(size 1.27 1.27)
-			)
-			(justify left)
-		)
-	)
 	(hierarchical_label "P0.06"
 		(shape input)
@@
 		)
 	)
+	(hierarchical_label "P0.25_QSPI_CSN"
+		(shape input)
+		(at 190.5 78.74 0)
+		(effects
+			(font
+				(size 1.27 1.27)
+			)
+			(justify left)
+		)
+	)
 	(hierarchical_label "P0.11{slash}6D_INT1"
 		(shape input)
@@
 		)
 	)
-	(hierarchical_label "P0.25"
+	(hierarchical_label "P0.25_QSPI_CSN"
 		(shape input)
 		(at 111.76 170.18 180)
@@
 		)
 	)
-	(hierarchical_label "P0.24"
+	(hierarchical_label "P0.24_QSPI_SIO_1"
 		(shape input)
 		(at 111.76 172.72 180)
@@
 		)
 	)
-	(hierarchical_label "P0.21"
-		(shape input)
-		(at 190.5 83.82 0)
-		(effects
-			(font
-				(size 1.27 1.27)
-			)
-			(justify left)
-		)
-	)
 	(hierarchical_label "P1.10"
 		(shape input)
@@
 		)
 	)
-	(hierarchical_label "P0.24"
+	(hierarchical_label "P0.20_QSPI_SIO_0"
 		(shape input)
-		(at 190.5 50.8 0)
+		(at 190.5 55.88 0)
 		(effects
 			(font
@@
 		)
 	)
-	(hierarchical_label "P0.21"
+	(hierarchical_label "P0.21_QSPI_SCK"
 		(shape input)
 		(at 147.32 175.26 0)
@@
 		)
 	)
-	(hierarchical_label "P0.25"
+	(hierarchical_label "P0.24_QSPI_SIO_1"
 		(shape input)
-		(at 190.5 78.74 0)
+		(at 190.5 50.8 0)
 		(effects
 			(font
@@
 		)
 	)
-	(hierarchical_label "P0.22"
+	(hierarchical_label "P0.22_QSPI_SIO_2"
 		(shape input)
 		(at 111.76 175.26 180)
@@
 	(symbol
 		(lib_id "power:+3V3")
-		(at 66.04 60.96 0)
+		(at 63.5 60.96 0)
 		(unit 1)
 		(exclude_from_sim no)
@@
 		(on_board yes)
 		(dnp no)
-		(fields_autoplaced yes)
 		(property "Reference" "#PWR015"
-			(at 66.04 64.77 0)
+			(at 63.5 64.77 0)
 			(effects
 				(font
@@
 		)
 		(property "Value" "+3V3"
-			(at 66.04 55.88 0)
+			(at 66.548 57.912 0)
 			(effects
 				(font
@@
 		)
 		(property "Footprint" ""
-			(at 66.04 60.96 0)
+			(at 63.5 60.96 0)
 			(effects
 				(font
@@
 		)
 		(property "Datasheet" ""
-			(at 66.04 60.96 0)
+			(at 63.5 60.96 0)
 			(effects
 				(font
@@
 		)
 		(property "Description" "Power symbol creates a global label with name \"+3V3\""
-			(at 66.04 60.96 0)
+			(at 63.5 60.96 0)
 			(effects
 				(font
@@
 	(symbol
 		(lib_id "Device:C_Small")
+		(at 63.5 63.5 0)
+		(unit 1)
+		(exclude_from_sim no)
+		(in_bom yes)
+		(on_board yes)
+		(dnp no)
+		(fields_autoplaced yes)
+		(property "Reference" "C44"
+			(at 66.04 62.2362 0)
+			(effects
+				(font
+					(size 1.27 1.27)
+				)
+				(justify left)
+			)
+		)
+		(property "Value" "2.2uF"
+			(at 66.04 64.7762 0)
+			(effects
+				(font
+					(size 1.27 1.27)
+				)
+				(justify left)
+			)
+		)
+		(property "Footprint" "Capacitor_SMD:C_0402_1005Metric"
+			(at 63.5 63.5 0)
+			(effects
+				(font
+					(size 1.27 1.27)
+				)
+				(hide yes)
+			)
+		)
+		(property "Datasheet" "https://jlcpcb.com/partdetail/13164-CL05A225MQ5NSNC/C12530"
+			(at 63.5 63.5 0)
+			(effects
+				(font
+					(size 1.27 1.27)
+				)
+				(hide yes)
+			)
+		)
+		(property "Description" "Unpolarized capacitor, small symbol"
+			(at 63.5 63.5 0)
+			(effects
+				(font
+					(size 1.27 1.27)
+				)
+				(hide yes)
+			)
+		)
+		(property "LCSC" "C12530"
+			(at 63.5 63.5 0)
+			(effects
+				(font
+					(size 1.27 1.27)
+				)
+				(hide yes)
+			)
+		)
+		(pin "2"
+		)
+		(pin "1"
+		)
+		(instances
+			(project "bornhack2026-hardware"
+				(path "/23bf5400-d19c-445b-8744-b63ebcca303d/b21ff704-9000-4580-ba18-c8ea70926409"
+					(reference "C44")
+					(unit 1)
+				)
+			)
+		)
+	)
+	(symbol
+		(lib_id "Device:C_Small")
 		(at 73.66 68.58 0)
 		(unit 1)
@@
 	(symbol
 		(lib_id "power:GND")
-		(at 66.04 63.5 0)
+		(at 63.5 66.04 0)
 		(unit 1)
 		(exclude_from_sim no)
@@
 		(fields_autoplaced yes)
 		(property "Reference" "#PWR016"
-			(at 66.04 69.85 0)
+			(at 63.5 72.39 0)
 			(effects
 				(font
@@
 		)
 		(property "Value" "GND"
-			(at 66.04 68.58 0)
+			(at 63.5 71.12 0)
 			(effects
 				(font
@@
 		)
 		(property "Footprint" ""
-			(at 66.04 63.5 0)
+			(at 63.5 66.04 0)
 			(effects
 				(font
@@
 		)
 		(property "Datasheet" ""
-			(at 66.04 63.5 0)
+			(at 63.5 66.04 0)
 			(effects
 				(font
@@
 		)
 		(property "Description" "Power symbol creates a global label with name \"GND\" , ground"
-			(at 66.04 63.5 0)
+			(at 63.5 66.04 0)
 			(effects
 				(font
@@
 		(on_board yes)
 		(dnp no)
-		(fields_autoplaced yes)
 		(property "Reference" "#PWR017"
 			(at 73.66 69.85 0)
@@
 		)
 		(property "Value" "+3V3"
-			(at 73.66 60.96 0)
+			(at 76.708 62.992 0)
 			(effects
 				(font

Commit message: Switched the LC filters from ceramic LoRa filter.
Parts:
- U5: LCSC (none) -> C5353550
Connections:
- net at R3.1: now also U1.AD6 (D+); no longer U1.B16 (D+)
Changed lines of the file:
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@@
 		(pin "L24"
 		)
-		(pin "B16"
+		(pin "AD6"
 		)
 		(pin "J1"
@@
 			)
 		)
-		(property "Datasheet" ""
+		(property "Datasheet" "https://jlcpcb.com/partdetail/Zetta-ZD25WQ16CTIGT/C5353550"
 			(at 129.54 173.99 0)
 			(effects
@@
 			(effects
 				(font
+					(size 1.27 1.27)
+				)
+				(hide yes)
+			)
+		)
+		(property "LCSC" "C5353550"
+			(at 129.54 173.99 0)
+			(effects
+				(font

Commit message: Progress, routed more stuff.
Parts:
- removed U1: NRF52840-QIAA-R, lcsc:AQFN-73_L7.0-W7.0-P0.50-BL-EP4.8, symbol lcsc:NRF52840-QIAA-R
- added U6: NRF52840-QIAA-R, lcsc:XCVR_NRF52840-QIAA-R, symbol NRF52840-QIAA-R:NRF52840-QIAA-R
- TP1, TP2, TP3, TP4, TP5, TP6: now left out of the parts list
Connections:
- net +3V3: now also C18.1, U6.A22 (VDD), U6.AD14 (VDD), U6.AD23 (VDD), U6.B1 (VDD), U6.W1 (VDD)
- net ANT: now also U6.H23 (ANT)
- net DEC4-6: now also U6.B5 (DEC4)
- net GND: now also U6.74 (VSS), U6.B7 (VSS), U6.F23 (VSS_PA)
- net P0.02: now also U6.A12 (P0.02/AIN0)
- net P0.03: now also U6.B13 (P0.03/AIN1)
- net P0.04: now also U6.J1 (P0.04/AIN2)
- net P0.05: now also U6.K2 (P0.05/AIN3)
- net P0.06: now also U6.L1 (P0.06)
- net P0.07: now also U6.M2 (P0.07/TRACECLK)
- net P0.08: now also U6.N1 (P0.08)
- net P0.09_NFC1: now also U6.L24 (P0.09/NFC1)
- net P0.10_NFC2: now also U6.J24 (P0.10/NFC2)
- net P0.11/6D_INT1: now also U6.T2 (P0.11/TRACEDATA2)
- net P0.12: now also U6.U1 (P0.12/TRACEDATA1)
- net P0.13: now also U6.AD8 (P0.13)
- net P0.14_READ_BAT: now also U6.AC9 (P0.14)
- net P0.15: now also U6.AD10 (P0.15)
- net P0.16: now also U6.AC11 (P0.16)
- net P0.17: now also U6.AD12 (P0.17)
- net P0.19: now also U6.AC15 (P0.19)
- net P0.20_QSPI_SIO_0: now also U6.AD16 (P0.20)
- net P0.21_QSPI_SCK: now also U6.AC17 (P0.21)
- net P0.22_QSPI_SIO_2: now also U6.AD18 (P0.22)
- net P0.23_QSPI_SIO_3: now also U6.AC19 (P0.23)
- net P0.24_QSPI_SIO_1: now also U6.AD20 (P0.24)
- net P0.25_QSPI_CSN: now also U6.AC21 (P0.25)
- net P0.26: now also U6.G1 (P0.26)
- net P0.27: now also U6.H2 (P0.27)
- net P0.28: now also U6.B11 (P0.28/AIN4)
- net P0.29: now also U6.A10 (P0.29/AIN5)
- net P0.30: now also U6.B9 (P0.30/AIN6)
- net P0.31: now also U6.A8 (P0.31/AIN7)
- net P1.00: now also U6.AD22 (P1.00/TRACEDATA0)
- net P1.01: now also U6.Y23 (P1.01)
- net P1.02: now also U6.W24 (P1.02)
- net P1.03: now also U6.V23 (P1.03)
- net P1.04: now also U6.U24 (P1.04)
- net P1.05: now also U6.T23 (P1.05)
- net P1.07: now also U6.P23 (P1.07)
- net P1.09: now also U6.R1 (P1.09/TRACEDATA3)
- net P1.10: now also U6.A20 (P1.10)
- net P1.11: now also U6.B19 (P1.11)
- net P1.12: now also U6.B17 (P1.12)
- net P1.13: now also U6.A16 (P1.13)
- net P1.14: now also U6.B15 (P1.14)
- net P1.15: now also U6.A14 (P1.15)
- net PWR_LED: now also U6.R24 (P1.06)
- net RESET: now also U6.AC13 (P0.18/NRESET)
- net SWDCLK: now also U6.AA24 (SWDCLK)
- net SWDIO: now also U6.AC24 (SWDIO)
- net VBUS: now also U6.AD2 (VBUS)
- net XC1: now also U6.B24 (XC1)
- net XC2: now also U6.A23 (XC2)
- net XL1: now also U6.D2 (P0.00/XL1)
- net XL2: now also U6.F2 (P0.01/XL2)
- net NRF_USB_D+: now reaches R3.1
- net NRF_USB_D+: now also U6.AD6 (D+)
- net DCC: now reaches L3.2
- net DCC: now also U6.B3 (DCC)
- net at C12.2: now also U6.D23 (DEC3)
- net at C11.2: now also U6.E24 (DEC6)
- net at C14.2: now also U6.A18 (DEC2)
- net at C17.1: now also U6.AC5 (DECUSB)
- net NRF_USB_D-: now reaches R4.1
- net NRF_USB_D-: now also U6.AD4 (D-)
- net at C10.2: now also U6.C1 (DEC1)
- net at C13.2: now also U6.N24 (DEC5)
- new net P1.08: U6.P2 (P1.08)
- new net VDDH: U6.Y2 (VDDH)
- no-connect marks 1 -> 3
Other:
- moved on the sheet: C10, C11, C12, C13, C14, C15, C16, C17, C18, C44, C8, C9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

Commit message: Bluetooth antenna should work better, NFC has IPEX for tuning.
Parts:
- added JP1: SolderJumper_2_Open, symbol Jumper:SolderJumper_2_Open
- added NT1: NetTie_2 (Feed to ground), lcsc:NetTie-2_SMD_SQ_Pad0.8mm, symbol Device:NetTie_2
Connections:
- net GND: now also NT1.1
- net at L1.1: now also JP1.1 (A), NT1.2; no longer C1.1
- net at C5.1, L2.1: now also JP1.2 (B); no longer L1.2
- new net: C1.1, L1.2
Other:
- note added: "Bluetooth antenna Implementing: https://www.lcsc.com/datasheet/C127620.pdf"
- note removed: "Bluetooth antenna"
- moved on the sheet: C1, C5, C7, L1, L2

Commit message: Routed buttons to MCU.
Parts:
- removed TP2: RESET, TestPoint:TestPoint_Pad_D1.5mm, symbol Connector:TestPoint
- TP5, TP6: footprint TestPoint:TestPoint_Pad_D1.5mm -> TestPoint:TestPoint_Pad_D1.0mm
Changed lines of the file:
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@@
-		)
-	)
-	(hierarchical_label "RESET"
-		(shape input)
-		(at 31.75 110.49 180)
-		(effects
-			(font
-				(size 1.27 1.27)
-			)
-			(justify right)
 		)
 	)
@@
 			)
 		)
-		(property "Footprint" "TestPoint:TestPoint_Pad_D1.5mm"
+		(property "Footprint" "TestPoint:TestPoint_Pad_D1.0mm"
 			(at 31.75 134.62 0)
 			(effects
@@
 			)
 		)
-		(property "Footprint" "TestPoint:TestPoint_Pad_D1.5mm"
+		(property "Footprint" "TestPoint:TestPoint_Pad_D1.0mm"
 			(at 31.75 139.7 0)
 			(effects
@@
 					(unit 1)
 				)
-			)
-		)
-	)
-	(symbol
-		(lib_id "Connector:TestPoint")
-		(at 31.75 110.49 270)
-		(unit 1)
-		(exclude_from_sim no)
-		(in_bom no)
-		(on_board yes)
-		(dnp no)
-		(fields_autoplaced yes)
-		(property "Reference" "TP2"
-			(at 36.83 109.2199 90)
-			(effects
-				(font
-					(size 1.27 1.27)
-				)
-				(justify left)
-			)
-		)
-		(property "Value" "RESET"
-			(at 36.83 111.7599 90)
-			(effects
-				(font
-					(size 1.27 1.27)
-				)
-				(justify left)
-			)
-		)
-		(property "Footprint" "TestPoint:TestPoint_Pad_D1.5mm"
-			(at 31.75 115.57 0)
-			(effects
-				(font
-					(size 1.27 1.27)
-				)
-				(hide yes)
-			)
-		)
-		(property "Datasheet" "~"
-			(at 31.75 115.57 0)
-			(effects
-				(font
-					(size 1.27 1.27)
-				)
-				(hide yes)
-			)
-		)
-		(property "Description" "test point"
-			(at 31.75 110.49 0)
-			(effects
-				(font
-					(size 1.27 1.27)
-				)
-				(hide yes)
-			)
-		)
-		(pin "1"
-		)
-		(instances
-			(project "bornhack2026-hardware"
-				(path "/23bf5400-d19c-445b-8744-b63ebcca303d/b21ff704-9000-4580-ba18-c8ea70926409"
-					(reference "TP2")
-					(unit 1)
-				)

Commit message: Fix tiny issues, add more vias.
Parts:
- added C68: 100nF, Capacitor_SMD:C_0402_1005Metric, symbol Device:C_Small
Connections:
- net +3V3: now also C68.1
- net GND: now also C68.2
Changed lines of the file:
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@@
 	)
 	(junction
+		(at 149.86 170.18)
+		(diameter 0)
+		(color 0 0 0 0)
+	)
+	(junction
 		(at 24.13 36.83)
 		(diameter 0)
@@
 	(wire
 		(pts
+			(xy 149.86 170.18) (xy 168.91 170.18)
+		)
+		(stroke
+			(width 0)
+			(type default)
+		)
+	)
+	(wire
+		(pts
 			(xy 139.7 53.34) (xy 186.69 53.34)
 		)
@@
 	(wire
 		(pts
+			(xy 168.91 170.18) (xy 168.91 176.53)
+		)
+		(stroke
+			(width 0)
+			(type default)
+		)
+	)
+	(wire
+		(pts
 			(xy 24.13 36.83) (xy 24.13 38.1)
 		)
@@
 	)
 	(symbol
+		(lib_id "Device:C_Small")
+		(at 168.91 179.07 0)
+		(unit 1)
+		(exclude_from_sim no)
+		(in_bom yes)
+		(on_board yes)
+		(dnp no)
+		(fields_autoplaced yes)
+		(property "Reference" "C68"
+			(at 171.45 177.8062 0)
+			(effects
+				(font
+					(size 1.27 1.27)
+				)
+				(justify left)
+			)
+		)
+		(property "Value" "100nF"
+			(at 171.45 180.3462 0)
+			(effects
+				(font
+					(size 1.27 1.27)
+				)
+				(justify left)
+			)
+		)
+		(property "Footprint" "Capacitor_SMD:C_0402_1005Metric"
+			(at 168.91 179.07 0)
+			(effects
+				(font
+					(size 1.27 1.27)
+				)
+				(hide yes)
+			)
+		)
+		(property "Datasheet" "https://jlcpcb.com/partdetail/1877-CL05B104KO5NNNC/C1525"
+			(at 168.91 179.07 0)
+			(effects
+				(font
+					(size 1.27 1.27)
+				)
+				(hide yes)
+			)
+		)
+		(property "Description" "Unpolarized capacitor, small symbol"
+			(at 168.91 179.07 0)
+			(effects
+				(font
+					(size 1.27 1.27)
+				)
+				(hide yes)
+			)
+		)
+		(property "LCSC" "C1525"
+			(at 168.91 179.07 90)
+			(effects
+				(font
+					(size 1.27 1.27)
+				)
+				(hide yes)
+			)
+		)
+		(pin "2"
+		)
+		(pin "1"
+		)
+		(instances
+			(project "bornhack2026-hardware"
+				(path "/23bf5400-d19c-445b-8744-b63ebcca303d/b21ff704-9000-4580-ba18-c8ea70926409"
+					(reference "C68")
+					(unit 1)
+				)
+			)
+		)
+	)
+	(symbol
 		(lib_id "power:GND")
 		(at 175.26 29.21 0)
@@
 					(unit 1)
 				)
+			)
+		)
+	)
+	(symbol
+		(lib_id "power:GND")
+		(at 168.91 181.61 0)
+		(unit 1)
+		(exclude_from_sim no)
+		(in_bom yes)
+		(on_board yes)
+		(dnp no)
+		(fields_autoplaced yes)
+		(property "Reference" "#PWR080"
+			(at 168.91 187.96 0)
+			(effects
+				(font
+					(size 1.27 1.27)
+				)
+				(hide yes)
+			)
+		)
+		(property "Value" "GND"
+			(at 168.91 186.69 0)
+			(effects
+				(font
+					(size 1.27 1.27)
+				)
+			)
+		)
+		(property "Footprint" ""
+			(at 168.91 181.61 0)
+			(effects
+				(font
+					(size 1.27 1.27)
+				)
+				(hide yes)
+			)
+		)
+		(property "Datasheet" ""
+			(at 168.91 181.61 0)
+			(effects
+				(font
+					(size 1.27 1.27)
+				)
+				(hide yes)
+			)
+		)
+		(property "Description" "Power symbol creates a global label with name \"GND\" , ground"
+			(at 168.91 181.61 0)
+			(effects
+				(font
+					(size 1.27 1.27)
+				)
+				(hide yes)
+			)
+		)
+		(pin "1"
+		)
+		(instances
+			(project "bornhack2026-hardware"
+				(path "/23bf5400-d19c-445b-8744-b63ebcca303d/b21ff704-9000-4580-ba18-c8ea70926409"
+					(reference "#PWR080")
+					(unit 1)
+				)
