File: nrf52840_mcu.kicad_sch (KiCad schematic)
At the start: 36 parts, among them J3 Conn_01x05, U5 ZD25WQ16CTIGT, U6 NRF52840-QIAA-R, X1 S201632M10PF10PPM, X3 32.768KHz

Commit message: Squashed in new battery connector, made NFC coil and Bluetooth fit as good and bad as possible.
Parts:
- removed TP5: NFC2, TestPoint:TestPoint_Pad_D1.0mm, symbol Connector:TestPoint
- removed TP6: NFC1, TestPoint:TestPoint_Pad_D1.0mm, symbol Connector:TestPoint
Changed lines of the file:
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@@
-		)
-	)
-	(hierarchical_label "P0.10_NFC2"
-		(shape input)
-		(at 34.29 53.34 180)
-		(effects
-			(font
-				(size 1.27 1.27)
-			)
-			(justify right)
 		)
 	)
@@
 			)
 			(justify left)
-		)
-	)
-	(hierarchical_label "P0.09_NFC1"
-		(shape input)
-		(at 34.29 58.42 180)
-		(effects
-			(font
-				(size 1.27 1.27)
-			)
-			(justify right)
 		)
 	)
@@
 	)
 	(symbol
-		(lib_id "Connector:TestPoint")
-		(at 34.29 53.34 270)
-		(unit 1)
-		(exclude_from_sim no)
-		(in_bom no)
-		(on_board yes)
-		(dnp no)
-		(fields_autoplaced yes)
-		(property "Reference" "TP5"
-			(at 39.37 52.0699 90)
-			(effects
-				(font
-					(size 1.27 1.27)
-				)
-				(justify left)
-				(hide yes)
-			)
-		)
-		(property "Value" "NFC2"
-			(at 39.37 54.6099 90)
-			(effects
-				(font
-					(size 1.27 1.27)
-				)
-				(justify left)
-			)
-		)
-		(property "Footprint" "TestPoint:TestPoint_Pad_D1.0mm"
-			(at 34.29 58.42 0)
-			(effects
-				(font
-					(size 1.27 1.27)
-				)
-				(hide yes)
-			)
-		)
-		(property "Datasheet" "~"
-			(at 34.29 58.42 0)
-			(effects
-				(font
-					(size 1.27 1.27)
-				)
-				(hide yes)
-			)
-		)
-		(property "Description" "test point"
-			(at 34.29 53.34 0)
-			(effects
-				(font
-					(size 1.27 1.27)
-				)
-				(hide yes)
-			)
-		)
-		(property "Resource" ""
-			(at 34.29 53.34 90)
-			(effects
-				(font
-					(size 1.27 1.27)
-				)
-				(hide yes)
-			)
-		)
-		(pin "1"
-		)
-		(instances
-			(project "bornhack2026-hardware"
-				(path "/23bf5400-d19c-445b-8744-b63ebcca303d/b21ff704-9000-4580-ba18-c8ea70926409"
-					(reference "TP5")
-					(unit 1)
-				)
-			)
-		)
-	)
-	(symbol
 		(lib_id "power:GND")
 		(at 179.07 144.78 0)
@@
 					(unit 1)
 				)
-			)
-		)
-	)
-	(symbol
-		(lib_id "Connector:TestPoint")
-		(at 34.29 58.42 270)
-		(unit 1)
-		(exclude_from_sim no)
-		(in_bom no)
-		(on_board yes)
-		(dnp no)
-		(fields_autoplaced yes)
-		(property "Reference" "TP6"
-			(at 39.37 57.1499 90)
-			(effects
-				(font
-					(size 1.27 1.27)
-				)
-				(justify left)
-				(hide yes)
-			)
-		)
-		(property "Value" "NFC1"
-			(at 39.37 59.6899 90)
-			(effects
-				(font
-					(size 1.27 1.27)
-				)
-				(justify left)
-			)
-		)
-		(property "Footprint" "TestPoint:TestPoint_Pad_D1.0mm"
-			(at 34.29 63.5 0)
-			(effects
-				(font
-					(size 1.27 1.27)
-				)
-				(hide yes)
-			)
-		)
-		(property "Datasheet" "~"
-			(at 34.29 63.5 0)
-			(effects
-				(font
-					(size 1.27 1.27)
-				)
-				(hide yes)
-			)
-		)
-		(property "Description" "test point"
-			(at 34.29 58.42 0)
-			(effects
-				(font
-					(size 1.27 1.27)
-				)
-				(hide yes)
-			)
-		)
-		(property "Resource" ""
-			(at 34.29 58.42 90)
-			(effects
-				(font
-					(size 1.27 1.27)
-				)
-				(hide yes)
-			)
-		)
-		(pin "1"
-		)
-		(instances
-			(project "bornhack2026-hardware"
-				(path "/23bf5400-d19c-445b-8744-b63ebcca303d/b21ff704-9000-4580-ba18-c8ea70926409"
-					(reference "TP6")
-					(unit 1)
-				)

Commit message: Replaced joystick with alternatie (cheaper) part.
Parts:
- AE2: footprint RF_Antenna:Texas_SWRA117D_2.4GHz_Left -> RF_Antenna:Texas_SWRA117D_2.4GHz_Right
- J3: now left out of the parts list
Changed lines of the file:
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@@
 		(unit 1)
 		(exclude_from_sim no)
-		(in_bom yes)
+		(in_bom no)
 		(on_board yes)
 		(dnp yes)
@@
 			)
 		)
-		(property "Footprint" "RF_Antenna:Texas_SWRA117D_2.4GHz_Left"
+		(property "Footprint" "RF_Antenna:Texas_SWRA117D_2.4GHz_Right"
 			(at 39.37 143.51 0)
 			(effects

Commit message: Add batteryvoltage and charge indicator circuit.
Parts:
- R3, R4: value 33 -> 0; LCSC C25105 -> C17168
Connections:
- net P1.06: no longer names the net of U6.R24 (P1.06)
- no-connect marks 1 -> 3
Other:
- note removed: "<-- Note: DK uses 10uF in series with 15nF here"
Changed lines of the file:
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@@
 		)
 	)
-	(text "<-- Note: DK uses 10uF in series with 15nF here"
-		(exclude_from_sim no)
-		(at 222.504 47.244 0)
-		(effects
-			(font
-				(size 1.27 1.27)
-				(thickness 0.254)
-				(bold yes)
-				(italic yes)
-				(color 255 0 0 1)
-			)
-		)
-	)
 	(text "Main MCU Clock oscillator"
 		(exclude_from_sim no)
@@
 	)
 	(no_connect
+		(at 173.99 92.71)
+	)
+	(no_connect
 		(at 173.99 49.53)
 	)
+	(no_connect
+		(at 187.96 110.49)
+	)
 	(wire
 		(pts
@@
 	)
 	(hierarchical_label "USB_D+"
-		(shape bidirectional)
+		(shape input)
 		(at 207.01 133.35 0)
 		(effects
@@
 		)
 	)
-	(hierarchical_label "P0.21_QSPI_SCK"
-		(shape input)
-		(at 118.11 110.49 180)
-		(effects
-			(font
-				(size 1.27 1.27)
-			)
-			(justify right)
-		)
-	)
 	(hierarchical_label "P1.13"
 		(shape input)
@@
 		)
 	)
-	(hierarchical_label "P1.06"
-		(shape input)
-		(at 173.99 92.71 0)
-		(effects
-			(font
-				(size 1.27 1.27)
-			)
-			(justify left)
-		)
-	)
 	(hierarchical_label "P0.23_QSPI_SIO_3"
 		(shape input)
@@
 		)
 	)
+	(hierarchical_label "P0.21_QSPI_SCK"
+		(shape input)
+		(at 118.11 110.49 180)
+		(effects
+			(font
+				(size 1.27 1.27)
+			)
+			(justify right)
+		)
+	)
 	(hierarchical_label "P0.03"
 		(shape input)
@@
 			)
 		)
-		(property "Value" "33"
+		(property "Value" "0"
 			(at 195.326 134.62 90)
 			(effects
@@
 			)
 		)
-		(property "Datasheet" "https://jlcpcb.com/partdetail/25848-0402WGF330JTCE/C25105"
+		(property "Datasheet" "https://jlcpcb.com/partdetail/17853-0402WGF0000TCE/C17168"
 			(at 193.04 133.35 0)
 			(effects
@@
 			)
 		)
-		(property "LCSC" "C25105"
+		(property "LCSC" "C17168"
 			(at 193.04 133.35 90)
 			(effects
@@
 			)
 		)
-		(property "Value" "33"
+		(property "Value" "0"
 			(at 203.2 137.16 90)
 			(effects
@@
 			)
 		)
-		(property "Datasheet" "https://jlcpcb.com/partdetail/25848-0402WGF330JTCE/C25105"
+		(property "Datasheet" "https://jlcpcb.com/partdetail/17853-0402WGF0000TCE/C17168"
 			(at 200.66 135.89 0)
 			(effects
@@
 			)
 		)
-		(property "LCSC" "C25105"
+		(property "LCSC" "C17168"
 			(at 200.66 135.89 90)
 			(effects

Commit message: Cleaned up pinout
Connections:
- net P0.02 renamed P0.02/AIN0
- net P0.03 renamed P0.03/AIN1
- net P0.04 renamed P0.04/AIN1
- net P0.05 renamed P0.05/AIN2
- net P0.14_READ_BAT renamed P0.14
- net P0.28 renamed P0.28/AIN4
- net P0.29 renamed P0.29/AIN5
- net P0.30 renamed P0.30/AIN6
- net P0.31 renamed P0.31/AIN7
Other:
- moved on the sheet: C73
Changed lines of the file:
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@@
 	)
 	(junction
-		(at 205.74 67.31)
-		(diameter 0)
-		(color 0 0 0 0)
-	)
-	(junction
 		(at 53.34 153.67)
 		(diameter 0)
@@
 	)
 	(junction
+		(at 207.01 62.23)
+		(diameter 0)
+		(color 0 0 0 0)
+	)
+	(junction
 		(at 196.85 67.31)
 		(diameter 0)
@@
 	)
 	(junction
+		(at 207.01 67.31)
+		(diameter 0)
+		(color 0 0 0 0)
+	)
+	(junction
 		(at 198.12 25.4)
 		(diameter 0)
@@
 	)
 	(junction
-		(at 196.85 62.23)
-		(diameter 0)
-		(color 0 0 0 0)
-	)
-	(junction
 		(at 250.19 54.61)
 		(diameter 0)
@@
 	(wire
 		(pts
-			(xy 205.74 76.2) (xy 205.74 80.01)
+			(xy 207.01 76.2) (xy 207.01 80.01)
 		)
 		(stroke
@@
 	(wire
 		(pts
-			(xy 205.74 67.31) (xy 237.49 67.31)
+			(xy 207.01 67.31) (xy 237.49 67.31)
 		)
 		(stroke
@@
 	(wire
 		(pts
-			(xy 196.85 80.01) (xy 205.74 80.01)
+			(xy 196.85 80.01) (xy 207.01 80.01)
 		)
 		(stroke
@@
 	(wire
 		(pts
-			(xy 205.74 67.31) (xy 205.74 71.12)
+			(xy 207.01 67.31) (xy 207.01 71.12)
 		)
 		(stroke
@@
 	(wire
 		(pts
-			(xy 173.99 62.23) (xy 196.85 62.23)
+			(xy 173.99 62.23) (xy 207.01 62.23)
 		)
 		(stroke
@@
 	(wire
 		(pts
-			(xy 196.85 67.31) (xy 205.74 67.31)
+			(xy 196.85 67.31) (xy 207.01 67.31)
 		)
 		(stroke
@@
 	(wire
 		(pts
-			(xy 196.85 62.23) (xy 196.85 67.31)
+			(xy 207.01 46.99) (xy 207.01 62.23)
 		)
 		(stroke
@@
 	(wire
 		(pts
-			(xy 26.67 33.02) (xy 31.75 33.02)
+			(xy 207.01 62.23) (xy 207.01 67.31)
 		)
 		(stroke
@@
 	(wire
 		(pts
-			(xy 67.31 161.29) (xy 102.87 161.29)
+			(xy 26.67 33.02) (xy 31.75 33.02)
 		)
 		(stroke
@@
 	(wire
 		(pts
-			(xy 207.01 46.99) (xy 207.01 62.23)
+			(xy 67.31 161.29) (xy 102.87 161.29)
 		)
 		(stroke
@@
 	(wire
 		(pts
-			(xy 207.01 62.23) (xy 196.85 62.23)
-		)
-		(stroke
-			(width 0)
-			(type default)
-		)
-	)
-	(wire
-		(pts
 			(xy 177.8 25.4) (xy 184.15 25.4)
 		)
@@
 		)
 	)
-	(hierarchical_label "P0.14_READ_BAT"
+	(hierarchical_label "P0.14"
 		(shape input)
 		(at 118.11 92.71 180)
@@
 		)
 	)
-	(hierarchical_label "P0.30"
+	(hierarchical_label "P0.30{slash}AIN6"
 		(shape input)
 		(at 118.11 133.35 180)
@@
 		)
 	)
-	(hierarchical_label "P0.04"
+	(hierarchical_label "P0.04{slash}AIN1"
 		(shape input)
 		(at 118.11 67.31 180)
@@
 		)
 	)
-	(hierarchical_label "P0.03"
+	(hierarchical_label "P0.03{slash}AIN1"
 		(shape input)
 		(at 118.11 64.77 180)
@@
 		)
 	)
-	(hierarchical_label "P0.02"
+	(hierarchical_label "P0.02{slash}AIN0"
 		(shape input)
 		(at 118.11 62.23 180)
@@
 		)
 	)
-	(hierarchical_label "P0.31"
+	(hierarchical_label "P0.31{slash}AIN7"
 		(shape input)
 		(at 118.11 135.89 180)
@@
 		)
 	)
-	(hierarchical_label "P0.05"
+	(hierarchical_label "P0.05{slash}AIN2"
 		(shape input)
 		(at 118.11 69.85 180)
@@
 		)
 	)
-	(hierarchical_label "P0.29"
+	(hierarchical_label "P0.29{slash}AIN5"
 		(shape input)
 		(at 118.11 130.81 180)
@@
 		)
 	)
-	(hierarchical_label "P0.28"
+	(hierarchical_label "P0.28{slash}AIN4"
 		(shape input)
 		(at 118.11 128.27 180)
@@
 	(symbol
 		(lib_id "Device:C_Small")
-		(at 205.74 73.66 0)
+		(at 207.01 73.66 0)
 		(unit 1)
 		(exclude_from_sim no)
@@
 		(dnp no)
 		(property "Reference" "C73"
-			(at 212.344 75.184 0)
+			(at 213.614 75.184 0)
 			(effects
 				(font
@@
 		)
 		(property "Value" "47nF"
-			(at 212.344 72.644 0)
+			(at 213.614 72.644 0)
 			(effects
 				(font
@@
 		)
 		(property "Footprint" "Capacitor_SMD:C_0402_1005Metric"
-			(at 205.74 73.66 0)
+			(at 207.01 73.66 0)
 			(effects
 				(font
@@
 		)
 		(property "Datasheet" "https://jlcpcb.com/partdetail/83376-0402B473K500NT/C82219"
-			(at 205.74 73.66 0)
+			(at 207.01 73.66 0)
 			(effects
 				(font
@@
 		)
 		(property "Description" "Unpolarized capacitor, small symbol"
-			(at 205.74 73.66 0)
+			(at 207.01 73.66 0)
 			(effects
 				(font
@@
 		)
 		(property "LCSC" "C82219"
-			(at 205.74 73.66 90)
+			(at 207.01 73.66 90)
 			(effects
 				(font
@@
 		)
 		(property "Resource" ""
-			(at 205.74 73.66 0)
+			(at 207.01 73.66 0)
 			(effects
 				(font

Commit message: 10-pin SWD interface added.
Parts:
- removed J3: Conn_01x05, Connector_PinHeader_2.54mm:PinHeader_1x05_P2.54mm_Vertical, symbol Connector_Generic:Conn_01x05
- added J4: Conn_02x05_Odd_Even, Connector_PinHeader_1.27mm:PinHeader_2x05_P1.27mm_Vertical_SMD, symbol Connector_Generic:Conn_02x05_Odd_Even
Connections:
- net +3V3: now also J4.1 (Pin_1)
- net GND: now also J4.3 (Pin_3), J4.5 (Pin_5), J4.9 (Pin_9)
- net P1.00: now also J4.6 (Pin_6)
- net RESET: now also J4.10 (Pin_10)
- net SWDCLK: now also J4.4 (Pin_4)
- net SWDIO: now also J4.2 (Pin_2)
- no-connect marks 3 -> 5
Other:
- note added: "SWD debug interface"

Commit message: Moved SWR connector to other side of board, reversed on/off switch UP -> ON.
Parts:
- added R36, R37, R38: 10k, Resistor_SMD:R_0402_1005Metric, symbol symbols:R
- added TP1: GND, TestPoint:TestPoint_Pad_D1.0mm, symbol Connector:TestPoint
- added TP2: SWDCLK, TestPoint:TestPoint_Pad_D1.0mm, symbol Connector:TestPoint
- added TP3: SWO, TestPoint:TestPoint_Pad_D1.0mm, symbol Connector:TestPoint
- added TP4: SWDIO, TestPoint:TestPoint_Pad_D1.0mm, symbol Connector:TestPoint
Connections:
- net +3V3: now also R36.2, R38.2
- net GND: now also R37.1, TP1.1
- net SWDCLK: now also R37.2, TP2.1
- net SWDIO: now also R36.1, TP4.1
- net P1.00 renamed P1.00_SWO
- net P1.00_SWO: now also R38.1, TP3.1
Other:
- moved on the sheet: J4

Commit message: Fixed PCBA rotations in using component property.
Parts:
- AE2, TP1, TP2, TP3, TP4: now left out of the parts list
- U5: FT Rotation Offset (none) -> 90
- U6: FT Rotation Offset (none) -> 270
Connections:
- net RESET renamed RESETn
Changed lines of the file:
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@@
 		)
 	)
-	(hierarchical_label "RESET"
+	(hierarchical_label "RESETn"
 		(shape input)
 		(at 118.11 102.87 180)
@@
 		)
 	)
-	(hierarchical_label "RESET"
+	(hierarchical_label "RESETn"
 		(shape output)
 		(at 48.26 90.17 0)
@@
 			)
 		)
+		(property "FT Rotation Offset" "270"
+			(at 146.05 90.17 0)
+			(effects
+				(font
+					(size 1.27 1.27)
+				)
+				(hide yes)
+			)
+		)
 		(pin "A16"
 		)
@@
 		(unit 1)
 		(exclude_from_sim no)
-		(in_bom yes)
+		(in_bom no)
 		(on_board yes)
 		(dnp no)
@@
 			)
 		)
+		(property "FT Rotation Offset" "90"
+			(at 129.54 181.61 0)
+			(effects
+				(font
+					(size 1.27 1.27)
+				)
+				(hide yes)
+			)
+		)
 		(pin "6"
 		)
@@
 		(unit 1)
 		(exclude_from_sim no)
-		(in_bom yes)
+		(in_bom no)
 		(on_board yes)
 		(dnp no)
@@
 		(unit 1)
 		(exclude_from_sim no)
-		(in_bom yes)
+		(in_bom no)
 		(on_board yes)
 		(dnp no)
@@
 		(unit 1)
 		(exclude_from_sim no)
-		(in_bom yes)
+		(in_bom no)
 		(on_board yes)
 		(dnp no)
@@
 		(unit 1)
 		(exclude_from_sim no)
-		(in_bom yes)
+		(in_bom no)
 		(on_board yes)
 		(dnp no)

Commit message: Optimized design to use more basic components.
Parts:
- AE2, NT3, TP1, TP2, TP3, TP4: now not fitted
- C3, C4: value 10n -> 10nF; LCSC C1524 -> C15195
- L14: LCSC C27143 -> C381880
- L2: LCSC C963987 -> C86065
- L3: LCSC C194437 -> C1035
- X1: value S201632M10PF10PPM -> S201632M10PF10PPM 32MHz
