File: bornhack2026-hardware.kicad_sch (KiCad schematic)
At the start: 4 parts, among them J1 USB device

Commit message: Routed buttons to MCU.
Parts:
- added H1, H2, H3: MountingHole_Pad, MountingHole:MountingHole_2.2mm_M2_DIN965_Pad, symbol Mechanical:MountingHole_Pad
- added L13: 400-1000MHZ-CHIP(B&T-1503), lcsc:ANT-SMD_L15.0-W3.0, symbol lcsc:400-1000MHZ-CHIP(B&T-1503)
- added R31, R32: 0, Resistor_SMD:R_0402_1005Metric, symbol Device:R_Small
Connections:
- net GND: now also H1.1, H2.1, H3.1
- net SX1262 LoRA/LORA_ANT: now also R31.2, R32.2; no longer RF1.1
- new net: R31.1, RF1.1
- new net: L13.1 (ANT), R32.1
- no-connect marks 4 -> 11
Other:
- sheet INPUT ports: added BTN_JOY_DOWN, BTN_JOY_FIRE, BTN_JOY_LEFT, BTN_JOY_RIGHT, BTN_JOY_UP; removed none
- moved on the sheet: RF1

Commit message: Fix tiny issues, add more vias.
Other:
- sheet POWER ports: added CHRG, PS_SYNC; removed none
Changed lines of the file:
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@@
 	(wire
 		(pts
+			(xy 137.16 88.9) (xy 121.92 88.9)
+		)
+		(stroke
+			(width 0)
+			(type default)
+		)
+	)
+	(wire
+		(pts
 			(xy 116.84 73.66) (xy 137.16 73.66)
 		)
@@
 	(wire
 		(pts
+			(xy 246.38 38.1) (xy 231.14 38.1)
+		)
+		(stroke
+			(width 0)
+			(type default)
+		)
+	)
+	(wire
+		(pts
 			(xy 80.01 90.17) (xy 100.33 90.17)
 		)
@@
 		)
 	)
+	(label "P0.17_PS_SYNC"
+		(at 121.92 88.9 0)
+		(effects
+			(font
+				(size 1.27 1.27)
+			)
+			(justify left bottom)
+		)
+	)
 	(label "P1.15_LORA_MOSI"
 		(at 100.33 82.55 180)
@@
 		)
 	)
+	(label "P0.17_PS_SYNC"
+		(at 231.14 38.1 0)
+		(effects
+			(font
+				(size 1.27 1.27)
+			)
+			(justify left bottom)
+		)
+	)
 	(label "P0.29_LORA_SPI_NSS"
 		(at 100.33 90.17 180)
@@
 	(sheet
 		(at 246.38 24.13)
-		(size 25.4 12.7)
+		(size 25.4 17.78)
 		(exclude_from_sim no)
 		(in_bom yes)
@@
 		)
 		(property "Sheetfile" "power.kicad_sch"
-			(at 246.38 37.4146 0)
+			(at 246.38 42.4946 0)
 			(effects
 				(font
@@
 			)
 		)
-		(pin "+3V3_OUT" input
-			(at 271.78 33.02 0)
-			(effects
-				(font
-					(size 1.27 1.27)
-				)
-				(justify right)
-			)
-		)
 		(pin "VBAT" input
 			(at 271.78 27.94 0)
@@
 			)
 		)
+		(pin "CHRG" output
+			(at 271.78 38.1 0)
+			(effects
+				(font
+					(size 1.27 1.27)
+				)
+				(justify right)
+			)
+		)
+		(pin "PS_SYNC" input
+			(at 246.38 38.1 180)
+			(effects
+				(font
+					(size 1.27 1.27)
+				)
+				(justify left)
+			)
+		)
+		(pin "+3V3_OUT" output
+			(at 271.78 33.02 0)
+			(effects
+				(font
+					(size 1.27 1.27)
+				)
+				(justify right)
+			)
+		)

Commit message: Moved SMA-connector Lora for VNA testing.
Parts:
- R31: now fitted; now in the parts list
Connections:
- net SX1262 LoRA/LORA_ANT: no longer R32.2
- net at R31.1, RF1.1: now also R32.2
Other:
- moved on the sheet: L13, R32, RF1

Commit message: WIP: Moved buttons, battery.
Parts:
- added C69: 0, Capacitor_SMD:C_0402_1005Metric, symbol Device:C_Small
- added C70, C71: DNP, Capacitor_SMD:C_0402_1005Metric, symbol Device:C_Small
- L13: value 400-1000MHZ-CHIP(B&T-1503) -> 866MHz LoRa antenna
Connections:
- net GND: now also C70.2, C71.2
- net at L13.1 (ANT): now also C69.1, C70.1; no longer R32.1
- new net: C69.2, C71.1, R32.1
Other:
- note added: "Prototype antenna or SMA"
- moved on the sheet: L13, R31, R32, RF1

Commit message: Connected up buttons, labeled buttons, added some via stitching.
Other:
- sheet INPUT ports: added BTN_EXECUTE; removed BTN_SELECT
Changed lines of the file:
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@@
 	)
 	(label "BTN_JOY_RIGHT"
-		(at 200.66 57.15 180)
+		(at 200.66 59.69 180)
 		(effects
 			(font
@@
 		)
 	)
-	(label "BTN_SELECT"
+	(label "BTN_EXECUTE"
 		(at 200.66 69.85 180)
 		(effects
@@
 	)
 	(label "BTN_JOY_DOWN"
-		(at 200.66 62.23 180)
+		(at 200.66 57.15 180)
 		(effects
 			(font
@@
 	)
 	(label "BTN_JOY_LEFT"
-		(at 200.66 64.77 180)
+		(at 200.66 67.31 180)
 		(effects
 			(font
@@
 	)
 	(label "BTN_JOY_UP"
-		(at 200.66 59.69 180)
+		(at 200.66 62.23 180)
 		(effects
 			(font
@@
 		)
 	)
-	(label "BTN_SELECT"
+	(label "BTN_EXECUTE"
 		(at 96.52 153.67 180)
 		(effects
@@
 	)
 	(label "BTN_JOY_FIRE"
-		(at 200.66 67.31 180)
+		(at 200.66 64.77 180)
 		(effects
 			(font
@@
 		(on_board yes)
 		(dnp no)
+		(fields_autoplaced yes)
 		(property "Reference" "J1"
-			(at 248.92 102.87 0)
+			(at 248.92 101.6 0)
 			(effects
 				(font
@@
 		)
 		(property "Value" "USB device"
-			(at 248.92 105.156 0)
+			(at 248.92 104.14 0)
 			(effects
 				(font
@@
 			)
 		)
-		(pin "BTN_SELECT" output
+		(pin "BTN_EXECUTE" output
 			(at 76.2 153.67 0)
 			(effects

Commit message: Remove mounting hole REFDES.
Parts:
- added N1: Board edge + art, lcsc:white-egg-svg2shenzhen, symbol Mechanical:Housing
Changed lines of the file:
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@@
+	)
+	(symbol
+		(lib_id "Mechanical:Housing")
+		(at 132.08 171.45 0)
+		(unit 1)
+		(exclude_from_sim no)
+		(in_bom yes)
+		(on_board yes)
+		(dnp no)
+		(fields_autoplaced yes)
+		(property "Reference" "N1"
+			(at 135.89 170.4974 0)
+			(effects
+				(font
+					(size 1.27 1.27)
+				)
+				(justify left)
+			)
+		)
+		(property "Value" "Board edge + art"
+			(at 135.89 173.0374 0)
+			(effects
+				(font
+					(size 1.27 1.27)
+				)
+				(justify left)
+			)
+		)
+		(property "Footprint" "lcsc:white-egg-svg2shenzhen"
+			(at 133.35 170.18 0)
+			(effects
+				(font
+					(size 1.27 1.27)
+				)
+				(hide yes)
+			)
+		)
+		(property "Datasheet" "~"
+			(at 133.35 170.18 0)
+			(effects
+				(font
+					(size 1.27 1.27)
+				)
+				(hide yes)
+			)
+		)
+		(property "Description" "Board edge + art"
+			(at 132.08 171.45 0)
+			(effects
+				(font
+					(size 1.27 1.27)
+				)
+				(hide yes)
+			)
+		)
+		(instances
+			(project ""
+				(path "/23bf5400-d19c-445b-8744-b63ebcca303d"
+					(reference "N1")
+					(unit 1)
+				)
+			)
+		)
 	)
 	(symbol

Commit message: Checked PCBA for JLCPCB.
Parts:
- L13: LCSC (none) -> C41368044
- N1: now left out of the parts list
Changed lines of the file:
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@@
 		(unit 1)
 		(exclude_from_sim no)
-		(in_bom yes)
+		(in_bom no)
 		(on_board yes)
 		(dnp no)
@@
 			(effects
 				(font
+					(size 1.27 1.27)
+				)
+				(hide yes)
+			)
+		)
+		(property "LCSC" "C41368044"
+			(at 40.64 21.59 0)
+			(effects
+				(font

Commit message: Changed antennas for PCB antennas, move stuff because of it.
Parts:
- removed C69: 0, Capacitor_SMD:C_0402_1005Metric, symbol Device:C_Small
- removed C70, C71: DNP, Capacitor_SMD:C_0402_1005Metric, symbol Device:C_Small
- removed L13: 866MHz LoRa antenna, lcsc:ANT-SMD_L15.0-W3.0, symbol lcsc:400-1000MHZ-CHIP(B&T-1503)
- added AE3: Antenna_Dipole, lcsc:Texas_SWRA416_868MHz_915MHz_right, symbol Device:Antenna
- N1: now not fitted
Connections:
- net at R32.1: now also AE3.1 (A)
- no-connect marks 11 -> 10
Other:
- note added: "JLCPCB Inpedance control Stackup used: JLC04161H-7628 Stackup Impendance calculator: https://jlcpcb.com/pcb-impedance-calculator"
