File: bornhack2026-hardware.kicad_sch (KiCad schematic)
At the start: 11 parts, among them J1 USB device

Commit message: Changed NFC coil + tune C's to match better with datasheet.
Parts:
- added N2: Ranzbak, defeest:goatse_01, symbol Mechanical:Housing
- AE3: footprint lcsc:Texas_SWRA416_868MHz_915MHz_right -> lcsc:Texas_SWRA416_868MHz_915MHz_right_v2; now not fitted; now left out of the parts list
Changed lines of the file:
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@@
+			)
+		)
+		(property "Resource" ""
+			(at 269.24 114.3 90)
+			(effects
+				(font
+					(size 1.27 1.27)
+				)
+				(hide yes)
 			)
 		)
@@
 			)
 		)
+		(property "Resource" ""
+			(at 35.56 173.99 0)
+			(effects
+				(font
+					(size 1.27 1.27)
+				)
+				(hide yes)
+			)
+		)
 		(pin "1"
 		)
@@
 			)
 		)
+		(property "Resource" ""
+			(at 82.55 173.99 0)
+			(effects
+				(font
+					(size 1.27 1.27)
+				)
+				(hide yes)
+			)
+		)
 		(pin "1"
 		)
@@
 			)
 		)
+		(property "Resource" ""
+			(at 59.69 173.99 0)
+			(effects
+				(font
+					(size 1.27 1.27)
+				)
+				(hide yes)
+			)
+		)
 		(pin "1"
 		)
@@
 		(unit 1)
 		(exclude_from_sim no)
-		(in_bom yes)
-		(on_board yes)
-		(dnp no)
+		(in_bom no)
+		(on_board yes)
+		(dnp yes)
 		(fields_autoplaced yes)
 		(property "Reference" "AE3"
@@
 			)
 		)
-		(property "Footprint" "lcsc:Texas_SWRA416_868MHz_915MHz_right"
+		(property "Footprint" "lcsc:Texas_SWRA416_868MHz_915MHz_right_v2"
 			(at 40.64 34.29 0)
 			(effects
@@
 		)
 		(property "Description" "Antenna"
+			(at 40.64 34.29 0)
+			(effects
+				(font
+					(size 1.27 1.27)
+				)
+				(hide yes)
+			)
+		)
+		(property "Resource" ""
 			(at 40.64 34.29 0)
 			(effects
@@
 			)
 		)
+		(property "Resource" ""
+			(at 40.64 57.15 90)
+			(effects
+				(font
+					(size 1.27 1.27)
+				)
+				(hide yes)
+			)
+		)
 		(pin "1"
 		)
@@
 		)
 		(property "LCSC" "C22467595"
+			(at 29.21 52.07 0)
+			(effects
+				(font
+					(size 1.27 1.27)
+				)
+				(hide yes)
+			)
+		)
+		(property "Resource" ""
 			(at 29.21 52.07 0)
 			(effects
@@
 			)
 		)
+		(property "Resource" ""
+			(at 132.08 171.45 0)
+			(effects
+				(font
+					(size 1.27 1.27)
+				)
+				(hide yes)
+			)
+		)
 		(instances
 			(project ""
@@
 			)
 		)
+		(property "Resource" ""
+			(at 40.64 48.26 90)
+			(effects
+				(font
+					(size 1.27 1.27)
+				)
+				(hide yes)
+			)
+		)
 		(pin "1"
 		)
@@
 		(property "LCSC" "C25905"
 			(at 269.24 116.84 0)
+			(effects
+				(font
+					(size 1.27 1.27)
+				)
+				(hide yes)
+			)
+		)
+		(property "Resource" ""
+			(at 269.24 116.84 90)
 			(effects
 				(font
@@
 			)
 		)
+		(property "Resource" ""
+			(at 248.92 124.46 0)
+			(effects
+				(font
+					(size 1.27 1.27)
+				)
+				(hide yes)
+			)
+		)
 		(pin "A1"
 		)
@@
 					(unit 1)
 				)
+			)
+		)
+	)
+	(symbol
+		(lib_id "Mechanical:Housing")
+		(at 130.81 184.15 0)
+		(unit 1)
+		(exclude_from_sim no)
+		(in_bom no)
+		(on_board yes)
+		(dnp yes)
+		(fields_autoplaced yes)
+		(property "Reference" "N2"
+			(at 134.62 183.1974 0)
+			(effects
+				(font
+					(size 1.27 1.27)
+				)
+				(justify left)
+			)
+		)
+		(property "Value" "Ranzbak"
+			(at 134.62 185.7374 0)
+			(effects
+				(font
+					(size 1.27 1.27)
+				)
+				(justify left)
+			)
+		)
+		(property "Footprint" "defeest:goatse_01"
+			(at 132.08 182.88 0)
+			(effects
+				(font
+					(size 1.27 1.27)
+				)
+				(hide yes)
+			)
+		)
+		(property "Datasheet" "~"
+			(at 132.08 182.88 0)
+			(effects
+				(font
+					(size 1.27 1.27)
+				)
+				(hide yes)
+			)
+		)
+		(property "Description" "Board edge + art"
+			(at 130.81 184.15 0)
+			(effects
+				(font
+					(size 1.27 1.27)
+				)
+				(hide yes)
+			)
+		)
+		(property "Resource" ""
+			(at 130.81 184.15 0)
+			(effects
+				(font
+					(size 1.27 1.27)
+				)
+				(hide yes)
+			)
+		)
+		(instances
+			(project "bornhack2026-hardware"
+				(path "/23bf5400-d19c-445b-8744-b63ebcca303d"
+					(reference "N2")
+					(unit 1)
+				)

Commit message: Moved LoRa radio closer to antenna
Parts:
- removed R31, R32: 0, Resistor_SMD:R_0402_1005Metric, symbol Device:R_Small
- removed RF1: A-IPEX1-1.25A, lcsc:IPEX-SMD_3P-L2.6-W2.6-LS3.0_RF1200001R, symbol lcsc:A-IPEX1-1.25A
Connections:
- net SX1262 LoRA/LORA_ANT: now also AE3.1 (A)
Other:
- moved on the sheet: AE3

Commit message: Added small Bornhack logo.
Parts:
- added N3: Bornhack, lcsc:bornhack-logo-10mm, symbol Mechanical:Housing
Other:
- moved on the sheet: N2
Changed lines of the file:
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@@
 		(at 132.08 171.45 0)
 		(unit 1)
-		(exclude_from_sim no)
+		(exclude_from_sim yes)
 		(in_bom no)
 		(on_board yes)
@@
 	(symbol
 		(lib_id "Mechanical:Housing")
-		(at 130.81 184.15 0)
-		(unit 1)
-		(exclude_from_sim no)
+		(at 162.56 171.45 0)
+		(unit 1)
+		(exclude_from_sim yes)
+		(in_bom no)
+		(on_board yes)
+		(dnp yes)
+		(fields_autoplaced yes)
+		(property "Reference" "N3"
+			(at 166.37 170.4974 0)
+			(effects
+				(font
+					(size 1.27 1.27)
+				)
+				(justify left)
+			)
+		)
+		(property "Value" "Bornhack"
+			(at 166.37 173.0374 0)
+			(effects
+				(font
+					(size 1.27 1.27)
+				)
+				(justify left)
+			)
+		)
+		(property "Footprint" "lcsc:bornhack-logo-10mm"
+			(at 163.83 170.18 0)
+			(effects
+				(font
+					(size 1.27 1.27)
+				)
+				(hide yes)
+			)
+		)
+		(property "Datasheet" "~"
+			(at 163.83 170.18 0)
+			(effects
+				(font
+					(size 1.27 1.27)
+				)
+				(hide yes)
+			)
+		)
+		(property "Description" "Board edge + art"
+			(at 162.56 171.45 0)
+			(effects
+				(font
+					(size 1.27 1.27)
+				)
+				(hide yes)
+			)
+		)
+		(property "Resource" ""
+			(at 162.56 171.45 0)
+			(effects
+				(font
+					(size 1.27 1.27)
+				)
+				(hide yes)
+			)
+		)
+		(instances
+			(project "bornhack2026-hardware"
+				(path "/23bf5400-d19c-445b-8744-b63ebcca303d"
+					(reference "N3")
+					(unit 1)
+				)
+			)
+		)
+	)
+	(symbol
+		(lib_id "Mechanical:Housing")
+		(at 132.08 184.15 0)
+		(unit 1)
+		(exclude_from_sim yes)
 		(in_bom no)
 		(on_board yes)
@@
 		(fields_autoplaced yes)
 		(property "Reference" "N2"
-			(at 134.62 183.1974 0)
+			(at 135.89 183.1974 0)
 			(effects
 				(font
@@
 		)
 		(property "Value" "Ranzbak"
-			(at 134.62 185.7374 0)
+			(at 135.89 185.7374 0)
 			(effects
 				(font
@@
 		)
 		(property "Footprint" "defeest:goatse_01"
-			(at 132.08 182.88 0)
+			(at 133.35 182.88 0)
 			(effects
 				(font
@@
 		)
 		(property "Datasheet" "~"
-			(at 132.08 182.88 0)
+			(at 133.35 182.88 0)
 			(effects
 				(font
@@
 		)
 		(property "Description" "Board edge + art"
-			(at 130.81 184.15 0)
+			(at 132.08 184.15 0)
 			(effects
 				(font
@@
 		)
 		(property "Resource" ""
-			(at 130.81 184.15 0)
-			(effects
-				(font
+			(at 132.08 184.15 0)
+			(effects
+				(font

Commit message: Badge.Team
Parts:
- N2: value Ranzbak -> Badge.Team; footprint defeest:goatse_01 -> symbols:stamp
Changed lines of the file:
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@@
 			)
 		)
-		(property "Value" "Ranzbak"
+		(property "Value" "Badge.Team"
 			(at 135.89 185.7374 0)
 			(effects
@@
 			)
 		)
-		(property "Footprint" "defeest:goatse_01"
+		(property "Footprint" "symbols:stamp"
 			(at 133.35 182.88 0)
 			(effects
@@
 			)
 		)
-		(property "Description" "Board edge + art"
+		(property "Description" ""
 			(at 132.08 184.15 0)
 			(effects

Commit message: Squashed in new battery connector, made NFC coil and Bluetooth fit as good and bad as possible.
Changed lines of the file:
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@@
 					(size 1.27 1.27)
 				)
-				(hide yes)
 			)
 		)

Commit message: Add QWIIC connector to design.
Connections:
- no-connect marks 10 -> 8
Other:
- added sheet QWIIC (qwiic.kicad_sch)
Changed lines of the file:
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@@
 	)
 	(no_connect
-		(at 180.34 80.01)
-	)
-	(no_connect
 		(at 271.78 27.94)
 	)
 	(no_connect
-		(at 180.34 77.47)
-	)
-	(no_connect
 		(at 180.34 72.39)
 	)
@@
 		)
 	)
+	(wire
+		(pts
+			(xy 180.34 77.47) (xy 200.66 77.47)
+		)
+		(stroke
+			(width 0)
+			(type default)
+		)
+	)
 	(bus
 		(pts
@@
 	(wire
 		(pts
+			(xy 251.46 57.15) (xy 231.14 57.15)
+		)
+		(stroke
+			(width 0)
+			(type default)
+		)
+	)
+	(wire
+		(pts
+			(xy 251.46 59.69) (xy 231.14 59.69)
+		)
+		(stroke
+			(width 0)
+			(type default)
+		)
+	)
+	(wire
+		(pts
 			(xy 200.66 62.23) (xy 180.34 62.23)
 		)
@@
 	(wire
 		(pts
+			(xy 180.34 80.01) (xy 200.66 80.01)
+		)
+		(stroke
+			(width 0)
+			(type default)
+		)
+	)
+	(wire
+		(pts
 			(xy 180.34 87.63) (xy 194.31 87.63)
 		)
@@
 		)
 	)
+	(label "P1.10_QWIIC_SDA"
+		(at 231.14 59.69 0)
+		(effects
+			(font
+				(size 1.27 1.27)
+			)
+			(justify left bottom)
+		)
+	)
 	(label "P1.14_MISO"
 		(at 194.31 87.63 180)
@@
 		)
 	)
+	(label "P1.11_QWIIC_SCL"
+		(at 231.14 57.15 0)
+		(effects
+			(font
+				(size 1.27 1.27)
+			)
+			(justify left bottom)
+		)
+	)
 	(label "P0.03_LORA_BUSY"
 		(at 116.84 53.34 0)
@@
 		)
 	)
+	(label "P1.10_QWIIC_SDA"
+		(at 200.66 77.47 180)
+		(effects
+			(font
+				(size 1.27 1.27)
+			)
+			(justify right bottom)
+		)
+	)
 	(label "BTN_JOY_LEFT"
 		(at 200.66 67.31 180)
@@
 		)
 	)
+	(label "P1.11_QWIIC_SCL"
+		(at 200.66 80.01 180)
+		(effects
+			(font
+				(size 1.27 1.27)
+			)
+			(justify right bottom)
+		)
+	)
 	(label "USB_D+"
 		(at 276.86 128.27 180)
@@
 				)
 			)
+		)
+	)
+	(sheet
+		(at 251.46 54.61)
+		(size 20.32 7.62)
+		(exclude_from_sim no)
+		(in_bom yes)
+		(on_board yes)
+		(dnp no)
+		(fields_autoplaced yes)
+		(stroke
+			(width 0.1524)
+			(type solid)
+		)
+		(fill
+			(color 0 0 0 0.0000)
+		)
+		(property "Sheetname" "QWIIC"
+			(at 251.46 53.8984 0)
+			(effects
+				(font
+					(size 1.27 1.27)
+				)
+				(justify left bottom)
+			)
+		)
+		(property "Sheetfile" "qwiic.kicad_sch"
+			(at 251.46 62.8146 0)
+			(effects
+				(font
+					(size 1.27 1.27)
+				)
+				(justify left top)
+			)
+		)
+		(pin "QWIIC_SCL" input
+			(at 251.46 57.15 180)
+			(effects
+				(font
+					(size 1.27 1.27)
+				)
+				(justify left)
+			)
+		)
+		(pin "QWIIC_SDA" input
+			(at 251.46 59.69 180)
+			(effects
+				(font
+					(size 1.27 1.27)
+				)
+				(justify left)
+			)
+		)
+		(instances
+			(project "bornhack2026-hardware"
+				(path "/23bf5400-d19c-445b-8744-b63ebcca303d"
+					(page "11")
+				)
+			)

Commit message: Replaced joystick with alternatie (cheaper) part.
Parts:
- J1: footprint Connector_USB:USB_C_Receptacle_HRO_TYPE-C-31-M-12 -> lcsc:USB_C_Receptacle_HRO_TYPE-C-31-M-12
Changed lines of the file:
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@@
+	)
+	(bus_entry
+		(at 200.66 80.01)
+		(size 2.54 -2.54)
+		(stroke
+			(width 0)
+			(type default)
+		)
+	)
+	(bus_entry
+		(at 231.14 57.15)
+		(size -2.54 -2.54)
+		(stroke
+			(width 0)
+			(type default)
+		)
 	)
 	(bus_entry
@@
 	)
 	(bus_entry
+		(at 231.14 59.69)
+		(size -2.54 -2.54)
+		(stroke
+			(width 0)
+			(type default)
+		)
+	)
+	(bus_entry
 		(at 201.93 95.25)
 		(size -2.54 2.54)
@@
 		)
 	)
+	(bus_entry
+		(at 200.66 77.47)
+		(size 2.54 -2.54)
+		(stroke
+			(width 0)
+			(type default)
+		)
+	)
 	(wire
 		(pts
@@
 	(bus
 		(pts
+			(xy 203.2 74.93) (xy 205.74 72.39)
+		)
+		(stroke
+			(width 0)
+			(type default)
+		)
+	)
+	(bus
+		(pts
 			(xy 201.93 92.71) (xy 204.47 90.17)
 		)
@@
 		)
 	)
+	(bus
+		(pts
+			(xy 226.06 72.39) (xy 228.6 69.85)
+		)
+		(stroke
+			(width 0)
+			(type default)
+		)
+	)
 	(wire
 		(pts
@@
 		)
 	)
+	(bus
+		(pts
+			(xy 228.6 54.61) (xy 228.6 57.15)
+		)
+		(stroke
+			(width 0)
+			(type default)
+		)
+	)
 	(wire
 		(pts
@@
 		)
 	)
+	(bus
+		(pts
+			(xy 205.74 72.39) (xy 226.06 72.39)
+		)
+		(stroke
+			(width 0)
+			(type default)
+		)
+	)
 	(wire
 		(pts
@@
 		)
 	)
+	(bus
+		(pts
+			(xy 203.2 74.93) (xy 203.2 77.47)
+		)
+		(stroke
+			(width 0)
+			(type default)
+		)
+	)
 	(wire
 		(pts
@@
 		(pts
 			(xy 180.34 87.63) (xy 194.31 87.63)
+		)
+		(stroke
+			(width 0)
+			(type default)
+		)
+	)
+	(bus
+		(pts
+			(xy 228.6 57.15) (xy 228.6 69.85)
 		)
 		(stroke
@@
 	)
 	(label "BTN_JOY_RIGHT"
-		(at 200.66 59.69 180)
+		(at 200.66 57.15 180)
 		(effects
 			(font
@@
 		)
 	)
+	(label "{P1.10_QWIIC_SDA P1.11_QWIIC_SCL }"
+		(at 205.74 72.39 0)
+		(effects
+			(font
+				(size 1.27 1.27)
+			)
+			(justify left bottom)
+		)
+	)
 	(label "MCU_RESET"
 		(at 31.75 147.32 0)
@@
 	)
 	(label "BTN_JOY_DOWN"
-		(at 200.66 57.15 180)
+		(at 200.66 62.23 180)
 		(effects
 			(font
@@
 	)
 	(label "BTN_JOY_UP"
-		(at 200.66 62.23 180)
+		(at 200.66 64.77 180)
 		(effects
 			(font
@@
 	)
 	(label "BTN_JOY_FIRE"
-		(at 200.66 64.77 180)
+		(at 200.66 59.69 180)
 		(effects
 			(font
@@
 			)
 		)
-		(property "Footprint" "Connector_USB:USB_C_Receptacle_HRO_TYPE-C-31-M-12"
+		(property "Footprint" "lcsc:USB_C_Receptacle_HRO_TYPE-C-31-M-12"
 			(at 252.73 124.46 0)
 			(effects

Commit message: Add batteryvoltage and charge indicator circuit.
Connections:
- no-connect marks 8 -> 16
Other:
- sheet INPUT ports: added none; removed BTN_CONFIRM
- sheet NRF52840_MCU ports: added P0.20_QSPI_SIO_0, P0.21_QSPI_SCK, P0.22_QSPI_SIO_2, P0.23_QSPI_SIO_3, P0.24_QSPI_SIO_1, P0.25_QSPI_CSN, P1.08; removed P0.20, P0.21, P0.22, P0.23, P0.24, P0.25, P1.08/6D_PWR
- sheet POWER ports: added VBAT_READ; removed VIN
