File: bornhack2026-hardware.kicad_sch (KiCad schematic)
At the start: 11 parts, among them J1 USB device, J2 Conn_01x06_Pin

Commit message: Fixed DRC errors, added the game.
Parts:
- added N4: Egg edge silk, lcsc:egg-edge-silk, symbol lcsc:Housing
- J2: value Conn_01x06_Pin -> Conn_01x07_Pin; footprint Connector_PinHeader_1.00mm:PinHeader_1x06_P1.00mm_Vertical_SMD_Pin1Left -> Connector_PinHeader_1.00mm:PinHeader_1x07_P1.00mm_Vertical_SMD_Pin1Left; symbol Connector:Conn_01x06_Pin -> Connector:Conn_01x07_Pin; now in the parts list
Connections:
- net +3V3: now also J2.6 (Pin_6); no longer J2.5 (Pin_5)
- net GND: now also J2.7 (Pin_7); no longer J2.6 (Pin_6)
- net P0.14_EXP1: now also J2.2 (Pin_2); no longer J2.1 (Pin_1)
- net P0.14_EXP2: now also J2.3 (Pin_3); no longer J2.2 (Pin_2)
- net P0.14_EXP3: now also J2.4 (Pin_4); no longer J2.3 (Pin_3)
- net P0.14_EXP4: now also J2.5 (Pin_5); no longer J2.4 (Pin_4)
- new net P0.14_EXP0: J2.1 (Pin_1)
- no-connect marks 11 -> 10
Changed lines of the file:
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@@
 	)
 	(no_connect
-		(at 137.16 91.44)
-	)
-	(no_connect
 		(at 137.16 96.52)
 	)
@@
 		)
 	)
+	(wire
+		(pts
+			(xy 137.16 91.44) (xy 116.84 91.44)
+		)
+		(stroke
+			(width 0)
+			(type default)
+		)
+	)
 	(bus
 		(pts
@@
 	(wire
 		(pts
+			(xy 120.65 139.7) (xy 140.97 139.7)
+		)
+		(stroke
+			(width 0)
+			(type default)
+		)
+	)
+	(wire
+		(pts
 			(xy 271.78 116.84) (xy 274.32 116.84)
 		)
@@
 	)
 	(label "P0.14_EXP3"
-		(at 116.84 86.36 0)
+		(at 116.84 91.44 0)
 		(effects
 			(font
@@
 		)
 	)
+	(label "P0.14_EXP0"
+		(at 140.97 139.7 180)
+		(effects
+			(font
+				(size 1.27 1.27)
+			)
+			(justify right bottom)
+		)
+	)
 	(label "P0.30_LORA_RST"
 		(at 96.52 93.98 180)
@@
 	)
 	(label "P0.14_EXP2"
-		(at 116.84 83.82 0)
+		(at 116.84 86.36 0)
 		(effects
 			(font
@@
 		)
 	)
+	(label "P0.14_EXP0"
+		(at 116.84 81.28 0)
+		(effects
+			(font
+				(size 1.27 1.27)
+			)
+			(justify left bottom)
+		)
+	)
 	(label "P0.27_DSP_MOSI"
 		(at 118.11 111.76 0)
@@
 	)
 	(label "P0.14_EXP1"
-		(at 116.84 81.28 0)
+		(at 116.84 83.82 0)
 		(effects
 			(font
@@
 	)
 	(symbol
-		(lib_id "Connector:Conn_01x06_Pin")
+		(lib_id "Connector:Conn_01x07_Pin")
 		(at 115.57 147.32 0)
 		(unit 1)
 		(exclude_from_sim no)
-		(in_bom no)
+		(in_bom yes)
 		(on_board yes)
 		(dnp yes)
 		(fields_autoplaced yes)
 		(property "Reference" "J2"
-			(at 116.205 137.16 0)
+			(at 116.205 134.62 0)
 			(effects
 				(font
@@
 			)
 		)
-		(property "Value" "Conn_01x06_Pin"
-			(at 116.205 139.7 0)
+		(property "Value" "Conn_01x07_Pin"
+			(at 116.205 137.16 0)
 			(effects
 				(font
@@
 			)
 		)
-		(property "Footprint" "Connector_PinHeader_1.00mm:PinHeader_1x06_P1.00mm_Vertical_SMD_Pin1Left"
+		(property "Footprint" "Connector_PinHeader_1.00mm:PinHeader_1x07_P1.00mm_Vertical_SMD_Pin1Left"
 			(at 115.57 147.32 0)
 			(effects
@@
 			)
 		)
-		(property "Description" "Generic connector, single row, 01x06, script generated"
+		(property "Description" "Generic connector, single row, 01x07, script generated"
 			(at 115.57 147.32 0)
 			(effects
@@
 		(pin "6"
 		)
+		(pin "7"
+		)
 		(instances
 			(project "bornhack2026-hardware"
@@
 					(unit 1)
 				)
+			)
+		)
+	)
+	(symbol
+		(lib_id "lcsc:Housing")
+		(at 162.56 182.88 0)
+		(unit 1)
+		(exclude_from_sim no)
+		(in_bom yes)
+		(on_board yes)
+		(dnp yes)
+		(fields_autoplaced yes)
+		(property "Reference" "N4"
+			(at 166.37 181.9274 0)
+			(effects
+				(font
+					(size 1.27 1.27)
+				)
+				(justify left)
+			)
+		)
+		(property "Value" "Egg edge silk"
+			(at 166.37 184.4674 0)
+			(effects
+				(font
+					(size 1.27 1.27)
+				)
+				(justify left)
+			)
+		)
+		(property "Footprint" "lcsc:egg-edge-silk"
+			(at 163.83 181.61 0)
+			(effects
+				(font
+					(size 1.27 1.27)
+				)
+				(hide yes)
+			)
+		)
+		(property "Datasheet" "~"
+			(at 163.83 181.61 0)
+			(effects
+				(font
+					(size 1.27 1.27)
+				)
+				(hide yes)
+			)
+		)
+		(property "Description" "Housing"
+			(at 162.56 182.88 0)
+			(effects
+				(font
+					(size 1.27 1.27)
+				)
+				(hide yes)
+			)
+		)
+		(property "Resource" ""
+			(at 162.56 182.88 0)
+			(effects
+				(font
+					(size 1.27 1.27)
+				)
+				(hide yes)
+			)
+		)
+		(instances
+			(project "bornhack2026-hardware"
+				(path "/23bf5400-d19c-445b-8744-b63ebcca303d"
+					(reference "N4")
+					(unit 1)
+				)
