File: power.kicad_sch (KiCad schematic)
At the start: 6 parts, among them Q1 JSM2301S, U2 SGM2040-3.3YUDH4G/TR_C5152920

Commit message: Fixed mistake in NRF52 footprint, add NAND FLASH, add NFC antenna schematic.
Parts:
- renumbered R8 to R5
Other:
- company: (none) -> Badge.Team
- title: (none) -> Bornhack 2026
Changed lines of the file:
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@@
 	(generator_version "9.0")
 	(paper "A4")
+	(title_block
+		(title "Bornhack 2026")
+		(rev "0.1")
+		(company "Badge.Team")
+	)
 	(junction
 		(at 87.63 58.42)
@@
 		(dnp no)
 		(fields_autoplaced yes)
-		(property "Reference" "#PWR07"
+		(property "Reference" "#PWR033"
 			(at 58.42 81.28 0)
 			(effects
@@
 			(project ""
 				(path "/23bf5400-d19c-445b-8744-b63ebcca303d/333d98a8-e6a2-433c-bb9c-6f407290c160"
-					(reference "#PWR07")
+					(reference "#PWR033")
 					(unit 1)
 				)
@@
 		(dnp no)
 		(fields_autoplaced yes)
-		(property "Reference" "#PWR026"
+		(property "Reference" "#PWR034"
 			(at 76.2 81.28 0)
 			(effects
@@
 			(project "bornhack2026-hardware"
 				(path "/23bf5400-d19c-445b-8744-b63ebcca303d/333d98a8-e6a2-433c-bb9c-6f407290c160"
-					(reference "#PWR026")
+					(reference "#PWR034")
 					(unit 1)
 				)
@@
 		(dnp no)
 		(fields_autoplaced yes)
-		(property "Reference" "R8"
+		(property "Reference" "R5"
 			(at 60.96 71.1199 0)
 			(effects
@@
 			(project ""
 				(path "/23bf5400-d19c-445b-8744-b63ebcca303d/333d98a8-e6a2-433c-bb9c-6f407290c160"
-					(reference "R8")
+					(reference "R5")
 					(unit 1)
 				)
@@
 		(dnp no)
 		(fields_autoplaced yes)
-		(property "Reference" "#PWR034"
+		(property "Reference" "#PWR036"
 			(at 114.3 81.28 0)
 			(effects
@@
 			(project "bornhack2026-hardware"
 				(path "/23bf5400-d19c-445b-8744-b63ebcca303d/333d98a8-e6a2-433c-bb9c-6f407290c160"
-					(reference "#PWR034")
+					(reference "#PWR036")
 					(unit 1)
 				)
@@
 		(dnp no)
 		(fields_autoplaced yes)
-		(property "Reference" "#PWR033"
+		(property "Reference" "#PWR035"
 			(at 107.95 81.28 0)
 			(effects
@@
 			(project "bornhack2026-hardware"
 				(path "/23bf5400-d19c-445b-8744-b63ebcca303d/333d98a8-e6a2-433c-bb9c-6f407290c160"
-					(reference "#PWR033")
+					(reference "#PWR035")
 					(unit 1)
 				)

Commit message: PCB layout egg shape, for reference.
Parts:
- added J11: Battery, library:CONN-SMD_PH-2AWB, symbol symbols:Conn_01x02_MountingPin
- added TP7: VBAT+, TestPoint:TestPoint_Pad_D1.0mm, symbol Connector:TestPoint
Connections:
- net GND: now also J11.2 (Pin_2), J11.MP (MountPin)
- net VBAT: now also J11.1 (Pin_1), TP7.1
Other:
- moved on the sheet: C19, C20, D2, Q1, R5, U2

Commit message: Switched the LC filters from ceramic LoRa filter.
Parts:
- removed U2: SGM2040-3.3YUDH4G/TR_C5152920, lcsc:UTDFN-4AL_L1.0-W1.0-P0.65-BL, symbol lcsc:SGM2040-3.3YUDH4G_TR_C5152920
- added U6: SGM2040-3.3YN5G/TR, lcsc:SOT-23-5_L2.9-W1.6-P0.95-LS2.8-BL, symbol lcsc:SGM2040-3.3YN5G_TR
- Q1: LCSC (none) -> C916399
Connections:
- net +3V3_OUT: now also U6.5 (OUT)
- net GND: now also U6.2 (GND)
- net VIN: now also U6.1 (IN), U6.3 (EN)
- no-connect marks 0 -> 1
Changed lines of the file:
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@@
-	)
-	(junction
-		(at 209.55 111.76)
-		(diameter 0)
-		(color 0 0 0 0)
 	)
 	(junction
@@
 	)
 	(junction
-		(at 236.22 114.3)
+		(at 208.28 111.76)
+		(diameter 0)
+		(color 0 0 0 0)
+	)
+	(junction
+		(at 236.22 111.76)
 		(diameter 0)
 		(color 0 0 0 0)
@@
 		(color 0 0 0 0)
 	)
-	(wire
-		(pts
-			(xy 229.87 111.76) (xy 229.87 128.27)
+	(no_connect
+		(at 227.33 116.84)
+	)
+	(wire
+		(pts
+			(xy 207.01 114.3) (xy 207.01 130.81)
 		)
 		(stroke
@@
 	(wire
 		(pts
-			(xy 227.33 111.76) (xy 229.87 111.76)
-		)
-		(stroke
-			(width 0)
-			(type default)
-		)
-	)
-	(wire
-		(pts
-			(xy 236.22 114.3) (xy 242.57 114.3)
+			(xy 236.22 111.76) (xy 242.57 111.76)
 		)
 		(stroke
@@
 	(wire
 		(pts
+			(xy 208.28 116.84) (xy 209.55 116.84)
+		)
+		(stroke
+			(width 0)
+			(type default)
+		)
+	)
+	(wire
+		(pts
+			(xy 208.28 111.76) (xy 208.28 116.84)
+		)
+		(stroke
+			(width 0)
+			(type default)
+		)
+	)
+	(wire
+		(pts
 			(xy 176.53 85.09) (xy 177.8 85.09)
 		)
@@
 	(wire
 		(pts
+			(xy 208.28 111.76) (xy 209.55 111.76)
+		)
+		(stroke
+			(width 0)
+			(type default)
+		)
+	)
+	(wire
+		(pts
 			(xy 198.12 111.76) (xy 198.12 114.3)
 		)
@@
 	(wire
 		(pts
-			(xy 209.55 111.76) (xy 209.55 114.3)
+			(xy 207.01 114.3) (xy 209.55 114.3)
+		)
+		(stroke
+			(width 0)
+			(type default)
+		)
+	)
+	(wire
+		(pts
+			(xy 236.22 111.76) (xy 236.22 114.3)
 		)
 		(stroke
@@
 	(wire
 		(pts
-			(xy 227.33 114.3) (xy 236.22 114.3)
+			(xy 227.33 111.76) (xy 236.22 111.76)
 		)
 		(stroke
@@
 	(wire
 		(pts
-			(xy 198.12 111.76) (xy 209.55 111.76)
+			(xy 198.12 111.76) (xy 208.28 111.76)
 		)
 		(stroke
@@
 	(hierarchical_label "+3V3_OUT"
 		(shape input)
-		(at 242.57 114.3 0)
+		(at 242.57 111.76 0)
 		(effects
 			(font
@@
 			)
 		)
-		(property "Datasheet" "https://lcsc.com/product-detail/MOSFET_JSMSEMI-JSM2301S_C916399.html"
+		(property "Datasheet" "https://jlcpcb.com/partdetail/JSMSEMI-JSM2301S/C916399"
 			(at 195.58 111.76 0)
 			(effects
@@
 		(property "LCSC Part" "C916399"
 			(at 198.12 111.76 0)
+			(effects
+				(font
+					(size 1.27 1.27)
+				)
+				(hide yes)
+			)
+		)
+		(property "LCSC" "C916399"
+			(at 180.34 111.76 90)
 			(effects
 				(font
@@
 	)
 	(symbol
+		(lib_id "lcsc:SGM2040-3.3YN5G_TR")
+		(at 218.44 114.3 0)
+		(unit 1)
+		(exclude_from_sim no)
+		(in_bom yes)
+		(on_board yes)
+		(dnp no)
+		(fields_autoplaced yes)
+		(property "Reference" "U6"
+			(at 218.44 104.14 0)
+			(effects
+				(font
+					(size 1.27 1.27)
+				)
+			)
+		)
+		(property "Value" "SGM2040-3.3YN5G/TR"
+			(at 218.44 106.68 0)
+			(effects
+				(font
+					(size 1.27 1.27)
+				)
+			)
+		)
+		(property "Footprint" "lcsc:SOT-23-5_L2.9-W1.6-P0.95-LS2.8-BL"
+			(at 218.44 124.46 0)
+			(effects
+				(font
+					(size 1.27 1.27)
+				)
+				(hide yes)
+			)
+		)
+		(property "Datasheet" "https://jlcpcb.com/partdetail/SGMICRO-SGM2040_3_3YN5GTR/C2890487"
+			(at 218.44 114.3 0)
+			(effects
+				(font
+					(size 1.27 1.27)
+				)
+				(hide yes)
+			)
+		)
+		(property "Description" "-40℃~+85℃@(Ta) 1 1.5uA 110mV@(100mA) 250mA 27dB@(1kHz) 3.3V 7.5V Fixed Over Current Protection Positive SOT-23-5 Voltage Regulators - Linear, Low Drop Out (LDO) Regulators ROHS"
+			(at 218.44 114.3 0)
+			(effects
+				(font
+					(size 1.27 1.27)
+				)
+				(hide yes)
+			)
+		)
+		(property "LCSC Part" "C2890487"
+			(at 218.44 127 0)
+			(effects
+				(font
+					(size 1.27 1.27)
+				)
+				(hide yes)
+			)
+		)
+		(property "LCSC" "C2890487"
+			(at 218.44 114.3 0)
+			(effects
+				(font
+					(size 1.27 1.27)
+				)
+				(hide yes)
+			)
+		)
+		(pin "5"
+		)
+		(pin "3"
+		)
+		(pin "2"
+		)
+		(pin "1"
+		)
+		(pin "4"
+		)
+		(instances
+			(project ""
+				(path "/23bf5400-d19c-445b-8744-b63ebcca303d/333d98a8-e6a2-433c-bb9c-6f407290c160"
+					(reference "U6")
+					(unit 1)
+				)
+			)
+		)
+	)
+	(symbol
 		(lib_id "symbols:Conn_01x02_MountingPin")
 		(at 182.88 85.09 0)
@@
 				(path "/23bf5400-d19c-445b-8744-b63ebcca303d/333d98a8-e6a2-433c-bb9c-6f407290c160"
 					(reference "J11")
-					(unit 1)
-				)
-			)
-		)
-	)
-	(symbol
-		(lib_id "lcsc:SGM2040-3.3YUDH4G_TR_C5152920")
-		(at 217.17 111.76 180)
-		(unit 1)
-		(exclude_from_sim no)
-		(in_bom yes)
-		(on_board yes)
-		(dnp no)
-		(fields_autoplaced yes)
-		(property "Reference" "U2"
-			(at 218.44 104.14 0)
-			(effects
-				(font
-					(size 1.27 1.27)
-				)
-			)
-		)
-		(property "Value" "SGM2040-3.3YUDH4G/TR_C5152920"
-			(at 218.44 106.68 0)
-			(effects
-				(font
-					(size 1.27 1.27)
-				)
-			)
-		)
-		(property "Footprint" "lcsc:UTDFN-4AL_L1.0-W1.0-P0.65-BL"
-			(at 217.17 104.14 0)
-			(effects
-				(font
-					(size 1.27 1.27)
-				)
-				(hide yes)
-			)
-		)
-		(property "Datasheet" ""
-			(at 217.17 111.76 0)
-			(effects
-				(font
-					(size 1.27 1.27)
-				)
-				(hide yes)
-			)
-		)
-		(property "Description" ""
-			(at 217.17 111.76 0)
-			(effects
-				(font
-					(size 1.27 1.27)
-				)
-				(hide yes)
-			)
-		)
-		(property "LCSC Part" "C5152920"
-			(at 217.17 101.6 0)
-			(effects
-				(font
-					(size 1.27 1.27)
-				)
-				(hide yes)
-			)
-		)
-		(pin "1"
-		)
-		(pin "4"
-		)
-		(pin "3"
-		)
-		(pin "2"
-		)
-		(instances
-			(project ""
-				(path "/23bf5400-d19c-445b-8744-b63ebcca303d/333d98a8-e6a2-433c-bb9c-6f407290c160"
-					(reference "U2")
 					(unit 1)
 				)
@@
 	(symbol
 		(lib_id "power:GND")
-		(at 229.87 128.27 0)
+		(at 207.01 130.81 0)
 		(unit 1)
 		(exclude_from_sim no)
@@
 		(fields_autoplaced yes)
 		(property "Reference" "#PWR035"
-			(at 229.87 134.62 0)
+			(at 207.01 137.16 0)
 			(effects
 				(font
@@
 		)
 		(property "Value" "GND"
-			(at 229.87 133.35 0)
+			(at 207.01 135.89 0)
 			(effects
 				(font
@@
 		)
 		(property "Footprint" ""
-			(at 229.87 128.27 0)
+			(at 207.01 130.81 0)
 			(effects
 				(font
@@
 		)
 		(property "Datasheet" ""
-			(at 229.87 128.27 0)
+			(at 207.01 130.81 0)
 			(effects
 				(font
@@
 		)
 		(property "Description" "Power symbol creates a global label with name \"GND\" , ground"
-			(at 229.87 128.27 0)
-			(effects
-				(font
+			(at 207.01 130.81 0)
+			(effects
+				(font

Commit message: Progress, routed more stuff.
Parts:
- removed C20: 2.2uF, Capacitor_SMD:C_0402_1005Metric, symbol Device:C_Small
- removed J11: Battery, library:CONN-SMD_PH-2AWB, symbol symbols:Conn_01x02_MountingPin
- removed TP7: VBAT+, TestPoint:TestPoint_Pad_D1.0mm, symbol Connector:TestPoint
- removed U6: SGM2040-3.3YN5G/TR, lcsc:SOT-23-5_L2.9-W1.6-P0.95-LS2.8-BL, symbol lcsc:SGM2040-3.3YN5G_TR
- added C54, C56: 10uF, Capacitor_SMD:C_0603_1608Metric, symbol symbols:C
- added C55, C57, C64: 100nF, Capacitor_SMD:C_0402_1005Metric, symbol symbols:C
- added C58, C62, C63: 22uF, Capacitor_SMD:C_0805_2012Metric, symbol Device:C
- added C60, C61: 10uF, Capacitor_SMD:C_0603_1608Metric, symbol Device:C
- added D1: ESD prot., Diode_SMD:D_SOD-323, symbol Device:D_TVS
- added D23: NSR0320MW2T1G, Diode_SMD:D_SOD-323, symbol symbols:D_Schottky
- added J9: Battery, lcsc:CONN-SMD_S2B-ZR-SM4A, symbol symbols:Conn_01x02_MountingPin
- added L4: CMLW6028S1R5MST, lcsc:IND-SMD_L6.0-W6.0, symbol lcsc:CMLW6028S1R5MST
- added R14, R16: 1k, Resistor_SMD:R_0402_1005Metric, symbol Device:R_Small
- added R17: 1M, Resistor_SMD:R_0402_1005Metric_Pad0.72x0.64mm_HandSolder, symbol Device:R
- added R24: 180k, Resistor_SMD:R_0402_1005Metric_Pad0.72x0.64mm_HandSolder, symbol Device:R
- added R25: 2k, Resistor_SMD:R_0402_1005Metric, symbol symbols:R
- added R26: 10k, Resistor_SMD:R_0402_1005Metric, symbol symbols:R
- added SW2: SK-3296S-01-L1, lcsc:SW-SMD_3P-P1.50_L2.7-W6.6, symbol lcsc:SK-3296S-01-L1
- added U4: XT4054K421MR-G, lcsc:SOT-23-5_L2.9-W1.6-P0.95-LS2.8-BL, symbol symbols:MCP73831-2-OT-Battery_Management
- added U7: TPS63020DSJR, lcsc:VSON-14_L4.0-W3.0-P0.50-BL-EP_TI_DSJ, symbol lcsc:TPS63020DSJR
- D2: value D -> B160_13F
Connections:
- net +3V3_OUT: now also R17.1, R26.2, U7.4 (VOUT), U7.5 (VOUT)
- net GND: now also C54.1, C55.1, C56.2, C57.2, C58.2, C60.2, C61.2, C62.2, C63.2, C64.2, D1.2 (A2), J9.1 (Pin_1), J9.MP (MountPin), R16.1, R24.2, R25.1, SW2.0, U4.2 (VSS), U7.15 (PGND), U7.2 (GND)
- net VBAT: now also C56.1, J9.2 (Pin_2), U4.3 (VBAT)
- net VBUS: now also D1.1 (A1), D23.2 (A)
- net VIN: now also C60.1, C61.1, U7.10 (VIN), U7.11 (VIN)
- new net: C57.1, R14.1, U7.1 (VINA), U7.13 (PS/SYNC)
- new net: SW2.2, U7.12 (EN)
- new net: R17.2, R24.1, U7.3 (FB)
- new net: L4.1, U7.6 (L2), U7.7 (L2)
- new net: L4.2, U7.8 (L1), U7.9 (L1)
- new net: C54.2, C55.2, D23.1 (K), U4.4 (VDD)
- new net: R25.2, U4.5 (PROG)
- new net: R14.2, SW2.1
- new net: R16.2, SW2.3
- new net +3V3: C58.1, C62.1, C63.1, C64.1
- new net CHRG: R26.1, U4.1 (STAT)
Other:
- note added: "3.3v DC/DC"
- note added: "Battery & battery charger"
- note added: "CHARGING is an open-drain output that gets pulled low when the charger is active (charging the battery)"
- note added: "IBAT = (1 / 2000) * 1000 = 500mA"
- note added: "place close to TPS63020DSJR"
- moved on the sheet: C19, D2, Q1, R5

Commit message: Fix tiny issues, add more vias.
Parts:
- added C66, C67: 2.2uF, Capacitor_SMD:C_0402_1005Metric, symbol Device:C_Small
- added R33: 1M, Resistor_SMD:R_0402_1005Metric_Pad0.72x0.64mm_HandSolder, symbol Device:R
Connections:
- net at C57.1, R14.1, U7.1 (VINA): now also C66.1, R33.1; no longer U7.13 (PS/SYNC)
- net at SW2.2, U7.12 (EN): now also C66.2, C67.1
- net at R16.2, SW2.3: now also C67.2
- new net PS_SYNC: R33.2, U7.13 (PS/SYNC)
Other:
- moved on the sheet: R16

Commit message: Checked PCBA for JLCPCB.
Parts:
- C58, C62, C63: LCSC C59461 -> C45783
- SW2: LCSC (none) -> C319020
Changed lines of the file:
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@@
 			)
 		)
-		(property "Datasheet" "https://jlcpcb.com/partdetail/60514-CL10A226MQ8NRNC/C59461"
+		(property "Datasheet" "https://jlcpcb.com/partdetail/46786-CL21A226MAQNNNE/C45783"
 			(at 226.06 35.56 0)
 			(effects
@@
 			)
 		)
-		(property "LCSC" "C59461"
+		(property "LCSC" "C45783 "
 			(at 226.06 35.56 0)
 			(effects
@@
 			)
 		)
-		(property "Datasheet" "https://jlcpcb.com/partdetail/60514-CL10A226MQ8NRNC/C59461"
+		(property "Datasheet" "https://jlcpcb.com/partdetail/46786-CL21A226MAQNNNE/C45783"
 			(at 213.36 35.56 0)
 			(effects
@@
 			)
 		)
-		(property "LCSC" "C59461"
+		(property "LCSC" "C45783 "
 			(at 213.36 35.56 0)
 			(effects
@@
 			)
 		)
+		(property "LCSC" "C319020"
+			(at 270.51 72.39 0)
+			(effects
+				(font
+					(size 1.27 1.27)
+				)
+				(hide yes)
+			)
+		)
 		(pin "0"
 		)
@@
 			)
 		)
-		(property "Datasheet" "https://jlcpcb.com/partdetail/60514-CL10A226MQ8NRNC/C59461"
+		(property "Datasheet" "https://jlcpcb.com/partdetail/46786-CL21A226MAQNNNE/C45783"
 			(at 201.93 35.56 0)
 			(effects
@@
 			)
 		)
-		(property "LCSC" "C59461"
+		(property "LCSC" "C45783 "
 			(at 201.93 35.56 0)
 			(effects
@@
 			)
 		)
-		(property "Datasheet" "https://www.lcsc.com/product-detail/Chip-Resistor-Surface-Mount_UNI-ROYAL-Uniroyal-Elec-0402WGF1002TCE_C25744.html"
+		(property "Datasheet" "https://jlcpcb.com/partdetail/26487-0402WGF1002TCE/C25744"
 			(at 90.17 153.67 0)
 			(effects
