File: power.kicad_sch (KiCad schematic)
At the start: 30 parts, among them J9 Battery, Q1 JSM2301S, SW2 SK-3296S-01-L1, U4 XT4054K421MR-G, U7 TPS63020DSJR

Commit message: Squashed in new battery connector, made NFC coil and Bluetooth fit as good and bad as possible.
Parts:
- removed J9: Battery, lcsc:CONN-SMD_S2B-ZR-SM4A, symbol symbols:Conn_01x02_MountingPin
- added U1: PH-2AWB, lcsc:CONN-SMD_PH-2AWB, symbol lcsc:PH-2AWB
Connections:
- net GND: now also U1.2, U1.3, U1.4
- net VBAT: now also U1.1

Commit message: Add batteryvoltage and charge indicator circuit.
Parts:
- removed C19: 2.2uF, Capacitor_SMD:C_0402_1005Metric, symbol Device:C_Small
- added R34: 1M, Resistor_SMD:R_0402_1005Metric, symbol Device:R_Small
- added R35: 510k, Resistor_SMD:R_0402_1005Metric, symbol Device:R_Small
Connections:
- net VBAT: now also R34.1, R35.2; no longer C56.1, Q1.3 (D), U1.1, U4.3 (VBAT)
- new net: C56.1, Q1.3 (D), R34.2, U1.1, U4.3 (VBAT)
- new net VBAT_READ: R35.1

Commit message: Fixed schematic enspect errors. Fixed jhaand name in silk screen.
Parts:
- U7: LCSC Part (none) -> C15483
Changed lines of the file:
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@@
-	)
-	(junction
-		(at 127 140.97)
-		(diameter 0)
-		(color 0 0 0 0)
 	)
 	(junction
@@
 	(wire
 		(pts
-			(xy 127 140.97) (xy 127 160.02)
-		)
-		(stroke
-			(width 0)
-			(type default)
-		)
-	)
-	(wire
-		(pts
 			(xy 232.41 88.9) (xy 241.3 88.9)
 		)
@@
 	(wire
 		(pts
-			(xy 127 135.89) (xy 127 140.97)
+			(xy 127 135.89) (xy 127 160.02)
 		)
 		(stroke
@@
 	)
 	(hierarchical_label "+3V3_OUT"
-		(shape input)
+		(shape output)
 		(at 163.83 62.23 180)
 		(effects
@@
 		(property "Component Class" ""
 			(at -181.61 140.97 0)
+			(effects
+				(font
+					(size 1.27 1.27)
+					(italic yes)
+				)
+			)
+		)
+	)
+	(netclass_flag ""
+		(length 2.54)
+		(shape round)
+		(at 149.86 160.02 0)
+		(fields_autoplaced yes)
+		(effects
+			(font
+				(size 1.27 1.27)
+			)
+			(justify left bottom)
+		)
+		(property "Netclass" "Power"
+			(at 150.5585 157.48 0)
+			(effects
+				(font
+					(size 1.27 1.27)
+				)
+				(justify left)
+			)
+		)
+		(property "Component Class" ""
+			(at -24.13 -1.27 0)
+			(effects
+				(font
+					(size 1.27 1.27)
+					(italic yes)
+				)
+			)
+		)
+	)
+	(netclass_flag ""
+		(length 2.54)
+		(shape round)
+		(at 172.72 62.23 0)
+		(fields_autoplaced yes)
+		(effects
+			(font
+				(size 1.27 1.27)
+			)
+			(justify left bottom)
+		)
+		(property "Netclass" "Power"
+			(at 173.4185 59.69 0)
+			(effects
+				(font
+					(size 1.27 1.27)
+				)
+				(justify left)
+			)
+		)
+		(property "Component Class" ""
+			(at -111.76 0 0)
+			(effects
+				(font
+					(size 1.27 1.27)
+					(italic yes)
+				)
+			)
+		)
+	)
+	(netclass_flag ""
+		(length 2.54)
+		(shape round)
+		(at 36.83 154.94 0)
+		(fields_autoplaced yes)
+		(effects
+			(font
+				(size 1.27 1.27)
+			)
+			(justify left bottom)
+		)
+		(property "Netclass" "Power"
+			(at 37.5285 152.4 0)
+			(effects
+				(font
+					(size 1.27 1.27)
+				)
+				(justify left)
+			)
+		)
+		(property "Component Class" ""
+			(at -66.04 8.89 0)
 			(effects
 				(font
@@
 			)
 		)
+		(property "LCSC Part" "C15483"
+			(at 201.93 102.87 0)
+			(effects
+				(font
+					(size 1.27 1.27)
+				)
+				(hide yes)
+			)
+		)
 		(pin "6"
 		)
@@
 			)
 		)
-		(property "Datasheet" "https://jlcpcb.com/partdetail/JSMSEMI-JSM2301S/C916399"
+		(property "Datasheet" "https://lcsc.com/product-detail/MOSFET_JSMSEMI-JSM2301S_C916399.html"
 			(at 152.4 160.02 0)
 			(effects
@@
 					(unit 1)
 				)
-			)
-		)
-	)
-	(symbol
-		(lib_id "symbols2:PWR_FLAG")
-		(at 127 140.97 90)
-		(unit 1)
-		(exclude_from_sim no)
-		(in_bom yes)
-		(on_board yes)
-		(dnp no)
-		(fields_autoplaced yes)
-		(property "Reference" "#FLG02"
-			(at 125.095 140.97 0)
-			(effects
-				(font
-					(size 1.27 1.27)
-				)
-				(hide yes)
-			)
-		)
-		(property "Value" "PWR_FLAG"
-			(at 123.19 140.9699 90)
-			(effects
-				(font
-					(size 1.27 1.27)
-				)
-				(justify left)
-			)
-		)
-		(property "Footprint" ""
-			(at 127 140.97 0)
-			(effects
-				(font
-					(size 1.27 1.27)
-				)
-				(hide yes)
-			)
-		)
-		(property "Datasheet" "~"
-			(at 127 140.97 0)
-			(effects
-				(font
-					(size 1.27 1.27)
-				)
-				(hide yes)
-			)
-		)
-		(property "Description" ""
-			(at 127 140.97 0)
-			(effects
-				(font
-					(size 1.27 1.27)
-				)
-				(hide yes)
-			)
-		)
-		(pin "1"
-		)
-		(instances
-			(project "bornhack2026-hardware"
-				(path "/23bf5400-d19c-445b-8744-b63ebcca303d/333d98a8-e6a2-433c-bb9c-6f407290c160"
-					(reference "#FLG02")
-					(unit 1)
-				)

Commit message: Add Readme, fix labels in schematic.
Connections:
- net CHRG renamed P1.08_CHRG
Changed lines of the file:
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@@
 		)
 	)
-	(hierarchical_label "CHRG"
+	(hierarchical_label "P1.08_CHRG"
 		(shape output)
 		(at 91.44 165.1 0)

Commit message: Moved SWR connector to other side of board, reversed on/off switch UP -> ON.
Connections:
- net at R14.2: now also SW2.3; no longer SW2.1
- net at C67.2, R16.2: now also SW2.1; no longer SW2.3
Other:
- moved on the sheet: SW2
Changed lines of the file:
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@@
 	(wire
 		(pts
-			(xy 259.08 69.85) (xy 262.89 69.85)
+			(xy 261.62 72.39) (xy 262.89 72.39)
 		)
 		(stroke
@@
 	(wire
 		(pts
+			(xy 261.62 72.39) (xy 261.62 69.85)
+		)
+		(stroke
+			(width 0)
+			(type default)
+		)
+	)
+	(wire
+		(pts
 			(xy 241.3 74.93) (xy 241.3 77.47)
 		)
@@
 	(wire
 		(pts
-			(xy 259.08 77.47) (xy 262.89 77.47)
+			(xy 261.62 80.01) (xy 262.89 80.01)
 		)
 		(stroke
@@
 	(wire
 		(pts
+			(xy 261.62 69.85) (xy 259.08 69.85)
+		)
+		(stroke
+			(width 0)
+			(type default)
+		)
+	)
+	(wire
+		(pts
 			(xy 186.69 80.01) (xy 186.69 82.55)
 		)
@@
 	(wire
 		(pts
-			(xy 280.67 69.85) (xy 280.67 91.44)
+			(xy 280.67 80.01) (xy 280.67 91.44)
 		)
 		(stroke
@@
 	(wire
 		(pts
-			(xy 278.13 69.85) (xy 280.67 69.85)
+			(xy 278.13 80.01) (xy 280.67 80.01)
 		)
 		(stroke
@@
 	(wire
 		(pts
-			(xy 259.08 77.47) (xy 259.08 81.28)
+			(xy 261.62 80.01) (xy 261.62 81.28)
 		)
 		(stroke
@@
 	(wire
 		(pts
-			(xy 248.92 81.28) (xy 259.08 81.28)
+			(xy 248.92 81.28) (xy 261.62 81.28)
 		)
 		(stroke
@@
 	(symbol
 		(lib_id "lcsc:SK-3296S-01-L1")
-		(at 270.51 72.39 0)
+		(at 270.51 77.47 0)
+		(mirror x)
 		(unit 1)
 		(exclude_from_sim no)
@@
 		(on_board yes)
 		(dnp no)
-		(fields_autoplaced yes)
 		(property "Reference" "SW2"
-			(at 270.51 62.23 0)
+			(at 270.51 87.63 0)
 			(effects
 				(font
@@
 		)
 		(property "Value" "SK-3296S-01-L1"
-			(at 270.51 64.77 0)
+			(at 270.51 85.09 0)
 			(effects
 				(font
@@
 		)
 		(property "Footprint" "lcsc:SW-SMD_3P-P1.50_L2.7-W6.6"
-			(at 270.51 85.09 0)
+			(at 270.51 64.77 0)
 			(effects
 				(font
@@
 		)
 		(property "Datasheet" "https://lcsc.com/product-detail/Toggle-Switches_XKB-Enterprise-SK-3296S-01-L1_C319020.html"
-			(at 270.51 87.63 0)
+			(at 270.51 62.23 0)
 			(effects
 				(font
@@
 		)
 		(property "Description" ""
-			(at 270.51 72.39 0)
+			(at 270.51 77.47 0)
 			(effects
 				(font
@@
 		)
 		(property "LCSC Part" "C319020"
-			(at 270.51 90.17 0)
+			(at 270.51 59.69 0)
 			(effects
 				(font
@@
 		)
 		(property "LCSC" "C319020"
-			(at 270.51 72.39 0)
+			(at 270.51 77.47 0)
 			(effects
 				(font
@@
 		)
 		(property "Resource" ""
-			(at 270.51 72.39 0)
+			(at 270.51 77.47 0)
 			(effects
 				(font

Commit message: Fixed PCBA rotations in using component property.
Parts:
- Q1, U4: FT Rotation Offset (none) -> 180
Changed lines of the file:
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@@
+			)
+		)
+		(property "FT Rotation Offset" "180"
+			(at 137.16 160.02 0)
+			(effects
+				(font
+					(size 1.27 1.27)
+				)
+				(hide yes)
 			)
 		)
@@
 			(at 77.47 162.56 0)
 			(effects
+				(font
+					(size 1.27 1.27)
+				)
+				(hide yes)
+			)
+		)
+		(property "FT Rotation Offset" "180"
+			(at 77.47 162.56 0)
+			(effects

Commit message: Optimized design to use more basic components.
Parts:
- R17, R24, R33: footprint Resistor_SMD:R_0402_1005Metric_Pad0.72x0.64mm_HandSolder -> Resistor_SMD:R_0402_1005Metric
- R5: LCSC C25530 -> C25741
- U1: LCSC (none) -> C20598817

Commit message: Replaced schottky diode with 1A version, fixed joystick footprint.
Parts:
- removed C57, C64: 100nF, Capacitor_SMD:C_0402_1005Metric, symbol symbols:C
- removed C58, C62, C63: 22uF, Capacitor_SMD:C_0805_2012Metric, symbol Device:C
- removed C60, C61: 10uF, Capacitor_SMD:C_0603_1608Metric, symbol Device:C
- removed D23: NSR0320MW2T1G, Diode_SMD:D_SOD-323, symbol symbols:D_Schottky
- removed L4: CMLW6028S1R5MST, lcsc:IND-SMD_L6.0-W6.0, symbol lcsc:CMLW6028S1R5MST
- removed R17, R33: 1M, Resistor_SMD:R_0402_1005Metric, symbol Device:R
- removed R24: 180k, Resistor_SMD:R_0402_1005Metric, symbol Device:R
- removed U7: TPS63020DSJR, lcsc:VSON-14_L4.0-W3.0-P0.50-BL-EP_TI_DSJ, symbol lcsc:TPS63020DSJR
- added C19, C57: 22uF, Capacitor_SMD:C_0603_1608Metric, symbol Device:C
- added C9: 10uF, Capacitor_SMD:C_0603_1608Metric, symbol Device:C
- added D7: 1N5819WS, Diode_SMD:D_SOD-323, symbol Diode:1N5819WS
- added L1: 0.47uH A-sat 5.4 DCR 7.6 mOhm, Inductor_SMD:L_Vishay_IFSC-1515AH_4x4x1.8mm, symbol Device:L_Small
- added R44: 1M, Resistor_SMD:R_0402_1005Metric, symbol Device:R
- added R45: 511k, Resistor_SMD:R_0402_1005Metric, symbol Device:R_Small
- added R46: 91k, Resistor_SMD:R_0402_1005Metric, symbol Device:R_Small
- added R47: 100k, Resistor_SMD:R_0402_1005Metric, symbol Device:R_Small
- added U10: TPS63805YFFR, lcsc:DSBGA-15_L2.3-W1.3-R5-C3-P0.40-TL, symbol lcsc:TPS63805YFFR
Connections:
- net +3V3: now also C57.1
- net +3V3_OUT: now also C19.1, R45.1, U10.E2 (VOUT), U10.E3 (VOUT)
- net GND: now also C19.2, C57.2, R46.2, U10.C1 (AGND), U10.C2 (GND), U10.C3 (GND)
- net PS_SYNC: now also R44.2, U10.B1 (MODE)
- net VBUS: now also D7.2 (A)
- net VIN: now also C66.1, R14.1, C9.1, R44.1, R47.1
- net at C66.2, C67.1, SW2.2: now also U10.A1 (EN)
- net at C54.2, C55.2, U4.4 (VDD): now also D7.1 (K)
- net VBAT_READ renamed VBAT_READ_EN
- new net: C9.2, U10.A2 (VIN), U10.A3 (VIN)
- new net: L1.2, U10.B2 (L1), U10.B3 (L1)
- new net: R45.2, R46.1, U10.D1 (FB)
- new net: L1.1, U10.D2 (L2), U10.D3 (L2)
- new net: R47.2, U10.E1 (PG)
- no-connect marks 1 -> 0
Other:
- note added: "Battery connector"
- note added: "place close to TPS63805YFFR"
- note removed: "place close to TPS63020DSJR"
- moved on the sheet: C66, C67, R14, R16, SW2
