File: power.kicad_sch (KiCad schematic)
At the start: 28 parts, among them Q1 JSM2301S, SW2 SK-3296S-01-L1, U1 PH-2AWB, U10 TPS63805YFFR, U4 XT4054K421MR-G

Commit message: Diodes in spec now for the display driver.
Parts:
- removed D2: B160_13F, Diode_SMD:D_SMA, symbol Device:D
- added D6: 1N5819WS, Diode_SMD:D_SOD-323, symbol Diode:1N5819WS
- U4: Datasheet EN (none) -> http://www.natlinear.com/en/Public/Home/default/static/PDF/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
Connections:
- net VBUS: now also D6.2 (A)
- net VIN: now also D6.1 (K)
- net VBAT renamed VBAT_READ
Other:
- note added: "R25 = R_PROG VPROG = 1V (constant current charging) IBAT = (1v/2k)*1000 = 0.5A"
- moved on the sheet: D1

Commit message: Switched to recycled e-ink screen, using the Tanoshii measuremens and distances.
Parts:
- removed D1: ESD prot., Diode_SMD:D_SOD-323, symbol Device:D_TVS

Commit message: Fix power supply, use PG signal to hold reset until the power is stable.
Parts:
- removed R47: 100k, Resistor_SMD:R_0402_1005Metric, symbol Device:R_Small
- removed SW2: SK-3296S-01-L1, lcsc:SW-SMD_3P-P1.50_L2.7-W6.6, symbol lcsc:SK-3296S-01-L1
- added SW3: MS-22D28-G020, lcsc:SW-SMD_MS-22D28-G020, symbol lcsc:MS-22D28-G020
Connections:
- net GND: now also C9.2, SW3.4
- net VIN: now also U10.A2 (VIN), U10.A3 (VIN)
- net at C66.2, C67.1, U10.A1 (EN): now also SW3.2
- net PG: now reaches U10.E1 (PG)
- net at R14.2: now also SW3.3
- net at C67.2, R16.2: now also SW3.1
Other:
- note added: "VIN: Range between VBAT and VBUS, 3.0 and 5.5V Absolete max 6.0V 3V3_OUT: Stabilized 3V3 using BUCK boost converter VBUS: Between 0 and 5.5V, directly from the USB-C connector"
- moved on the sheet: C9

Commit message: Fixed schematic to have 0 DRC errors, changed display connector.
Parts:
- added R20: 3.3k, Resistor_SMD:R_0402_1005Metric, symbol Device:R_Small
Connections:
- net GND: now also SW3.5, SW3.6
- net PG: now also R20.2; no longer U10.E1 (PG)
- new net: R20.1, U10.E1 (PG)
Other:
- note added: "Max 1mA sink on PG pin"
Changed lines of the file:
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@@
 		)
 	)
+	(text "Max 1mA sink on PG pin"
+		(exclude_from_sim no)
+		(at 226.568 54.356 0)
+		(effects
+			(font
+				(size 1.27 1.27)
+			)
+		)
+	)
 	(text "IBAT = (1 / 2000) * 1000 = 500mA"
 		(exclude_from_sim no)
@@
 	)
 	(junction
+		(at 57.15 154.94)
+		(diameter 0)
+		(color 0 0 0 0)
+	)
+	(junction
 		(at 149.86 160.02)
 		(diameter 0)
@@
 	)
 	(junction
+		(at 120.65 62.23)
+		(diameter 0)
+		(color 0 0 0 0)
+	)
+	(junction
 		(at 152.4 57.15)
 		(diameter 0)
@@
 		(color 0 0 0 0)
 	)
+	(junction
+		(at 120.65 67.31)
+		(diameter 0)
+		(color 0 0 0 0)
+	)
 	(wire
 		(pts
@@
 	(wire
 		(pts
+			(xy 120.65 62.23) (xy 120.65 67.31)
+		)
+		(stroke
+			(width 0)
+			(type default)
+		)
+	)
+	(wire
+		(pts
 			(xy 219.71 69.85) (xy 219.71 72.39)
 		)
@@
 	(wire
 		(pts
+			(xy 120.65 59.69) (xy 123.19 59.69)
+		)
+		(stroke
+			(width 0)
+			(type default)
+		)
+	)
+	(wire
+		(pts
 			(xy 189.23 80.01) (xy 193.04 80.01)
 		)
@@
 	(wire
 		(pts
-			(xy 77.47 154.94) (xy 50.8 154.94)
+			(xy 77.47 154.94) (xy 57.15 154.94)
 		)
 		(stroke
@@
 	(wire
 		(pts
+			(xy 245.11 57.15) (xy 255.27 57.15)
+		)
+		(stroke
+			(width 0)
+			(type default)
+		)
+	)
+	(wire
+		(pts
 			(xy 189.23 82.55) (xy 193.04 82.55)
 		)
@@
 	(wire
 		(pts
+			(xy 120.65 62.23) (xy 123.19 62.23)
+		)
+		(stroke
+			(width 0)
+			(type default)
+		)
+	)
+	(wire
+		(pts
 			(xy 229.87 62.23) (xy 241.3 62.23)
 		)
@@
 	(wire
 		(pts
+			(xy 57.15 154.94) (xy 50.8 154.94)
+		)
+		(stroke
+			(width 0)
+			(type default)
+		)
+	)
+	(wire
+		(pts
 			(xy 152.4 68.58) (xy 152.4 69.85)
 		)
@@
 	(wire
 		(pts
-			(xy 219.71 57.15) (xy 255.27 57.15)
+			(xy 219.71 57.15) (xy 240.03 57.15)
 		)
 		(stroke
@@
 	(wire
 		(pts
+			(xy 120.65 59.69) (xy 120.65 62.23)
+		)
+		(stroke
+			(width 0)
+			(type default)
+		)
+	)
+	(wire
+		(pts
 			(xy 152.4 68.58) (xy 139.7 68.58)
 		)
@@
 	)
 	(symbol
+		(lib_id "power:PWR_FLAG")
+		(at 57.15 154.94 0)
+		(unit 1)
+		(exclude_from_sim no)
+		(in_bom yes)
+		(on_board yes)
+		(dnp no)
+		(fields_autoplaced yes)
+		(property "Reference" "#FLG01"
+			(at 57.15 153.035 0)
+			(effects
+				(font
+					(size 1.27 1.27)
+				)
+				(hide yes)
+			)
+		)
+		(property "Value" "PWR_FLAG"
+			(at 57.15 149.86 0)
+			(effects
+				(font
+					(size 1.27 1.27)
+				)
+			)
+		)
+		(property "Footprint" ""
+			(at 57.15 154.94 0)
+			(effects
+				(font
+					(size 1.27 1.27)
+				)
+				(hide yes)
+			)
+		)
+		(property "Datasheet" "~"
+			(at 57.15 154.94 0)
+			(effects
+				(font
+					(size 1.27 1.27)
+				)
+				(hide yes)
+			)
+		)
+		(property "Description" "Special symbol for telling ERC where power comes from"
+			(at 57.15 154.94 0)
+			(effects
+				(font
+					(size 1.27 1.27)
+				)
+				(hide yes)
+			)
+		)
+		(pin "1"
+		)
+		(instances
+			(project ""
+				(path "/23bf5400-d19c-445b-8744-b63ebcca303d/333d98a8-e6a2-433c-bb9c-6f407290c160"
+					(reference "#FLG01")
+					(unit 1)
+				)
+			)
+		)
+	)
+	(symbol
 		(lib_id "power:GND")
 		(at 185.42 57.15 0)
@@
 					(unit 1)
 				)
+			)
+		)
+	)
+	(symbol
+		(lib_id "Device:R_Small")
+		(at 242.57 57.15 90)
+		(unit 1)
+		(exclude_from_sim no)
+		(in_bom yes)
+		(on_board yes)
+		(dnp no)
+		(fields_autoplaced yes)
+		(property "Reference" "R20"
+			(at 242.57 52.07 90)
+			(effects
+				(font
+					(size 1.016 1.016)
+				)
+			)
+		)
+		(property "Value" "3.3k"
+			(at 242.57 54.61 90)
+			(effects
+				(font
+					(size 1.27 1.27)
+				)
+			)
+		)
+		(property "Footprint" "Resistor_SMD:R_0402_1005Metric"
+			(at 242.57 57.15 0)
+			(effects
+				(font
+					(size 1.27 1.27)
+				)
+				(hide yes)
+			)
+		)
+		(property "Datasheet" "https://jlcpcb.com/partdetail/26633-0402WGF3301TCE/C25890"
+			(at 242.57 57.15 0)
+			(effects
+				(font
+					(size 1.27 1.27)
+				)
+				(hide yes)
+			)
+		)
+		(property "Description" "Resistor, small symbol"
+			(at 242.57 57.15 0)
+			(effects
+				(font
+					(size 1.27 1.27)
+				)
+				(hide yes)
+			)
+		)
+		(property "LCSC" "C25890"
+			(at 242.57 57.15 90)
+			(effects
+				(font
+					(size 1.27 1.27)
+				)
+				(hide yes)
+			)
+		)
+		(pin "2"
+		)
+		(pin "1"
+		)
+		(instances
+			(project ""
+				(path "/23bf5400-d19c-445b-8744-b63ebcca303d/333d98a8-e6a2-433c-bb9c-6f407290c160"
+					(reference "R20")
+					(unit 1)
+				)

Commit message: Add MA logo, test points, tuned RF LoRa.
Parts:
- added TP10, TP5, TP6, TP7, TP8, TP9: TestPoint, TestPoint:TestPoint_Pad_1.0x1.0mm, symbol Connector:TestPoint
Connections:
- net GND: now also TP10.1, TP6.1, TP8.1
- net VBUS: now also TP7.1
- net VIN: now also TP9.1
- net at C56.1, Q1.3 (D), R34.2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: now also TP5.1

Commit message: dotting the i's , list checks before V2 order.
Parts:
- added TP12, TP13: TestPoint, TestPoint:TestPoint_Pad_1.0x1.0mm, symbol Connector:TestPoint
- SW3: LCSC (none) -> C963205
- TP10, TP6, TP8: now not fitted
- TP5, TP7, TP9: now not fitted; now left out of the parts list
Connections:
- net PS_SYNC: now also TP13.1
- net at R20.1, U10.E1 (PG): now also TP12.1
Other:
- moved on the sheet: R44

Commit message: Updated readme.md for Prototype V2. Simplified NRF IO net names.
Parts:
- SW3: FT Rotation Offset (none) -> 180
Connections:
- net P1.08_CHRG renamed BAT_CHARGE
Changed lines of the file:
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@@
 		)
 	)
-	(hierarchical_label "P1.08_CHRG"
+	(hierarchical_label "BAT_CHARGE"
 		(shape output)
 		(at 91.44 165.1 0)
@@
 			(at 130.81 62.23 90)
 			(effects
+				(font
+					(size 1.27 1.27)
+				)
+				(hide yes)
+			)
+		)
+		(property "FT Rotation Offset" "180"
+			(at 130.81 62.23 90)
+			(effects
