File: sx1262.kicad_sch (KiCad schematic)
At the start: 21 parts, among them U3 SX1262IMLTRT, U4 BGS12SN6E6327XTSA1, X2 S201632M10PF10PPM

Commit message: Fixed mistake in NRF52 footprint, add NAND FLASH, add NFC antenna schematic.
Parts:
- renumbered C28 to C21, C31 to C22, C29 to C23, C30 to C24, C21 to C25, C22 to C26, C23 to C27, C24 to C28, C25 to C29, C26 to C30, C27 to C31, L8 to L4, L7 to L5, L5 to L6, L4 to L7, L6 to L8
Other:
- note added: "TODO: Implement the switchless design, because cheaper"
- company: (none) -> Badge.Team
- title: (none) -> Bornhack 2026

Commit message: PCB layout egg shape, for reference.
Parts:
- C22: footprint (none) -> Capacitor_SMD:C_0603_1608Metric; LCSC (none) -> C1623
- C25: footprint (none) -> Capacitor_SMD:C_0603_1608Metric; LCSC (none) -> C1622
- C26, C29: footprint (none) -> Capacitor_SMD:C_0402_1005Metric; LCSC (none) -> C472454
- C27: footprint (none) -> Capacitor_SMD:C_0402_1005Metric; LCSC (none) -> C1523
- C28: value C_Small -> 1nF; footprint (none) -> Capacitor_SMD:C_0402_1005Metric; LCSC (none) -> C1523
- C30, C31: footprint (none) -> Capacitor_SMD:C_0402_1005Metric; LCSC (none) -> C52052
Changed lines of the file:
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@@
 	)
 	(junction
-		(at 232.41 105.41)
+		(at 44.45 99.06)
 		(diameter 0)
 		(color 0 0 0 0)
 	)
 	(junction
-		(at 31.75 35.56)
+		(at 232.41 105.41)
 		(diameter 0)
 		(color 0 0 0 0)
 	)
 	(junction
-		(at 266.7 86.36)
+		(at 31.75 35.56)
 		(diameter 0)
 		(color 0 0 0 0)
 	)
 	(junction
-		(at 46.99 99.06)
+		(at 266.7 86.36)
 		(diameter 0)
 		(color 0 0 0 0)
@@
 	(wire
 		(pts
+			(xy 44.45 99.06) (xy 46.99 99.06)
+		)
+		(stroke
+			(width 0)
+			(type default)
+		)
+	)
+	(wire
+		(pts
 			(xy 232.41 105.41) (xy 240.03 105.41)
 		)
@@
 	(wire
 		(pts
-			(xy 46.99 93.98) (xy 46.99 99.06)
+			(xy 44.45 93.98) (xy 44.45 99.06)
 		)
 		(stroke
@@
 	(wire
 		(pts
-			(xy 46.99 93.98) (xy 83.82 93.98)
+			(xy 44.45 93.98) (xy 83.82 93.98)
 		)
 		(stroke
@@
 	(wire
 		(pts
-			(xy 40.64 99.06) (xy 46.99 99.06)
+			(xy 40.64 99.06) (xy 44.45 99.06)
 		)
 		(stroke
@@
 		(on_board yes)
 		(dnp no)
-		(fields_autoplaced yes)
 		(property "Reference" "L5"
-			(at 49.53 93.98 90)
+			(at 49.53 97.028 90)
 			(effects
 				(font
@@
 		)
 		(property "Value" "15uH"
-			(at 49.53 96.52 90)
+			(at 49.53 100.584 90)
 			(effects
 				(font
@@
 			)
 		)
-		(property "Footprint" ""
+		(property "Footprint" "Capacitor_SMD:C_0402_1005Metric"
 			(at 250.19 91.44 0)
 			(effects
@@
 			)
 		)
-		(property "Datasheet" "~"
+		(property "Datasheet" "https://jlcpcb.com/partdetail/53065-0402CG3R6C500NT/C52052"
 			(at 250.19 91.44 0)
 			(effects
@@
 			)
 		)
+		(property "LCSC" "C52052"
+			(at 250.19 91.44 0)
+			(effects
+				(font
+					(size 1.27 1.27)
+				)
+				(hide yes)
+			)
+		)
 		(pin "2"
 		)
@@
 			)
 		)
-		(property "Value" "C_Small"
+		(property "Value" "1nF"
 			(at 234.95 111.7662 0)
 			(effects
@@
 			)
 		)
-		(property "Footprint" ""
+		(property "Footprint" "Capacitor_SMD:C_0402_1005Metric"
 			(at 232.41 110.49 0)
 			(effects
@@
 			)
 		)
-		(property "Datasheet" "~"
+		(property "Datasheet" "https://jlcpcb.com/partdetail/1875-0402B102K500NT/C1523"
 			(at 232.41 110.49 0)
 			(effects
@@
 			)
 		)
+		(property "LCSC" "C1523"
+			(at 232.41 110.49 0)
+			(effects
+				(font
+					(size 1.27 1.27)
+				)
+				(hide yes)
+			)
+		)
 		(pin "2"
 		)
@@
 			)
 		)
-		(property "Footprint" ""
+		(property "Footprint" "Capacitor_SMD:C_0603_1608Metric"
 			(at 40.64 106.68 0)
 			(effects
@@
 			)
 		)
-		(property "Datasheet" "~"
+		(property "Datasheet" "https://jlcpcb.com/partdetail/1975-CL10B474KA8NNNC/C1623"
 			(at 40.64 106.68 0)
 			(effects
@@
 			)
 		)
+		(property "LCSC" "C1623"
+			(at 40.64 106.68 0)
+			(effects
+				(font
+					(size 1.27 1.27)
+				)
+				(hide yes)
+			)
+		)
 		(pin "2"
 		)
@@
 			)
 		)
-		(property "Footprint" ""
+		(property "Footprint" "Capacitor_SMD:C_0402_1005Metric"
 			(at 158.75 68.58 0)
 			(effects
@@
 			)
 		)
-		(property "Datasheet" "~"
+		(property "Datasheet" "https://jlcpcb.com/partdetail/478910-CL05C470JB51PNC/C472454"
 			(at 158.75 68.58 0)
 			(effects
@@
 			)
 		)
+		(property "LCSC" "C472454"
+			(at 158.75 68.58 90)
+			(effects
+				(font
+					(size 1.27 1.27)
+				)
+				(hide yes)
+			)
+		)
 		(pin "1"
 		)
@@
 			)
 		)
-		(property "Footprint" ""
+		(property "Footprint" "Capacitor_SMD:C_0402_1005Metric"
 			(at 266.7 91.44 0)
 			(effects
@@
 			)
 		)
-		(property "Datasheet" "~"
+		(property "Datasheet" "https://jlcpcb.com/partdetail/53065-0402CG3R6C500NT/C52052"
 			(at 266.7 91.44 0)
 			(effects
@@
 			)
 		)
+		(property "LCSC" "C52052"
+			(at 266.7 91.44 0)
+			(effects
+				(font
+					(size 1.27 1.27)
+				)
+				(hide yes)
+			)
+		)
 		(pin "2"
 		)
@@
 			)
 		)
-		(property "Footprint" ""
+		(property "Footprint" "Capacitor_SMD:C_0603_1608Metric"
 			(at 152.4 68.58 0)
 			(effects
@@
 			)
 		)
-		(property "Datasheet" "~"
+		(property "Datasheet" "https://jlcpcb.com/partdetail/1974-CL10B473KB8NNNC/C1622"
 			(at 152.4 68.58 0)
 			(effects
@@
 			)
 		)
+		(property "LCSC" "C1622"
+			(at 152.4 68.58 90)
+			(effects
+				(font
+					(size 1.27 1.27)
+				)
+				(hide yes)
+			)
+		)
 		(pin "1"
 		)
@@
 			)
 		)
-		(property "Footprint" ""
+		(property "Footprint" "Capacitor_SMD:C_0402_1005Metric"
 			(at 228.6 66.04 0)
 			(effects
@@
 			)
 		)
-		(property "Datasheet" "~"
+		(property "Datasheet" "https://jlcpcb.com/partdetail/1875-0402B102K500NT/C1523"
 			(at 228.6 66.04 0)
 			(effects
@@
 			)
 		)
+		(property "LCSC" "C1523"
+			(at 228.6 66.04 0)
+			(effects
+				(font
+					(size 1.27 1.27)
+				)
+				(hide yes)
+			)
+		)
 		(pin "2"
 		)
@@
 			)
 		)
-		(property "Footprint" ""
+		(property "Footprint" "Capacitor_SMD:C_0402_1005Metric"
 			(at 245.11 86.36 0)
 			(effects
@@
 			)
 		)
-		(property "Datasheet" "~"
+		(property "Datasheet" "https://jlcpcb.com/partdetail/478910-CL05C470JB51PNC/C472454"
 			(at 245.11 86.36 0)
 			(effects
@@
 			(effects
 				(font
+					(size 1.27 1.27)
+				)
+				(hide yes)
+			)
+		)
+		(property "LCSC" "C472454"
+			(at 245.11 86.36 90)
+			(effects
+				(font

Commit message: Switched the LC filters from ceramic LoRa filter.
Parts:
- removed L4: 15uH, symbol Device:L_Small
- removed L7: 0900FM15D0039001E, lcsc:FILTER-SMD_10P-L2.0-W1.3-BL, symbol lcsc:0900FM15D0039001E
- removed U4: BGS12SN6E6327XTSA1, lcsc:TSNP-6_L1.1-W0.7-P0.40-BL, symbol lcsc:BGS12SN6E6327XTSA1
- added C45: 3pF, Capacitor_SMD:C_0402_1005Metric, symbol Device:C_Small
- added C46: C_Small, Capacitor_SMD:C_0402_1005Metric, symbol Device:C_Small
- added C47: 5.6pF, Capacitor_SMD:C_0402_1005Metric, symbol Device:C_Small
- added C48: 39pF, Capacitor_SMD:C_0402_1005Metric, symbol Device:C_Small
- added C49, C50: 1.8pF, Capacitor_SMD:C_0402_1005Metric, symbol Device:C_Small
- added C51: 2.4pF, Capacitor_SMD:C_0402_1005Metric, symbol Device:C_Small
- added C52: C_Small, symbol Device:C_Small
- added C53: 1uF, symbol Device:C_Small
- added L10: 4.7nH, Inductor_SMD:L_0402_1005Metric, symbol Device:L_Small
- added L11: 0, Inductor_SMD:L_0402_1005Metric, symbol Device:L_Small
- added L12: 15nH, Capacitor_SMD:C_0402_1005Metric, symbol Device:L_Small
- added L7: 2.5nH, Capacitor_SMD:C_0402_1005Metric, symbol Device:L_Small
- added U2: TPE4259-63, lcsc:SOT-363-6_L2.0-W1.3-P0.65-LS2.1-BL, symbol lcsc:TPE4259-63
- L5: footprint (none) -> Inductor_SMD:L_0603_1608Metric; LCSC (none) -> C486329
- L6: footprint (none) -> Inductor_SMD:L_0402_1005Metric; LCSC (none) -> C27151
- L8: footprint (none) -> Inductor_SMD:L_0402_1005Metric; LCSC (none) -> C142213
- R10, R9: LCSC (none) -> C25076
- U3: LCSC (none) -> C191341
Connections:
- net 3V3: now also U3.1 (VDD_IN), C53.1
- net DIO2: now also R10.1; no longer R9.1
- net GND: now also C46.1, C47.2, C49.2, C50.1, C52.1, C53.2, U2.2 (GND)
- net LORA_RF_SW1: now also R9.1; no longer R10.1
- net at L6.2: now also C45.1, C46.2, L11.2, L7.1; no longer U3.23 (RFO)
- net at U3.22 (RFI_N): now also C51.2, L12.2
- net at U3.21 (RFI_P): now also C50.2, L12.1
- net at C28.1, R10.2: now also U2.4 (VC1)
- net at C27.1, R9.2: now also U2.6 (VC2)
- net at C29.1: now also U2.5 (RFC)
- new net: C48.2, L10.1
- new net: C49.1, L10.2, U2.1 (RF2)
- new net: C45.2, C47.1, C48.1, L7.2
- new net: C51.1, C52.2, U2.3 (RF1)
- new net: L11.1, U3.23 (RFO)
Other:
- note added: "DC-DC SW @ 3.25MHz"
- note removed: "More expensive ceramic filter 866MHz But simpler :-)"
- moved on the sheet: C27, C28, C29, C30, C31, L8, R10, R9

Commit message: Progress, routed more stuff.
Parts:
- C45: LCSC (none) -> C318583
- C47: LCSC (none) -> C16193755
- C48: LCSC (none) -> C86288
- C49, C50: LCSC (none) -> C22374861
- C51: LCSC (none) -> C48346
- C52: footprint (none) -> Capacitor_SMD:C_0402_1005Metric
- C53: footprint (none) -> Capacitor_SMD:C_0603_1608Metric; LCSC (none) -> C5199872
- L10: LCSC (none) -> C963987
- L11: LCSC (none) -> C17168
- L12: LCSC (none) -> C381880
- L7: footprint Capacitor_SMD:C_0402_1005Metric -> Inductor_SMD:L_0402_1005Metric; LCSC (none) -> C778764
- R10, R9: footprint (none) -> Resistor_SMD:R_0402_1005Metric
Connections:
- net DIO3: no longer names the net of U3.6 (DIO3)
- no-connect marks 0 -> 1

Commit message: Routed buttons to MCU.
Parts:
- C25: footprint Capacitor_SMD:C_0603_1608Metric -> Capacitor_SMD:C_0402_1005Metric; LCSC C1622 -> C82219
Changed lines of the file:
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@@
-		(length 2.54)
-		(shape diamond)
-		(at 162.56 64.77 0)
-		(fields_autoplaced yes)
-		(effects
-			(font
-				(size 1.27 1.27)
-			)
-			(justify left bottom)
-		)
-		(property "Netclass" "LORA-RF"
-			(at 163.7665 62.23 0)
-			(effects
-				(font
-					(size 1.27 1.27)
-				)
-				(justify left)
-			)
-		)
-		(property "Component Class" ""
-			(at -50.8 -6.35 0)
-			(effects
-				(font
-					(size 1.27 1.27)
-					(italic yes)
-				)
-			)
-		)
-	)
-	(netclass_flag ""
 		(length 2.54)
 		(shape diamond)
@@
 			)
 		)
-		(property "Footprint" "Capacitor_SMD:C_0603_1608Metric"
+		(property "Footprint" "Capacitor_SMD:C_0402_1005Metric"
 			(at 152.4 68.58 0)
 			(effects
@@
 			)
 		)
-		(property "Datasheet" "https://jlcpcb.com/partdetail/1974-CL10B473KB8NNNC/C1622"
+		(property "Datasheet" "https://jlcpcb.com/partdetail/83376-0402B473K500NT/C82219"
 			(at 152.4 68.58 0)
 			(effects
@@
 			)
 		)
-		(property "LCSC" "C1622"
+		(property "LCSC" "C82219"
 			(at 152.4 68.58 90)
 			(effects

Commit message: Checked PCBA for JLCPCB.
Parts:
- C45: LCSC C318583 -> C41361091
- L8: LCSC C142213 -> C98003
Changed lines of the file:
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@@
 			)
 		)
-		(property "Datasheet" "https://jlcpcb.com/partdetail/299712-CL05C030BB5NNNC/C318583"
+		(property "Datasheet" "https://jlcpcb.com/partdetail/HRE-CGA0402C0G3R0C500GT/C41361091"
 			(at 179.07 68.58 0)
 			(effects
@@
 			)
 		)
-		(property "LCSC" "C318583"
+		(property "LCSC" "C41361091"
 			(at 179.07 68.58 90)
 			(effects
@@
 			)
 		)
-		(property "Datasheet" "https://jlcpcb.com/partdetail/ChilisinElec-CLH1005T_8N2J_SNP/C142213"
+		(property "Datasheet" "https://jlcpcb.com/partdetail/MurataElectronics-LQG15HS8N2J02D/C98003"
 			(at 260.35 86.36 0)
 			(effects
@@
 			)
 		)
-		(property "LCSC" "C142213"
+		(property "LCSC" "C98003"
 			(at 260.35 86.36 90)
 			(effects

Commit message: Moved LoRa radio closer to antenna
Parts:
- added R31, R32: 0, Resistor_SMD:R_0402_1005Metric, symbol Device:R_Small
- added RF1: A-IPEX1-1.25A, lcsc:IPEX-SMD_3P-L2.6-W2.6-LS3.0_RF1200001R, symbol lcsc:A-IPEX1-1.25A
Connections:
- net GND: now also RF1.2, RF1.3
- net at C29.1: now also R31.2; no longer U2.5 (RFC)
- new net: R31.1, R32.2, RF1.1
- new net: R32.1, U2.5 (RFC)
Other:
- moved on the sheet: C29, C30, C31, L8
