File: sx1262.kicad_sch (KiCad schematic)
At the start: 35 parts, among them U2 TPE4259-63, U3 SX1262IMLTRT, X2 S201632M10PF10PPM

Commit message: Fixed PCBA rotations in using component property.
Parts:
- U2: FT Rotation Offset (none) -> 180
- U3: FT Rotation Offset (none) -> 270
Changed lines of the file:
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@@
+			)
+		)
+		(property "FT Rotation Offset" "270"
+			(at 101.6 91.44 0)
+			(effects
+				(font
+					(size 1.27 1.27)
+				)
+				(hide yes)
 			)
 		)
@@
 			(at 227.33 86.36 0)
 			(effects
+				(font
+					(size 1.27 1.27)
+				)
+				(hide yes)
+			)
+		)
+		(property "FT Rotation Offset" "180"
+			(at 227.33 86.36 0)
+			(effects

Commit message: Optimized design to use more basic components.
Parts:
- C30, C31: LCSC C52052 -> C161321
- L10: LCSC C963987 -> C86065
- L12: footprint Capacitor_SMD:C_0402_1005Metric -> Inductor_SMD:L_0402_1005Metric
- X2: value S201632M10PF10PPM -> S201632M10PF10PPM 32MHz

Commit message: Module version with ra-01sh LoRa
Parts:
- removed C21, C23: 10pF, Capacitor_SMD:C_0402_1005Metric, symbol Device:C_Small
- removed C22: 470nF, Capacitor_SMD:C_0603_1608Metric, symbol Device:C_Small
- removed C24: 100nF, Capacitor_SMD:C_0402_1005Metric, symbol Device:C_Small
- removed C25: 47nF, Capacitor_SMD:C_0402_1005Metric, symbol Device:C_Small
- removed C26, C29: 47pF, Capacitor_SMD:C_0402_1005Metric, symbol Device:C_Small
- removed C27, C28: 1nF, Capacitor_SMD:C_0402_1005Metric, symbol Device:C_Small
- removed C45: 3pF, Capacitor_SMD:C_0402_1005Metric, symbol Device:C_Small
- removed C46, C52: C_Small, Capacitor_SMD:C_0402_1005Metric, symbol Device:C_Small
- removed C47: 5.6pF, Capacitor_SMD:C_0402_1005Metric, symbol Device:C_Small
- removed C48: 39pF, Capacitor_SMD:C_0402_1005Metric, symbol Device:C_Small
- removed C49, C50: 1.8pF, Capacitor_SMD:C_0402_1005Metric, symbol Device:C_Small
- removed C51: 2.4pF, Capacitor_SMD:C_0402_1005Metric, symbol Device:C_Small
- removed C53: 1uF, Capacitor_SMD:C_0603_1608Metric, symbol Device:C_Small
- removed L10: 4.7nH, Inductor_SMD:L_0402_1005Metric, symbol Device:L_Small
- removed L11: 0, Inductor_SMD:L_0402_1005Metric, symbol Device:L_Small
- removed L12: 15nH, Inductor_SMD:L_0402_1005Metric, symbol Device:L_Small
- removed L5: 15uH, Inductor_SMD:L_0603_1608Metric, symbol Device:L_Small
- removed L6: 47nH, Inductor_SMD:L_0402_1005Metric, symbol Device:L_Small
- removed L7: 2.5nH, Inductor_SMD:L_0402_1005Metric, symbol Device:L_Small
- removed L8: 8.2nH, Inductor_SMD:L_0402_1005Metric, symbol Device:L_Small
- removed R10: 100, Resistor_SMD:R_0402_1005Metric, symbol Device:R_Small
- removed R31, R32: 0, Resistor_SMD:R_0402_1005Metric, symbol Device:R_Small
- removed RF1: A-IPEX1-1.25A, lcsc:IPEX-SMD_3P-L2.6-W2.6-LS3.0_RF1200001R, symbol lcsc:A-IPEX1-1.25A
- removed U2: TPE4259-63, lcsc:SOT-363-6_L2.0-W1.3-P0.65-LS2.1-BL, symbol lcsc:TPE4259-63
- removed U3: SX1262IMLTRT, lcsc:QFN-24_L4.0-W4.0-P0.50-BL-EP2.6, symbol lcsc:SX1262IMLTRT
- removed X2: S201632M10PF10PPM 32MHz, lcsc:CRYSTAL-SMD_4P-L2.0-W1.6-BL, symbol lcsc:S201632M10PF10PPM
- added C19: 100nF, Capacitor_SMD:C_0402_1005Metric, symbol Device:C_Small
- added C9: 1uF, Capacitor_SMD:C_0603_1608Metric, symbol Device:C_Small
- added L1: RA-01SH, lcsc:WIRELM-SMD_RA-01SH, symbol lcsc:RA-01SH
- C30, C31: now not fitted; now left out of the parts list
- R9: value 100 -> 0; LCSC C25076 -> C17168
Connections:
- net LORA_RF_SW1 is gone; now on an unnamed net: R9.1
- net 3V3: now also C19.2, C9.1, L1.3 (3.3V)
- net GND: now also C19.1, C9.2, L1.16 (GND), L1.2 (GND), L1.9 (GND)
- net LORA_ANT: now also R9.2
- net LORA_BUSY: now also L1.10 (BUSY)
- net LORA_DIO1: now also L1.6 (DIO1)
- net LORA_RST: now also L1.4 (RESET)
- net LORA_SPI_MISO: now also L1.13 (MISO)
- net LORA_SPI_MOSI: now also L1.14 (MOSI)
- net LORA_SPI_NSS: now also L1.15 (NSS)
- net LORA_SPI_SCK: now also L1.12 (SCK)
- net at C30.1: now also L1.1 (ANT)
- no-connect marks 1 -> 4
Other:
- note removed: "AN1200.91 Layout reference Page 5"
- note removed: "DC-DC SW @ 3.25MHz"
- note removed: "Main MCU Clock oscillator"
- note removed: "Reference design AN1200.54 BOM page 19"
- note removed: "TODO: Implement the switchless design, because cheaper"
