File: sx1262.kicad_sch (KiCad schematic)
At the start: 35 parts, among them U2 TPE4259-63, U3 SX1262IMLTRT, X2 S201632M10PF10PPM 32MHz

Commit message: Improvements, now need to know the specs for the new display module.
Parts:
- C21, C23: now not fitted; now left out of the parts list
Changed lines of the file:
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@@
 		(unit 1)
 		(exclude_from_sim no)
-		(in_bom yes)
+		(in_bom no)
 		(on_board yes)
-		(dnp no)
+		(dnp yes)
 		(fields_autoplaced yes)
 		(property "Reference" "C23"
@@
 		(unit 1)
 		(exclude_from_sim no)
-		(in_bom yes)
+		(in_bom no)
 		(on_board yes)
-		(dnp no)
+		(dnp yes)
 		(fields_autoplaced yes)
 		(property "Reference" "C21"

Commit message: Changed out RF switch and display connector for parts that are stil available.
Parts:
- U2: value TPE4259-63 -> ZHHXDZ HXCKRF2179MM26-C4; LCSC C47117600 -> C49010109
Changed lines of the file:
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@@
 			)
 		)
-		(property "Value" "TPE4259-63"
+		(property "Value" "ZHHXDZ HXCKRF2179MM26-C4"
 			(at 227.33 78.74 0)
 			(effects
@@
 			)
 		)
-		(property "Datasheet" "https://jlcpcb.com/partdetail/TECHPUBLIC-TPE425963/C47117600"
+		(property "Datasheet" "https://jlcpcb.com/partdetail/ZHHXDZ-HXCKRF2179MM26C4/C49010109"
 			(at 227.33 86.36 0)
 			(effects
@@
 			)
 		)
-		(property "Description" "0.6dB 0Hz~2.5GHz 30dB 31dBm SPDT SOT-363 RF Switches ROHS"
+		(property "Description" "0.65dB 32dBm 39dB 50MHz~3GHz SPDT SOT-363 RF Switches ROHS"
 			(at 227.33 86.36 0)
 			(effects
@@
 			)
 		)
-		(property "LCSC" "C47117600"
+		(property "LCSC" "C49010109"
 			(at 227.33 99.06 0)
 			(effects

Commit message: Add MA logo, test points, tuned RF LoRa.
Parts:
- removed C21, C23: 10pF, Capacitor_SMD:C_0402_1005Metric, symbol Device:C_Small
- C30: value 3.6pF -> 1.8pF; LCSC C161321 -> C22374861
- C31: now not fitted; now left out of the parts list
- C45: value 3pF -> 3.3pF; LCSC C41361091 -> C2941931
- C49: value 1.8pF -> 2.2pF; LCSC C22374861 -> C325452
- L8: value 8.2nH -> 7.5nH; LCSC C98003 -> C98001; Resource (none) -> https://www.ti.com/lit/an/swra496a/swra496a.pdf?ts=17717855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
Other:
- note added: "https://www.ti.com/lit/an/swra496a/swra496a.pdf?ts=1771785552812 Page 35/36 Matching circuit 50 Ohm RF source to antenna"
- moved on the sheet: C53
