File: input.kicad_sch (KiCad schematic)
At the start: 0 parts

Commit message: Progress, routed more stuff.
Parts:
- added R15: 10k, Resistor_SMD:R_0402_1005Metric, symbol Device:R_Small
- added SW1: TS-1187A-B-A-B, lcsc:SW-SMD_4P-L5.1-W5.1-P3.70-LS6.5-TL_H1.5, symbol lcsc:TS-1187A-B-A-B
Connections:
- net 3V3: now also R15.1
- net BTN_RESET: now also R15.2, SW1.2 (B)
- new net GND: SW1.3 (C)
- no-connect marks 0 -> 2
Other:
- removed sheet CANCEL
- removed sheet GAMES_SNACKS
- removed sheet MEAL
- removed sheet MEDICINE_DISCIPLINE
- removed sheet RESET
- removed sheet SELECT
- note added: "Based On Tamagotchi Buttons: https://www.jnlgame.com/cdn/shop/files/81tR9PHvDtL._AC_SL1500.jpg?v=1702227711&width=5760"
- note added: "https://jlcpcb.com/partdetail/ALPSALPINE-SKPMAME010/C115348 Betere knop"
- note added: "https://jlcpcb.com/partdetail/ALPSALPINE-SKRHABE010/C139794 knoppen"
- note removed: "Based On Tamagotchi Buttons: https://tamagotchicrossing.com/tamagotchi/yasashii/log1/yasashiibuttons.jpg"

Commit message: Bluetooth antenna should work better, NFC has IPEX for tuning.
Parts:
- added R18, R22, R23, R27, R28: 10k, Resistor_SMD:R_0402_1005Metric, symbol Device:R_Small
- added SW3: SKRHABE010, lcsc:SW-SMD_SKRHABE010, symbol lcsc:SKRHABE010
- SW1: Label (none) -> RESET
Connections:
- net 3V3: now also R18.1, R22.1, R23.1, R27.1, R28.1
- net GND: now also SW3.5 (COM), SW3.7, SW3.8
- new net BTN_JOY_DOWN: R18.2, SW3.6 (B)
- new net BTN_JOY_FIRE: R23.2, SW3.2 (CEN)
- new net BTN_JOY_LEFT: R28.2, SW3.3 (C)
- new net BTN_JOY_RIGHT: R22.2, SW3.4 (D)
- new net BTN_JOY_UP: R27.2, SW3.1 (A)

Commit message: Connected up buttons, labeled buttons, added some via stitching.
Other:
- sheet STATS renamed CANCEL
- sheet TOILET renamed EXECUTE
- removed sheet LIGHTS
Changed lines of the file:
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@@
-	)
-	(junction
-		(at 55.88 72.39)
-		(diameter 0)
-		(color 0 0 0 0)
 	)
 	(junction
@@
 	(wire
 		(pts
-			(xy 55.88 82.55) (xy 58.42 82.55)
+			(xy 55.88 71.12) (xy 58.42 71.12)
 		)
 		(stroke
@@
 	(wire
 		(pts
-			(xy 87.63 72.39) (xy 99.06 72.39)
-		)
-		(stroke
-			(width 0)
-			(type default)
-		)
-	)
-	(wire
-		(pts
 			(xy 176.53 86.36) (xy 198.12 86.36)
 		)
@@
 	(wire
 		(pts
-			(xy 55.88 72.39) (xy 58.42 72.39)
-		)
-		(stroke
-			(width 0)
-			(type default)
-		)
-	)
-	(wire
-		(pts
 			(xy 55.88 109.22) (xy 55.88 115.57)
 		)
@@
 	(wire
 		(pts
-			(xy 87.63 82.55) (xy 99.06 82.55)
+			(xy 87.63 71.12) (xy 99.06 71.12)
 		)
 		(stroke
@@
 	(wire
 		(pts
-			(xy 55.88 72.39) (xy 55.88 82.55)
+			(xy 55.88 62.23) (xy 55.88 71.12)
 		)
 		(stroke
@@
 		(pts
 			(xy 176.53 67.31) (xy 176.53 68.58)
-		)
-		(stroke
-			(width 0)
-			(type default)
-		)
-	)
-	(wire
-		(pts
-			(xy 55.88 62.23) (xy 55.88 72.39)
 		)
 		(stroke
@@
 		)
 	)
-	(hierarchical_label "BTN_SELECT"
+	(hierarchical_label "BTN_EXECUTE"
 		(shape output)
 		(at 99.06 62.23 0)
@@
 		)
 	)
-	(hierarchical_label "BTN_CONFIRM"
-		(shape output)
-		(at 99.06 72.39 0)
-		(effects
-			(font
-				(size 1.27 1.27)
-			)
-			(justify left)
-		)
-	)
 	(hierarchical_label "BTN_JOY_LEFT"
 		(shape output)
@@
 	(hierarchical_label "BTN_CANCEL"
 		(shape output)
-		(at 99.06 82.55 0)
+		(at 99.06 71.12 0)
 		(effects
 			(font
@@
 	)
 	(sheet
-		(at 58.42 80.01)
+		(at 58.42 68.58)
 		(size 29.21 5.08)
 		(exclude_from_sim no)
@@
 			(color 0 0 0 0.0000)
 		)
-		(property "Sheetname" "STATS"
-			(at 58.42 78.74 0)
+		(property "Sheetname" "CANCEL"
+			(at 58.42 67.31 0)
 			(effects
 				(font
@@
 		)
 		(property "Sheetfile" "gen_button.kicad_sch"
-			(at 58.42 85.6746 0)
+			(at 58.42 74.2446 0)
 			(effects
 				(font
@@
 		)
 		(pin "3V3" input
-			(at 58.42 82.55 180)
+			(at 58.42 71.12 180)
 			(effects
 				(font
@@
 		)
 		(pin "BTN_OUT" output
-			(at 87.63 82.55 0)
+			(at 87.63 71.12 0)
 			(effects
 				(font
@@
 				(path "/23bf5400-d19c-445b-8744-b63ebcca303d/1f4fc1c2-c6dd-4c37-a48b-5ed4d54351cc"
 					(page "15")
-				)
-			)
-		)
-	)
-	(sheet
-		(at 58.42 69.85)
-		(size 29.21 5.08)
-		(exclude_from_sim no)
-		(in_bom no)
-		(on_board no)
-		(dnp yes)
-		(stroke
-			(width 0.1524)
-			(type solid)
-		)
-		(fill
-			(color 0 0 0 0.0000)
-		)
-		(property "Sheetname" "LIGHTS"
-			(at 58.42 68.58 0)
-			(effects
-				(font
-					(size 1.27 1.27)
-				)
-				(justify left bottom)
-				(hide yes)
-			)
-		)
-		(property "Sheetfile" "gen_button.kicad_sch"
-			(at 58.42 75.5146 0)
-			(effects
-				(font
-					(size 1.27 1.27)
-				)
-				(justify left top)
-			)
-		)
-		(pin "3V3" input
-			(at 58.42 72.39 180)
-			(effects
-				(font
-					(size 1.27 1.27)
-				)
-				(justify left)
-			)
-		)
-		(pin "BTN_OUT" output
-			(at 87.63 72.39 0)
-			(effects
-				(font
-					(size 1.27 1.27)
-				)
-				(justify right)
-			)
-		)
-		(instances
-			(project "bornhack2026-hardware"
-				(path "/23bf5400-d19c-445b-8744-b63ebcca303d/1f4fc1c2-c6dd-4c37-a48b-5ed4d54351cc"
-					(page "14")
 				)
 			)
@@
 			(color 0 0 0 0.0000)
 		)
-		(property "Sheetname" "TOILET"
+		(property "Sheetname" "EXECUTE"
 			(at 58.42 58.42 0)
 			(effects

Commit message: Moved battery connector out of the way of the battery.
Parts:
- added C72: 1uF, Capacitor_SMD:C_0603_1608Metric, symbol symbols:C
Connections:
- net BTN_RESET: now also C72.2
- net GND: now also C72.1
Changed lines of the file:
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@@
+	(wire
+		(pts
+			(xy 82.55 109.22) (xy 82.55 115.57)
+		)
+		(stroke
+			(width 0)
+			(type default)
+		)
+	)
 	(wire
 		(pts
@@
 	)
 	(symbol
+		(lib_id "power:GND")
+		(at 82.55 115.57 0)
+		(unit 1)
+		(exclude_from_sim no)
+		(in_bom yes)
+		(on_board yes)
+		(dnp no)
+		(fields_autoplaced yes)
+		(property "Reference" "#PWR019"
+			(at 82.55 121.92 0)
+			(effects
+				(font
+					(size 1.27 1.27)
+				)
+				(hide yes)
+			)
+		)
+		(property "Value" "GND"
+			(at 82.55 120.65 0)
+			(effects
+				(font
+					(size 1.27 1.27)
+				)
+			)
+		)
+		(property "Footprint" ""
+			(at 82.55 115.57 0)
+			(effects
+				(font
+					(size 1.27 1.27)
+				)
+				(hide yes)
+			)
+		)
+		(property "Datasheet" ""
+			(at 82.55 115.57 0)
+			(effects
+				(font
+					(size 1.27 1.27)
+				)
+				(hide yes)
+			)
+		)
+		(property "Description" "Power symbol creates a global label with name \"GND\" , ground"
+			(at 82.55 115.57 0)
+			(effects
+				(font
+					(size 1.27 1.27)
+				)
+				(hide yes)
+			)
+		)
+		(pin "1"
+		)
+		(instances
+			(project "bornhack2026-hardware"
+				(path "/23bf5400-d19c-445b-8744-b63ebcca303d/1f4fc1c2-c6dd-4c37-a48b-5ed4d54351cc"
+					(reference "#PWR019")
+					(unit 1)
+				)
+			)
+		)
+	)
+	(symbol
 		(lib_id "lcsc:TS-1187A-B-A-B")
 		(at 68.58 104.14 0)
@@
 					(unit 1)
 				)
+			)
+		)
+	)
+	(symbol
+		(lib_id "symbols:C")
+		(at 82.55 105.41 180)
+		(unit 1)
+		(exclude_from_sim no)
+		(in_bom yes)
+		(on_board yes)
+		(dnp no)
+		(property "Reference" "C72"
+			(at 88.9 104.14 0)
+			(effects
+				(font
+					(size 1.27 1.27)
+				)
+				(justify left)
+			)
+		)
+		(property "Value" "1uF"
+			(at 87.63 106.68 0)
+			(effects
+				(font
+					(size 1.27 1.27)
+				)
+				(justify left)
+			)
+		)
+		(property "Footprint" "Capacitor_SMD:C_0603_1608Metric"
+			(at 81.5848 101.6 0)
+			(effects
+				(font
+					(size 1.27 1.27)
+				)
+				(hide yes)
+			)
+		)
+		(property "Datasheet" "https://jlcpcb.com/partdetail/5885909-CL10B105KB8NQNC/C5199872"
+			(at 82.55 105.41 0)
+			(effects
+				(font
+					(size 1.27 1.27)
+				)
+				(hide yes)
+			)
+		)
+		(property "Description" ""
+			(at 82.55 105.41 0)
+			(effects
+				(font
+					(size 1.27 1.27)
+				)
+				(hide yes)
+			)
+		)
+		(property "LCSC" "C5199872"
+			(at 82.55 105.41 0)
+			(effects
+				(font
+					(size 1.27 1.27)
+				)
+				(hide yes)
+			)
+		)
+		(pin "1"
+		)
+		(pin "2"
+		)
+		(instances
+			(project "bornhack2026-hardware"
+				(path "/23bf5400-d19c-445b-8744-b63ebcca303d/1f4fc1c2-c6dd-4c37-a48b-5ed4d54351cc"
+					(reference "C72")
+					(unit 1)
+				)

Commit message: Checked PCBA for JLCPCB.
Parts:
- SW1: LCSC (none) -> C318884
- SW3: LCSC (none) -> C139794
Changed lines of the file:
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@@
+			)
+		)
+		(property "LCSC" "C318884"
+			(at 68.58 104.14 0)
+			(effects
+				(font
+					(size 1.27 1.27)
+				)
+				(hide yes)
 			)
 		)
@@
 			(effects
 				(font
+					(size 1.27 1.27)
+				)
+				(hide yes)
+			)
+		)
+		(property "LCSC" "C139794"
+			(at 208.28 82.55 0)
+			(effects
+				(font

Commit message: Replaced joystick with alternatie (cheaper) part.
Parts:
- removed SW3: SKRHABE010, lcsc:SW-SMD_SKRHABE010, symbol lcsc:SKRHABE010
- added SW4: 7*7*5-6P WX, lcsc:SW-SMD_6P-L7.0-W7.0-P1.40-LS7.4-TL, symbol lcsc:7*7*5-6PWX
Connections:
- net BTN_JOY_DOWN: now also SW4.4
- net BTN_JOY_FIRE: now also R22.2, SW4.5; no longer R23.2
- net BTN_JOY_LEFT: now also R23.2, SW4.3; no longer R28.2
- net BTN_JOY_RIGHT: now also R27.2, SW4.6; no longer R22.2
- net BTN_JOY_UP: now also R28.2, SW4.1; no longer R27.2
- net GND: now also SW4.2, SW4.7, SW4.8
Other:
- moved on the sheet: R18, R22, R23, R27, R28
