File: input.kicad_sch (KiCad schematic)
At the start: 9 parts, among them SW1 TS-1187A-B-A-B, SW4 7*7*5-6P WX

Commit message: Add Readme, fix labels in schematic.
Connections:
- net BTN_JOY_DOWN renamed P1.03_BTN_JOY_DOWN
- net BTN_JOY_FIRE renamed P1.02_BTN_JOY_FIRE
- net BTN_JOY_LEFT renamed P1.05_BTN_JOY_LEFT
- net BTN_JOY_RIGHT renamed P1.01_BTN_JOY_RIGHT
- net BTN_JOY_UP renamed P1.04_BTN_JOY_UP
Changed lines of the file:
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@@
 		)
 	)
-	(hierarchical_label "BTN_JOY_RIGHT"
+	(hierarchical_label "P1.01_BTN_JOY_RIGHT"
 		(shape output)
 		(at 233.68 99.06 0)
@@
 		)
 	)
-	(hierarchical_label "BTN_EXECUTE"
+	(hierarchical_label "P0.26_BTN_EXECUTE"
 		(shape output)
 		(at 99.06 62.23 0)
@@
 		)
 	)
-	(hierarchical_label "BTN_JOY_UP"
+	(hierarchical_label "P1.04_BTN_JOY_UP"
 		(shape output)
 		(at 148.59 99.06 180)
@@
 		)
 	)
-	(hierarchical_label "BTN_JOY_LEFT"
+	(hierarchical_label "P1.05_BTN_JOY_LEFT"
 		(shape output)
 		(at 148.59 109.22 180)
@@
 		)
 	)
-	(hierarchical_label "BTN_JOY_FIRE"
+	(hierarchical_label "P1.02_BTN_JOY_FIRE"
 		(shape output)
 		(at 233.68 104.14 0)
@@
 		)
 	)
-	(hierarchical_label "BTN_JOY_DOWN"
+	(hierarchical_label "P1.03_BTN_JOY_DOWN"
 		(shape output)
 		(at 233.68 109.22 0)

Commit message: Moved SWR connector to other side of board, reversed on/off switch UP -> ON.
Parts:
- SW1: value TS-1187A-B-A-B -> RESET
Changed lines of the file:
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@@
 			)
 		)
-		(property "Value" "TS-1187A-B-A-B"
+		(property "Value" "RESET"
 			(at 68.58 99.06 0)
 			(effects

Commit message: Fixed PCBA rotations in using component property.
Connections:
- net BTN_RESET renamed BTN_RESETn
Changed lines of the file:
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@@
 		)
 	)
-	(hierarchical_label "BTN_RESET"
+	(hierarchical_label "BTN_RESETn"
 		(shape output)
 		(at 99.06 101.6 0)

Commit message: Optimized design to use more basic components.
Parts:
- SW4: LCSC (none) -> C2858286; LCSC Part C2858286 -> (none)

Commit message: Add capacitors, add DC pin to epaper-display.
Parts:
- added C62, C63, C64, C69, C70: 100nF, Capacitor_SMD:C_0402_1005Metric, symbol symbols:C
Connections:
- net GND: now also C62.1, C63.1, C64.1, C69.1, C70.1
- net P1.01_BTN_JOY_RIGHT: now also C64.2
- net P1.02_BTN_JOY_FIRE: now also C63.2
- net P1.03_BTN_JOY_DOWN: now also C62.2
- net P1.04_BTN_JOY_UP: now also C70.2
- net P1.05_BTN_JOY_LEFT: now also C69.2

Commit message: Fixed schematic to have 0 DRC errors, changed display connector.
Parts:
- R15: value 10k -> 47k; LCSC C25744 -> C25792
Changed lines of the file:
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@@
 			)
 		)
-		(property "Value" "10k"
+		(property "Value" "47k"
 			(at 85.09 97.7899 0)
 			(effects
@@
 			)
 		)
-		(property "Datasheet" "https://jlcpcb.com/partdetail/26487-0402WGF1002TCE/C25744"
+		(property "Datasheet" "https://jlcpcb.com/partdetail/26535-0402WGF4702TCE/C25792"
 			(at 82.55 96.52 0)
 			(effects
@@
 			)
 		)
-		(property "LCSC" "C25744"
+		(property "LCSC" "C25792"
 			(at 82.55 96.52 0)
 			(effects

Commit message: Add MA logo, test points, tuned RF LoRa.
Parts:
- added TP11: TestPoint, TestPoint:TestPoint_Pad_1.0x1.0mm, symbol Connector:TestPoint
Connections:
- net BTN_RESETn: now also TP11.1
Changed lines of the file:
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@@
+	)
+	(junction
+		(at 95.25 101.6)
+		(diameter 0)
+		(color 0 0 0 0)
 	)
 	(junction
@@
 	(wire
 		(pts
-			(xy 82.55 101.6) (xy 99.06 101.6)
+			(xy 82.55 101.6) (xy 95.25 101.6)
 		)
 		(stroke
@@
 		(pts
 			(xy 170.18 104.14) (xy 175.26 104.14)
+		)
+		(stroke
+			(width 0)
+			(type default)
+		)
+	)
+	(wire
+		(pts
+			(xy 95.25 101.6) (xy 104.14 101.6)
 		)
 		(stroke
@@
 	(hierarchical_label "BTN_RESETn"
 		(shape output)
-		(at 99.06 101.6 0)
+		(at 104.14 101.6 0)
 		(effects
 			(font
@@
 		)
 	)
+	(symbol
+		(lib_id "Connector:TestPoint")
+		(at 95.25 101.6 0)
+		(unit 1)
+		(exclude_from_sim no)
+		(in_bom yes)
+		(on_board yes)
+		(dnp no)
+		(property "Reference" "TP11"
+			(at 97.79 97.0279 0)
+			(effects
+				(font
+					(size 1.27 1.27)
+				)
+				(justify left)
+			)
+		)
+		(property "Value" "TestPoint"
+			(at 97.79 99.5679 0)
+			(effects
+				(font
+					(size 1.27 1.27)
+				)
+				(justify left)
+				(hide yes)
+			)
+		)
+		(property "Footprint" "TestPoint:TestPoint_Pad_1.0x1.0mm"
+			(at 100.33 101.6 0)
+			(effects
+				(font
+					(size 1.27 1.27)
+				)
+				(hide yes)
+			)
+		)
+		(property "Datasheet" "~"
+			(at 100.33 101.6 0)
+			(effects
+				(font
+					(size 1.27 1.27)
+				)
+				(hide yes)
+			)
+		)
+		(property "Description" "test point"
+			(at 95.25 101.6 0)
+			(effects
+				(font
+					(size 1.27 1.27)
+				)
+				(hide yes)
+			)
+		)
+		(property "name" "RSTn"
+			(at 98.806 98.806 0)
+			(effects
+				(font
+					(size 1.27 1.27)
+				)
+			)
+		)
+		(pin "1"
+		)
+		(instances
+			(project "bornhack2026-hardware"
+				(path "/23bf5400-d19c-445b-8744-b63ebcca303d/1f4fc1c2-c6dd-4c37-a48b-5ed4d54351cc"
+					(reference "TP11")
+					(unit 1)
+				)
+			)
+		)
+	)
