File: input.kicad_sch (KiCad schematic)
At the start: 15 parts, among them SW1 RESET, SW4 7*7*5-6P WX

Commit message: dotting the i's , list checks before V2 order.
Parts:
- TP11: now not fitted; now left out of the parts list
Changed lines of the file:
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@@
 		(unit 1)
 		(exclude_from_sim no)
-		(in_bom yes)
+		(in_bom no)
 		(on_board yes)
-		(dnp no)
+		(dnp yes)
 		(property "Reference" "TP11"
 			(at 97.79 97.0279 0)

Commit message: Updated readme.md for Prototype V2. Simplified NRF IO net names.
Connections:
- net P1.01_BTN_JOY_RIGHT renamed JOY_RIGHT
- net P1.02_BTN_JOY_FIRE renamed JOY_FIRE
- net P1.03_BTN_JOY_DOWN renamed JOY_DOWN
- net P1.04_BTN_JOY_UP renamed JOY_UP
- net P1.05_BTN_JOY_LEFT renamed JOY_LEFT
Changed lines of the file:
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@@
 		)
 	)
-	(hierarchical_label "P1.01_BTN_JOY_RIGHT"
+	(hierarchical_label "JOY_RIGHT"
 		(shape output)
 		(at 233.68 99.06 0)
@@
 		)
 	)
-	(hierarchical_label "P0.26_BTN_EXECUTE"
+	(hierarchical_label "BTN_EXECUTE"
 		(shape output)
 		(at 99.06 62.23 0)
@@
 		)
 	)
-	(hierarchical_label "P1.04_BTN_JOY_UP"
+	(hierarchical_label "JOY_UP"
 		(shape output)
 		(at 148.59 99.06 180)
@@
 		)
 	)
-	(hierarchical_label "P1.05_BTN_JOY_LEFT"
+	(hierarchical_label "JOY_LEFT"
 		(shape output)
 		(at 148.59 109.22 180)
@@
 		)
 	)
-	(hierarchical_label "P1.02_BTN_JOY_FIRE"
+	(hierarchical_label "JOY_FIRE"
 		(shape output)
 		(at 233.68 104.14 0)
@@
 		)
 	)
-	(hierarchical_label "P1.03_BTN_JOY_DOWN"
+	(hierarchical_label "JOY_DOWN"
 		(shape output)
 		(at 233.68 109.22 0)
