File: display.kicad_sch (KiCad schematic)
At the start: 19 parts, among them J2 E-Paper, Q2 AP2302B

Commit message: PCB layout egg shape, for reference.
Parts:
- J2: footprint library:Hirose_FH12-24S-0.5SH_1x24-1MP_P0.50mm_Horizontal -> lcsc:FPC-SMD_FH12-24S-0.5SH-55
Changed lines of the file:
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@@
 			)
 		)
-		(property "Footprint" "library:Hirose_FH12-24S-0.5SH_1x24-1MP_P0.50mm_Horizontal"
+		(property "Footprint" "lcsc:FPC-SMD_FH12-24S-0.5SH-55"
 			(at 175.26 87.63 0)
 			(effects
@@
 			)
 		)
-		(property "Description" ""
+		(property "Description" "E-paper connector"
 			(at 175.26 87.63 0)
 			(effects

Commit message: Switched the LC filters from ceramic LoRa filter.
Parts:
- R12: LCSC C25741 -> C25530
Changed lines of the file:
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@@
 			)
 		)
-		(property "Datasheet" "https://www.lcsc.com/product-detail/Chip-Resistor-Surface-Mount_UNI-ROYAL-Uniroyal-Elec-0402WGF1003TCE_C25741.html"
+		(property "Datasheet" "https://jlcpcb.com/partdetail/26273-0402WGJ0104TCE/C25530"
 			(at 106.68 71.12 0)
 			(effects
@@
 			)
 		)
-		(property "LCSC" "C25741"
+		(property "LCSC" "C25530"
 			(at 106.68 71.12 0)
 			(effects
@@
 			)
 		)
-		(property "Datasheet" "https://datasheet.lcsc.com/lcsc/1912111437_ALLPOWER-ShenZhen-Quan-Li-Semiconductor-AP2302B_C406812.pdf"
+		(property "Datasheet" "https://jlcpcb.com/partdetail/395073-AP2302B/C406812"
 			(at 101.6 59.69 0)
 			(effects

Commit message: Progress, routed more stuff.
Parts:
- C32: value 4.7u -> 4.7uF
- C33, C34, C35, C36, C37, C38, C39, C40: value 1u -> 1uF
- D3, D4, D5: footprint library:D_SOD-323 -> Diode_SMD:D_SOD-323
- L9: value 47u -> 47uH; footprint library:L_1210_3225Metric -> Inductor_SMD:L_1210_3225Metric
- Q2: footprint library:SOT-23 -> lcsc:SOT-23-3_L2.9-W1.3-P1.90-LS2.4-BR
Changed lines of the file:
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@@
 			)
 		)
-		(property "Value" "1u"
+		(property "Value" "1uF"
 			(at 129.54 128.27 0)
 			(effects
@@
 			)
 		)
-		(property "Datasheet" "https://datasheet.lcsc.com/lcsc/2304140030_Samsung-Electro-Mechanics-CL05A105KQ5NNNC_C107372.pdf"
+		(property "Datasheet" "https://jlcpcb.com/partdetail/5885909-CL10B105KB8NQNC/C5199872"
 			(at 124.46 127 0)
 			(effects
@@
 			)
 		)
-		(property "Footprint" "library:D_SOD-323"
+		(property "Footprint" "Diode_SMD:D_SOD-323"
 			(at 100.33 107.95 0)
 			(effects
@@
 			)
 		)
-		(property "Value" "4.7u"
+		(property "Value" "4.7uF"
 			(at 76.708 72.136 0)
 			(effects
@@
 			)
 		)
-		(property "Value" "1u"
+		(property "Value" "1uF"
 			(at 156.21 128.27 0)
 			(effects
@@
 			)
 		)
-		(property "Datasheet" "https://datasheet.lcsc.com/lcsc/2304140030_Samsung-Electro-Mechanics-CL05A105KQ5NNNC_C107372.pdf"
+		(property "Datasheet" "https://jlcpcb.com/partdetail/5885909-CL10B105KB8NQNC/C5199872"
 			(at 151.13 127 0)
 			(effects
@@
 			)
 		)
-		(property "Footprint" "library:D_SOD-323"
+		(property "Footprint" "Diode_SMD:D_SOD-323"
 			(at 80.01 123.19 0)
 			(effects
@@
 			)
 		)
-		(property "Footprint" "library:SOT-23"
+		(property "Footprint" "lcsc:SOT-23-3_L2.9-W1.3-P1.90-LS2.4-BR"
 			(at 96.52 57.15 0)
 			(effects
@@
 			)
 		)
-		(property "Footprint" "library:D_SOD-323"
+		(property "Footprint" "Diode_SMD:D_SOD-323"
 			(at 87.63 123.19 0)
 			(effects
@@
 			)
 		)
-		(property "Value" "1u"
+		(property "Value" "1uF"
 			(at 147.32 128.27 0)
 			(effects
@@
 			)
 		)
-		(property "Datasheet" "https://datasheet.lcsc.com/lcsc/2304140030_Samsung-Electro-Mechanics-CL05A105KQ5NNNC_C107372.pdf"
+		(property "Datasheet" "https://jlcpcb.com/partdetail/5885909-CL10B105KB8NQNC/C5199872"
 			(at 142.24 127 0)
 			(effects
@@
 			)
 		)
-		(property "Value" "1u"
+		(property "Value" "1uF"
 			(at 111.76 128.27 0)
 			(effects
@@
 			)
 		)
-		(property "Datasheet" "https://datasheet.lcsc.com/lcsc/2304140030_Samsung-Electro-Mechanics-CL05A105KQ5NNNC_C107372.pdf"
+		(property "Datasheet" "https://jlcpcb.com/partdetail/5885909-CL10B105KB8NQNC/C5199872"
 			(at 106.68 127 0)
 			(effects
@@
 			)
 		)
-		(property "Value" "1u"
+		(property "Value" "1uF"
 			(at 138.43 128.27 0)
 			(effects
@@
 			)
 		)
-		(property "Datasheet" "https://datasheet.lcsc.com/lcsc/2304140030_Samsung-Electro-Mechanics-CL05A105KQ5NNNC_C107372.pdf"
+		(property "Datasheet" "https://jlcpcb.com/partdetail/5885909-CL10B105KB8NQNC/C5199872"
 			(at 133.35 127 0)
 			(effects
@@
 			)
 		)
-		(property "Value" "1u"
+		(property "Value" "1uF"
 			(at 85.09 134.62 0)
 			(effects
@@
 			)
 		)
-		(property "Datasheet" "https://datasheet.lcsc.com/lcsc/2304140030_Samsung-Electro-Mechanics-CL05A105KQ5NNNC_C107372.pdf"
+		(property "Datasheet" "https://jlcpcb.com/partdetail/5885909-CL10B105KB8NQNC/C5199872"
 			(at 83.82 129.54 0)
 			(effects
@@
 			)
 		)
-		(property "Value" "1u"
+		(property "Value" "1uF"
 			(at 88.9 115.57 0)
 			(effects
@@
 			)
 		)
-		(property "Datasheet" "https://datasheet.lcsc.com/lcsc/2304140030_Samsung-Electro-Mechanics-CL05A105KQ5NNNC_C107372.pdf"
+		(property "Datasheet" "https://jlcpcb.com/partdetail/5885909-CL10B105KB8NQNC/C5199872"
 			(at 83.82 114.3 0)
 			(effects
@@
 			)
 		)
-		(property "Value" "47u"
+		(property "Value" "47uH"
 			(at 100.33 49.53 0)
 			(effects
@@
 			)
 		)
-		(property "Footprint" "library:L_1210_3225Metric"
+		(property "Footprint" "Inductor_SMD:L_1210_3225Metric"
 			(at 99.06 48.26 0)
 			(effects
@@
 			)
 		)
-		(property "Value" "1u"
+		(property "Value" "1uF"
 			(at 120.65 128.27 0)
 			(effects
@@
 			)
 		)
-		(property "Datasheet" "https://datasheet.lcsc.com/lcsc/2304140030_Samsung-Electro-Mechanics-CL05A105KQ5NNNC_C107372.pdf"
+		(property "Datasheet" "https://jlcpcb.com/partdetail/5885909-CL10B105KB8NQNC/C5199872"
 			(at 115.57 127 0)
 			(effects

Commit message: Checked PCBA for JLCPCB.
Parts:
- C41: value 470n -> 470nF
Changed lines of the file:
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@@
 			)
 		)
-		(property "Value" "470n"
+		(property "Value" "470nF"
 			(at 162.56 128.27 0)
 			(effects

Commit message: Display
Parts:
- C36: now not fitted; now left out of the parts list
- J2: footprint lcsc:FPC-SMD_FH12-24S-0.5SH-55 -> symbols:FPC-SMD_XUNPU_FPC-0.5AS-24PWBH20; LCSC C202112 -> C3446073
Other:
- note added: "Pin numbering of connector is reversed compared to display datasheet"
- note removed: "TODO: Adjust the circuit for this badge design, this is copy pasted from Kami."
Changed lines of the file:
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@@
 		)
 	)
-	(text "TODO: Adjust the circuit for this badge design, this is copy pasted from Kami."
+	(text "Pin numbering of connector is reversed\ncompared to display datasheet"
 		(exclude_from_sim no)
-		(at 120.142 29.464 0)
+		(at 199.39 84.582 0)
 		(effects
 			(font
@@
 	(text "BS1"
 		(exclude_from_sim no)
-		(at 160.02 74.93 0)
+		(at 160.02 75.946 0)
 		(effects
 			(font
@@
 	(wire
 		(pts
-			(xy 135.89 102.87) (xy 138.43 100.33)
+			(xy 133.35 102.87) (xy 138.43 102.87)
 		)
 		(stroke
@@
 	(wire
 		(pts
+			(xy 138.43 100.33) (xy 138.43 102.87)
+		)
+		(stroke
+			(width 0)
+			(type default)
+		)
+	)
+	(wire
+		(pts
 			(xy 87.63 118.11) (xy 87.63 119.38)
 		)
@@
 	(wire
 		(pts
-			(xy 133.35 102.87) (xy 135.89 102.87)
-		)
-		(stroke
-			(width 0)
-			(type default)
-		)
-	)
-	(wire
-		(pts
 			(xy 87.63 129.54) (xy 99.06 129.54)
 		)
@@
 			)
 		)
-		(property "Footprint" "lcsc:FPC-SMD_FH12-24S-0.5SH-55"
+		(property "Footprint" "symbols:FPC-SMD_XUNPU_FPC-0.5AS-24PWBH20"
 			(at 175.26 87.63 0)
 			(effects
@@
 			)
 		)
-		(property "Datasheet" "https://datasheet.lcsc.com/lcsc/2304140030_HRS-Hirose-FH12-24S-0-5SH-55_C202112.pdf"
+		(property "Datasheet" "https://www.lcsc.com/product-detail/C3446073.html"
 			(at 175.26 87.63 0)
 			(effects
@@
 			)
 		)
-		(property "LCSC" "C202112"
+		(property "LCSC" "C3446073"
 			(at 175.26 87.63 0)
 			(effects
@@
 		(unit 1)
 		(exclude_from_sim no)
-		(in_bom yes)
+		(in_bom no)
 		(on_board yes)
-		(dnp no)
+		(dnp yes)
 		(property "Reference" "C36"
 			(at 121.92 125.73 0)

Commit message: Fixed PCBA rotations in using component property.
Parts:
- removed J2: E-Paper, symbols:FPC-SMD_XUNPU_FPC-0.5AS-24PWBH20, symbol symbols:Conn_01x24_MountingPin
- added FPC1: 0.5-24P CTSJ-H2.0 119, lcsc:FPC-SMD_24P-P0.50_SHOU-HAN_CTSJ-H2.0, symbol lcsc:0.5-24PCTSJ-H2.0119
- Q2: FT Rotation Offset (none) -> 180
Connections:
- net 3V3: now also FPC1.10, FPC1.9
- net BUSY: now also FPC1.16
- net CS: now also FPC1.13
- net DC: now also FPC1.14
- net GDR: now also FPC1.23
- net GND: now also FPC1.17, FPC1.25, FPC1.26, FPC1.8
- net MOSI: now also FPC1.11
- net PREVGH: now also FPC1.4
- net PREVGL: now also FPC1.2
- net RESE: now also FPC1.22
- net SCK: now also FPC1.12
- net VCOM: now also FPC1.1
- net VGH: now also FPC1.20
- net VGL: now also FPC1.21
- net VSH: now also FPC1.5
- net VSL: now also FPC1.3
- net at C38.2, R13.2: now also FPC1.7
- new net RESETn: FPC1.15
Changed lines of the file:
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@@
 	(text "Pin numbering of connector is reversed\ncompared to display datasheet"
 		(exclude_from_sim no)
-		(at 199.39 84.582 0)
+		(at 200.66 84.582 0)
 		(effects
 			(font
@@
 	(wire
 		(pts
+			(xy 179.07 48.26) (xy 181.61 48.26)
+		)
+		(stroke
+			(width 0)
+			(type default)
+		)
+	)
+	(wire
+		(pts
 			(xy 133.35 95.25) (xy 170.18 95.25)
 		)
@@
 	(wire
 		(pts
-			(xy 175.26 51.435) (xy 175.895 51.435)
-		)
-		(stroke
-			(width 0)
-			(type default)
-		)
-	)
-	(wire
-		(pts
 			(xy 99.06 53.34) (xy 99.06 54.61)
 		)
@@
 	(wire
 		(pts
+			(xy 179.07 48.26) (xy 179.07 52.07)
+		)
+		(stroke
+			(width 0)
+			(type default)
+		)
+	)
+	(wire
+		(pts
 			(xy 99.06 52.07) (xy 99.06 53.34)
 		)
@@
 	(wire
 		(pts
-			(xy 175.26 51.435) (xy 175.26 52.07)
+			(xy 179.07 123.825) (xy 181.61 123.825)
 		)
 		(stroke
@@
 		(pts
 			(xy 167.64 97.79) (xy 170.18 97.79)
+		)
+		(stroke
+			(width 0)
+			(type default)
+		)
+	)
+	(wire
+		(pts
+			(xy 179.07 123.825) (xy 179.07 120.65)
 		)
 		(stroke
@@
 		)
 	)
-	(hierarchical_label "RESET"
+	(hierarchical_label "RESETn"
 		(shape bidirectional)
 		(at 165.1 80.01 180)
@@
 	)
 	(symbol
-		(lib_id "symbols:Conn_01x24_MountingPin")
-		(at 175.26 87.63 0)
-		(mirror x)
-		(unit 1)
-		(exclude_from_sim no)
-		(in_bom yes)
-		(on_board yes)
-		(dnp no)
-		(property "Reference" "J2"
-			(at 175.26 121.92 0)
-			(effects
-				(font
-					(size 1.27 1.27)
-				)
-			)
-		)
-		(property "Value" "E-Paper"
-			(at 175.26 119.38 0)
-			(effects
-				(font
-					(size 1.27 1.27)
-				)
-			)
-		)
-		(property "Footprint" "symbols:FPC-SMD_XUNPU_FPC-0.5AS-24PWBH20"
-			(at 175.26 87.63 0)
-			(effects
-				(font
-					(size 1.27 1.27)
-				)
-				(hide yes)
-			)
-		)
-		(property "Datasheet" "https://www.lcsc.com/product-detail/C3446073.html"
-			(at 175.26 87.63 0)
-			(effects
-				(font
-					(size 1.27 1.27)
-				)
-				(hide yes)
-			)
-		)
-		(property "Description" "E-paper connector"
-			(at 175.26 87.63 0)
-			(effects
-				(font
-					(size 1.27 1.27)
-				)
-				(hide yes)
-			)
-		)
-		(property "LCSC" "C3446073"
-			(at 175.26 87.63 0)
-			(effects
-				(font
-					(size 1.27 1.27)
-				)
-				(hide yes)
-			)
-		)
-		(property "Resource" ""
-			(at 175.26 87.63 0)
-			(effects
-				(font
-					(size 1.27 1.27)
-				)
-				(hide yes)
-			)
-		)
-		(pin "1"
-		)
-		(pin "10"
-		)
-		(pin "11"
-		)
-		(pin "12"
-		)
-		(pin "13"
-		)
-		(pin "14"
-		)
-		(pin "15"
-		)
-		(pin "16"
-		)
-		(pin "17"
-		)
-		(pin "18"
-		)
-		(pin "19"
-		)
-		(pin "2"
-		)
-		(pin "20"
-		)
-		(pin "21"
-		)
-		(pin "22"
-		)
-		(pin "23"
-		)
-		(pin "24"
-		)
-		(pin "3"
-		)
-		(pin "4"
-		)
-		(pin "5"
-		)
-		(pin "6"
-		)
-		(pin "7"
-		)
-		(pin "8"
-		)
-		(pin "9"
-		)
-		(pin "MP"
-		)
-		(instances
-			(project "bornhack2026-hardware"
-				(path "/23bf5400-d19c-445b-8744-b63ebcca303d/9cdecd3d-2b1f-4dfc-b0b2-cc7367cb6c39"
-					(reference "J2")
-					(unit 1)
-				)
-			)
-		)
-	)
-	(symbol
 		(lib_id "symbols:C")
 		(at 124.46 127 180)
@@
 				(path "/23bf5400-d19c-445b-8744-b63ebcca303d/9cdecd3d-2b1f-4dfc-b0b2-cc7367cb6c39"
 					(reference "C37")
+					(unit 1)
+				)
+			)
+		)
+	)
+	(symbol
+		(lib_id "symbols2:GND")
+		(at 181.61 123.825 90)
+		(mirror x)
+		(unit 1)
+		(exclude_from_sim no)
+		(in_bom yes)
+		(on_board yes)
+		(dnp no)
+		(property "Reference" "#PWR077"
+			(at 187.96 123.825 0)
+			(effects
+				(font
+					(size 1.27 1.27)
+				)
+				(hide yes)
+			)
+		)
+		(property "Value" "GND"
+			(at 186.0042 123.952 0)
+			(effects
+				(font
+					(size 1.27 1.27)
+				)
+			)
+		)
+		(property "Footprint" ""
+			(at 181.61 123.825 0)
+			(effects
+				(font
+					(size 1.27 1.27)
+				)
+				(hide yes)
+			)
+		)
+		(property "Datasheet" ""
+			(at 181.61 123.825 0)
+			(effects
+				(font
+					(size 1.27 1.27)
+				)
+				(hide yes)
+			)
+		)
+		(property "Description" "Power symbol creates a global label with name \"GND\" , ground"
+			(at 181.61 123.825 0)
+			(effects
+				(font
+					(size 1.27 1.27)
+				)
+				(hide yes)
+			)
+		)
+		(pin "1"
+		)
+		(instances
+			(project "bornhack2026-hardware"
+				(path "/23bf5400-d19c-445b-8744-b63ebcca303d/9cdecd3d-2b1f-4dfc-b0b2-cc7367cb6c39"
+					(reference "#PWR077")
 					(unit 1)
 				)
@@
 	)
 	(symbol
+		(lib_id "lcsc:0.5-24PCTSJ-H2.0119")
+		(at 175.26 86.36 0)
+		(mirror x)
+		(unit 1)
+		(exclude_from_sim no)
+		(in_bom yes)
+		(on_board yes)
+		(dnp no)
+		(property "Reference" "FPC1"
+			(at 181.61 87.6301 0)
+			(effects
+				(font
+					(size 1.27 1.27)
+				)
+				(justify left)
+			)
+		)
+		(property "Value" "0.5-24P CTSJ-H2.0 119"
+			(at 181.61 85.0901 0)
+			(effects
+				(font
+					(size 1.27 1.27)
+				)
+				(justify left)
+			)
+		)
+		(property "Footprint" "lcsc:FPC-SMD_24P-P0.50_SHOU-HAN_CTSJ-H2.0"
+			(at 175.26 44.45 0)
+			(effects
+				(font
+					(size 1.27 1.27)
+				)
+				(hide yes)
+			)
+		)
+		(property "Datasheet" "https://jlcpcb.com/partdetail/SHOUHAN-0_5_24P_CTSJ_H2_0119/C2858299"
+			(at 175.26 86.36 0)
+			(effects
+				(font
+					(size 1.27 1.27)
+				)
+				(hide yes)
+			)
+		)
+		(property "Description" "-25℃~+85℃ 0.3mm 0.5mm 24P 2mm 50V Phosphor Bronze Slide Lock Surface Mount, Right Angle Tin Top Contact SMD,P=0.5mm,Surface Mount，Right Angle FFC, FPC (Flat Flexible) Connector Assemblies ROHS"
+			(at 175.26 86.36 0)
+			(effects
+				(font
+					(size 1.27 1.27)
+				)
+				(hide yes)
+			)
+		)
+		(property "LCSC Part" "C2858299"
+			(at 175.26 41.91 0)
+			(effects
+				(font
+					(size 1.27 1.27)
+				)
+				(hide yes)
+			)
+		)
+		(pin "9"
+		)
+		(pin "12"
+		)
+		(pin "18"
+		)
+		(pin "26"
+		)
+		(pin "15"
+		)
+		(pin "24"
+		)
+		(pin "5"
+		)
+		(pin "4"
+		)
+		(pin "1"
+		)
+		(pin "25"
+		)
+		(pin "8"
+		)
+		(pin "10"
+		)
+		(pin "13"
+		)
+		(pin "16"
+		)
+		(pin "11"
+		)
+		(pin "22"
+		)
+		(pin "21"
+		)
+		(pin "14"
+		)
+		(pin "3"
+		)
+		(pin "2"
+		)
+		(pin "20"
+		)
+		(pin "17"
+		)
+		(pin "6"
+		)
+		(pin "7"
+		)
+		(pin "19"
+		)
+		(pin "23"
+		)
+		(instances
+			(project ""
+				(path "/23bf5400-d19c-445b-8744-b63ebcca303d/9cdecd3d-2b1f-4dfc-b0b2-cc7367cb6c39"
+					(reference "FPC1")
+					(unit 1)
+				)
+			)
+		)
+	)
+	(symbol
 		(lib_id "symbols:D_Schottky")
 		(at 80.01 123.19 270)
@@
 			)
 		)
+		(property "FT Rotation Offset" "180"
+			(at 101.6 59.69 0)
+			(effects
+				(font
+					(size 1.27 1.27)
+				)
+				(hide yes)
+			)
+		)
 		(pin "1"
 		)
@@
 	(symbol
 		(lib_id "symbols2:GND")
-		(at 175.895 51.435 90)
+		(at 181.61 48.26 90)
 		(unit 1)
 		(exclude_from_sim no)
@@
 		(dnp no)
 		(property "Reference" "#PWR064"
-			(at 182.245 51.435 0)
+			(at 187.96 48.26 0)
 			(effects
 				(font
@@
 		)
 		(property "Value" "GND"
-			(at 180.2892 51.308 0)
+			(at 186.0042 48.133 0)
 			(effects
 				(font
@@
 		)
 		(property "Footprint" ""
-			(at 175.895 51.435 0)
+			(at 181.61 48.26 0)
 			(effects
 				(font
@@
 		)
 		(property "Datasheet" ""
-			(at 175.895 51.435 0)
+			(at 181.61 48.26 0)
 			(effects
 				(font
@@
 		)
 		(property "Description" "Power symbol creates a global label with name \"GND\" , ground"
-			(at 175.895 51.435 0)
-			(effects
-				(font
+			(at 181.61 48.26 0)
+			(effects
+				(font
