File: display.kicad_sch (KiCad schematic)
At the start: 19 parts, among them Q2 AP2302B

Commit message: Optimized design to use more basic components.
Parts:
- C36: LCSC C5199872 -> C15849
- FPC1: LCSC (none) -> C2858299
- R12: LCSC C25530 -> C25741

Commit message: Replaced schottky diode with 1A version, fixed joystick footprint.
Parts:
- removed D3, D4, D5: NSR0320MW2T1G, Diode_SMD:D_SOD-323, symbol symbols:D_Schottky
- added D3, D5, D8: 1N5819WS, Diode_SMD:D_SOD-323, symbol Diode:1N5819WS
Connections:
- net GND: now also D5.1 (K)
- net PREVGH: now also D8.1 (K)
- net PREVGL: now also D3.2 (A)
- net at C33.2, L9.2, Q2.3 (D): now also D8.2 (A)
- net at C33.1: now also D3.1 (K), D5.2 (A)

Commit message: Diodes in spec now for the display driver.
Parts:
- D3, D5, D8: value 1N5819WS -> B0530WS; LCSC C191023 -> C22466873
Other:
- note added: "Diode requirements Vrev > 30V Io > 500mA Vfw < 430mV"
- note added: "Schematic Page 12 https://cdn-learn.adafruit.com/assets/assets/000/097/631/original/SSD1680_Datasheet.pdf?1607625960"

Commit message: Add ESD protoction to USB-C, small fixes
Changed lines of the file:
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@@
 	(text "Pin numbering of connector is reversed\ncompared to display datasheet"
 		(exclude_from_sim no)
-		(at 200.66 84.582 0)
+		(at 201.93 78.74 0)
 		(effects
 			(font

Commit message: Switched to recycled e-ink screen, using the Tanoshii measuremens and distances.
Parts:
- removed FPC1: 0.5-24P CTSJ-H2.0 119, lcsc:FPC-SMD_24P-P0.50_SHOU-HAN_CTSJ-H2.0, symbol lcsc:0.5-24PCTSJ-H2.0119
- added J6: E-Paper, Connector_FFC-FPC:Hirose_FH12-24S-0.5SH_1x24-1MP_P0.50mm_Horizontal, symbol symbols:Conn_01x24_MountingPin
Connections:
- net 3V3: now also J6.10 (Pin_10), J6.9 (Pin_9)
- net BUSY: now also J6.16 (Pin_16)
- net CS: now also J6.13 (Pin_13)
- net DC: now also J6.14 (Pin_14)
- net GDR: now also J6.23 (Pin_23)
- net GND: now also J6.17 (Pin_17), J6.8 (Pin_8), J6.MP (MountPin)
- net MOSI: now also J6.11 (Pin_11)
- net PREVGH: now also J6.4 (Pin_4)
- net PREVGL: now also J6.2 (Pin_2)
- net RESE: now also J6.22 (Pin_22)
- net RESETn: now also J6.15 (Pin_15)
- net SCK: now also J6.12 (Pin_12)
- net VCOM: now also J6.1 (Pin_1)
- net VGH: now also J6.20 (Pin_20)
- net VGL: now also J6.21 (Pin_21)
- net VSH: now also J6.5 (Pin_5)
- net VSL: now also J6.3 (Pin_3)
- net at C38.2, R13.2: now also J6.7 (Pin_7)

Commit message: Changed out RF switch and display connector for parts that are stil available.
Parts:
- removed J6: E-Paper, Connector_FFC-FPC:Hirose_FH12-24S-0.5SH_1x24-1MP_P0.50mm_Horizontal, symbol symbols:Conn_01x24_MountingPin
- added CN1: TF31-24S-0.5SH(800), lcsc:FPC-SMD_24P-P0.50_TF31-24S-0.5SH, symbol lcsc:TF31-24S-0.5SH(800)
Connections:
- net 3V3: now also CN1.10, CN1.9
- net BUSY: now also CN1.16
- net CS: now also CN1.13
- net DC: now also CN1.14
- net GDR: now also CN1.23
- net GND: now also CN1.17, CN1.25, CN1.26, CN1.8
- net MOSI: now also CN1.11
- net PREVGH: now also CN1.4
- net PREVGL: now also CN1.2
- net RESE: now also CN1.22
- net RESETn: now also CN1.15
- net SCK: now also CN1.12
- net VCOM: now also CN1.1
- net VGH: now also CN1.20
- net VGL: now also CN1.21
- net VSH: now also CN1.5
- net VSL: now also CN1.3
- net at C38.2, R13.2: now also CN1.7
Changed lines of the file:
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@@
 	(wire
 		(pts
-			(xy 175.26 48.26) (xy 177.8 48.26)
+			(xy 181.61 48.26) (xy 184.15 48.26)
 		)
 		(stroke
@@
 	(wire
 		(pts
-			(xy 175.26 48.26) (xy 175.26 52.07)
+			(xy 181.61 48.26) (xy 181.61 52.07)
 		)
 		(stroke
@@
 	(wire
 		(pts
+			(xy 181.61 124.46) (xy 184.15 124.46)
+		)
+		(stroke
+			(width 0)
+			(type default)
+		)
+	)
+	(wire
+		(pts
 			(xy 165.1 80.01) (xy 170.18 80.01)
 		)
@@
 	(wire
 		(pts
+			(xy 181.61 124.46) (xy 181.61 120.65)
+		)
+		(stroke
+			(width 0)
+			(type default)
+		)
+	)
+	(wire
+		(pts
 			(xy 167.64 97.79) (xy 170.18 97.79)
 		)
@@
 	)
 	(symbol
-		(lib_id "symbols:Conn_01x24_MountingPin")
-		(at 175.26 87.63 0)
-		(mirror x)
-		(unit 1)
-		(exclude_from_sim no)
-		(in_bom yes)
-		(on_board yes)
-		(dnp no)
-		(property "Reference" "J6"
-			(at 175.26 121.92 0)
-			(effects
-				(font
-					(size 1.27 1.27)
-				)
-			)
-		)
-		(property "Value" "E-Paper"
-			(at 175.26 119.38 0)
-			(effects
-				(font
-					(size 1.27 1.27)
-				)
-			)
-		)
-		(property "Footprint" "Connector_FFC-FPC:Hirose_FH12-24S-0.5SH_1x24-1MP_P0.50mm_Horizontal"
-			(at 175.26 87.63 0)
-			(effects
-				(font
-					(size 1.27 1.27)
-				)
-				(hide yes)
-			)
-		)
-		(property "Datasheet" "https://datasheet.lcsc.com/lcsc/2304140030_HRS-Hirose-FH12-24S-0-5SH-55_C202112.pdf"
-			(at 175.26 87.63 0)
-			(effects
-				(font
-					(size 1.27 1.27)
-				)
-				(hide yes)
-			)
-		)
-		(property "Description" ""
-			(at 175.26 87.63 0)
-			(effects
-				(font
-					(size 1.27 1.27)
-				)
-				(hide yes)
-			)
-		)
-		(property "LCSC" "C202112"
-			(at 175.26 87.63 0)
-			(effects
-				(font
-					(size 1.27 1.27)
-				)
-				(hide yes)
-			)
-		)
-		(pin "1"
-		)
-		(pin "10"
-		)
-		(pin "11"
-		)
-		(pin "12"
-		)
-		(pin "13"
-		)
-		(pin "14"
-		)
-		(pin "15"
-		)
-		(pin "16"
-		)
-		(pin "17"
-		)
-		(pin "18"
-		)
-		(pin "19"
-		)
-		(pin "2"
-		)
-		(pin "20"
-		)
-		(pin "21"
-		)
-		(pin "22"
-		)
-		(pin "23"
-		)
-		(pin "24"
-		)
-		(pin "3"
-		)
-		(pin "4"
-		)
-		(pin "5"
-		)
-		(pin "6"
-		)
-		(pin "7"
-		)
-		(pin "8"
-		)
-		(pin "9"
-		)
-		(pin "MP"
-		)
-		(instances
-			(project "bornhack2026-hardware"
-				(path "/23bf5400-d19c-445b-8744-b63ebcca303d/9cdecd3d-2b1f-4dfc-b0b2-cc7367cb6c39"
-					(reference "J6")
-					(unit 1)
-				)
-			)
-		)
-	)
-	(symbol
 		(lib_id "symbols:C")
 		(at 124.46 127 180)
@@
 	)
 	(symbol
+		(lib_id "symbols2:GND")
+		(at 184.15 124.46 90)
+		(mirror x)
+		(unit 1)
+		(exclude_from_sim no)
+		(in_bom yes)
+		(on_board yes)
+		(dnp no)
+		(property "Reference" "#PWR02"
+			(at 190.5 124.46 0)
+			(effects
+				(font
+					(size 1.27 1.27)
+				)
+				(hide yes)
+			)
+		)
+		(property "Value" "GND"
+			(at 188.5442 124.587 0)
+			(effects
+				(font
+					(size 1.27 1.27)
+				)
+			)
+		)
+		(property "Footprint" ""
+			(at 184.15 124.46 0)
+			(effects
+				(font
+					(size 1.27 1.27)
+				)
+				(hide yes)
+			)
+		)
+		(property "Datasheet" ""
+			(at 184.15 124.46 0)
+			(effects
+				(font
+					(size 1.27 1.27)
+				)
+				(hide yes)
+			)
+		)
+		(property "Description" "Power symbol creates a global label with name \"GND\" , ground"
+			(at 184.15 124.46 0)
+			(effects
+				(font
+					(size 1.27 1.27)
+				)
+				(hide yes)
+			)
+		)
+		(pin "1"
+		)
+		(instances
+			(project "bornhack2026-hardware"
+				(path "/23bf5400-d19c-445b-8744-b63ebcca303d/9cdecd3d-2b1f-4dfc-b0b2-cc7367cb6c39"
+					(reference "#PWR02")
+					(unit 1)
+				)
+			)
+		)
+	)
+	(symbol
 		(lib_id "Diode:1N5819WS")
 		(at 80.01 123.19 90)
@@
 	(symbol
 		(lib_id "symbols2:GND")
-		(at 177.8 48.26 90)
+		(at 184.15 48.26 90)
 		(unit 1)
 		(exclude_from_sim no)
@@
 		(dnp no)
 		(property "Reference" "#PWR064"
-			(at 184.15 48.26 0)
+			(at 190.5 48.26 0)
 			(effects
 				(font
@@
 		)
 		(property "Value" "GND"
-			(at 182.1942 48.133 0)
+			(at 188.5442 48.133 0)
 			(effects
 				(font
@@
 		)
 		(property "Footprint" ""
-			(at 177.8 48.26 0)
+			(at 184.15 48.26 0)
 			(effects
 				(font
@@
 		)
 		(property "Datasheet" ""
-			(at 177.8 48.26 0)
+			(at 184.15 48.26 0)
 			(effects
 				(font
@@
 		)
 		(property "Description" "Power symbol creates a global label with name \"GND\" , ground"
-			(at 177.8 48.26 0)
+			(at 184.15 48.26 0)
 			(effects
 				(font
@@
 					(unit 1)
 				)
+			)
+		)
+	)
+	(symbol
+		(lib_id "lcsc:TF31-24S-0.5SH(800)")
+		(at 175.26 86.36 0)
+		(mirror x)
+		(unit 1)
+		(exclude_from_sim no)
+		(in_bom yes)
+		(on_board yes)
+		(dnp no)
+		(property "Reference" "CN1"
+			(at 184.15 87.6301 0)
+			(effects
+				(font
+					(size 1.27 1.27)
+				)
+				(justify left)
+			)
+		)
+		(property "Value" "TF31-24S-0.5SH(800)"
+			(at 184.15 85.0901 0)
+			(effects
+				(font
+					(size 1.27 1.27)
+				)
+				(justify left)
+			)
+		)
+		(property "Footprint" "lcsc:FPC-SMD_24P-P0.50_TF31-24S-0.5SH"
+			(at 175.26 44.45 0)
+			(effects
+				(font
+					(size 1.27 1.27)
+				)
+				(hide yes)
+			)
+		)
+		(property "Datasheet" ""
+			(at 175.26 86.36 0)
+			(effects
+				(font
+					(size 1.27 1.27)
+				)
+				(hide yes)
+			)
+		)
+		(property "Description" ""
+			(at 175.26 86.36 0)
+			(effects
+				(font
+					(size 1.27 1.27)
+				)
+				(hide yes)
+			)
+		)
+		(property "LCSC Part" "C3169854"
+			(at 175.26 41.91 0)
+			(effects
+				(font
+					(size 1.27 1.27)
+				)
+				(hide yes)
+			)
+		)
+		(pin "19"
+		)
+		(pin "4"
+		)
+		(pin "21"
+		)
+		(pin "18"
+		)
+		(pin "9"
+		)
+		(pin "26"
+		)
+		(pin "25"
+		)
+		(pin "13"
+		)
+		(pin "23"
+		)
+		(pin "5"
+		)
+		(pin "14"
+		)
+		(pin "20"
+		)
+		(pin "2"
+		)
+		(pin "1"
+		)
+		(pin "22"
+		)
+		(pin "12"
+		)
+		(pin "15"
+		)
+		(pin "24"
+		)
+		(pin "17"
+		)
+		(pin "6"
+		)
+		(pin "10"
+		)
+		(pin "7"
+		)
+		(pin "11"
+		)
+		(pin "8"
+		)
+		(pin "3"
+		)
+		(pin "16"
+		)
+		(instances
+			(project ""
+				(path "/23bf5400-d19c-445b-8744-b63ebcca303d/9cdecd3d-2b1f-4dfc-b0b2-cc7367cb6c39"
+					(reference "CN1")
+					(unit 1)
+				)

Commit message: Fixed schematic to have 0 DRC errors, changed display connector.
Parts:
- removed CN1: TF31-24S-0.5SH(800), lcsc:FPC-SMD_24P-P0.50_TF31-24S-0.5SH, symbol lcsc:TF31-24S-0.5SH(800)
- added FPC1: GT-F0501SR10-24S1101, lcsc:FPC-SMD_24P-P0.50_GT-F0501SR10-24S1101, symbol lcsc:GT-F0501SR10-24S1101
Connections:
- net 3V3: now also FPC1.10, FPC1.9
- net BUSY: now also FPC1.16
- net CS: now also FPC1.13
- net DC: now also FPC1.14
- net GDR: now also FPC1.23
- net GND: now also FPC1.17, FPC1.25, FPC1.26, FPC1.8
- net MOSI: now also FPC1.11
- net PREVGH: now also FPC1.4
- net PREVGL: now also FPC1.2
- net RESE: now also FPC1.22
- net RESETn: now also FPC1.15
- net SCK: now also FPC1.12
- net VCOM: now also FPC1.1
- net VGH: now also FPC1.20
- net VGL: now also FPC1.21
- net VSH: now also FPC1.5
- net VSL: now also FPC1.3
- net at C38.2, R13.2: now also FPC1.7
Changed lines of the file:
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@@
 	(wire
 		(pts
-			(xy 181.61 48.26) (xy 184.15 48.26)
+			(xy 179.07 48.26) (xy 181.61 48.26)
 		)
 		(stroke
@@
 	(wire
 		(pts
-			(xy 181.61 48.26) (xy 181.61 52.07)
+			(xy 179.07 48.26) (xy 179.07 52.07)
 		)
 		(stroke
@@
 	(wire
 		(pts
-			(xy 181.61 124.46) (xy 184.15 124.46)
+			(xy 179.07 124.46) (xy 181.61 124.46)
 		)
 		(stroke
@@
 	(wire
 		(pts
-			(xy 181.61 124.46) (xy 181.61 120.65)
+			(xy 179.07 124.46) (xy 179.07 120.65)
 		)
 		(stroke
@@
 	(symbol
 		(lib_id "symbols2:GND")
-		(at 184.15 124.46 90)
+		(at 181.61 124.46 90)
 		(mirror x)
 		(unit 1)
@@
 		(dnp no)
 		(property "Reference" "#PWR02"
-			(at 190.5 124.46 0)
+			(at 187.96 124.46 0)
 			(effects
 				(font
@@
 		)
 		(property "Value" "GND"
-			(at 188.5442 124.587 0)
+			(at 186.0042 124.587 0)
 			(effects
 				(font
@@
 		)
 		(property "Footprint" ""
-			(at 184.15 124.46 0)
+			(at 181.61 124.46 0)
 			(effects
 				(font
@@
 		)
 		(property "Datasheet" ""
-			(at 184.15 124.46 0)
+			(at 181.61 124.46 0)
 			(effects
 				(font
@@
 		)
 		(property "Description" "Power symbol creates a global label with name \"GND\" , ground"
-			(at 184.15 124.46 0)
+			(at 181.61 124.46 0)
 			(effects
 				(font
@@
 	(symbol
 		(lib_id "symbols2:GND")
-		(at 184.15 48.26 90)
+		(at 181.61 48.26 90)
 		(unit 1)
 		(exclude_from_sim no)
@@
 		(dnp no)
 		(property "Reference" "#PWR064"
-			(at 190.5 48.26 0)
+			(at 187.96 48.26 0)
 			(effects
 				(font
@@
 		)
 		(property "Value" "GND"
-			(at 188.5442 48.133 0)
+			(at 186.0042 48.133 0)
 			(effects
 				(font
@@
 		)
 		(property "Footprint" ""
-			(at 184.15 48.26 0)
+			(at 181.61 48.26 0)
 			(effects
 				(font
@@
 		)
 		(property "Datasheet" ""
-			(at 184.15 48.26 0)
+			(at 181.61 48.26 0)
 			(effects
 				(font
@@
 		)
 		(property "Description" "Power symbol creates a global label with name \"GND\" , ground"
-			(at 184.15 48.26 0)
+			(at 181.61 48.26 0)
 			(effects
 				(font
@@
 	)
 	(symbol
+		(lib_id "lcsc:GT-F0501SR10-24S1101")
+		(at 175.26 86.36 0)
+		(mirror x)
+		(unit 1)
+		(exclude_from_sim no)
+		(in_bom yes)
+		(on_board yes)
+		(dnp no)
+		(property "Reference" "FPC1"
+			(at 182.88 87.6301 0)
+			(effects
+				(font
+					(size 1.27 1.27)
+				)
+				(justify left)
+			)
+		)
+		(property "Value" "GT-F0501SR10-24S1101"
+			(at 182.88 85.0901 0)
+			(effects
+				(font
+					(size 1.27 1.27)
+				)
+				(justify left)
+			)
+		)
+		(property "Footprint" "lcsc:FPC-SMD_24P-P0.50_GT-F0501SR10-24S1101"
+			(at 175.26 44.45 0)
+			(effects
+				(font
+					(size 1.27 1.27)
+				)
+				(hide yes)
+			)
+		)
+		(property "Datasheet" ""
+			(at 175.26 86.36 0)
+			(effects
+				(font
+					(size 1.27 1.27)
+				)
+				(hide yes)
+			)
+		)
+		(property "Description" ""
+			(at 175.26 86.36 0)
+			(effects
+				(font
+					(size 1.27 1.27)
+				)
+				(hide yes)
+			)
+		)
+		(property "LCSC Part" "C22380687"
+			(at 175.26 41.91 0)
+			(effects
+				(font
+					(size 1.27 1.27)
+				)
+				(hide yes)
+			)
+		)
+		(pin "9"
+		)
+		(pin "12"
+		)
+		(pin "19"
+		)
+		(pin "22"
+		)
+		(pin "17"
+		)
+		(pin "4"
+		)
+		(pin "2"
+		)
+		(pin "14"
+		)
+		(pin "18"
+		)
+		(pin "21"
+		)
+		(pin "1"
+		)
+		(pin "3"
+		)
+		(pin "15"
+		)
+		(pin "8"
+		)
+		(pin "7"
+		)
+		(pin "24"
+		)
+		(pin "5"
+		)
+		(pin "25"
+		)
+		(pin "6"
+		)
+		(pin "13"
+		)
+		(pin "26"
+		)
+		(pin "11"
+		)
+		(pin "10"
+		)
+		(pin "23"
+		)
+		(pin "16"
+		)
+		(pin "20"
+		)
+		(instances
+			(project ""
+				(path "/23bf5400-d19c-445b-8744-b63ebcca303d/9cdecd3d-2b1f-4dfc-b0b2-cc7367cb6c39"
+					(reference "FPC1")
+					(unit 1)
+				)
+			)
+		)
+	)
+	(symbol
 		(lib_id "symbols:R")
 		(at 99.06 71.12 180)
@@
 					(unit 1)
 				)
-			)
-		)
-	)
-	(symbol
-		(lib_id "lcsc:TF31-24S-0.5SH(800)")
-		(at 175.26 86.36 0)
-		(mirror x)
-		(unit 1)
-		(exclude_from_sim no)
-		(in_bom yes)
-		(on_board yes)
-		(dnp no)
-		(property "Reference" "CN1"
-			(at 184.15 87.6301 0)
-			(effects
-				(font
-					(size 1.27 1.27)
-				)
-				(justify left)
-			)
-		)
-		(property "Value" "TF31-24S-0.5SH(800)"
-			(at 184.15 85.0901 0)
-			(effects
-				(font
-					(size 1.27 1.27)
-				)
-				(justify left)
-			)
-		)
-		(property "Footprint" "lcsc:FPC-SMD_24P-P0.50_TF31-24S-0.5SH"
-			(at 175.26 44.45 0)
-			(effects
-				(font
-					(size 1.27 1.27)
-				)
-				(hide yes)
-			)
-		)
-		(property "Datasheet" ""
-			(at 175.26 86.36 0)
-			(effects
-				(font
-					(size 1.27 1.27)
-				)
-				(hide yes)
-			)
-		)
-		(property "Description" ""
-			(at 175.26 86.36 0)
-			(effects
-				(font
-					(size 1.27 1.27)
-				)
-				(hide yes)
-			)
-		)
-		(property "LCSC Part" "C3169854"
-			(at 175.26 41.91 0)
-			(effects
-				(font
-					(size 1.27 1.27)
-				)
-				(hide yes)
-			)
-		)
-		(pin "19"
-		)
-		(pin "4"
-		)
-		(pin "21"
-		)
-		(pin "18"
-		)
-		(pin "9"
-		)
-		(pin "26"
-		)
-		(pin "25"
-		)
-		(pin "13"
-		)
-		(pin "23"
-		)
-		(pin "5"
-		)
-		(pin "14"
-		)
-		(pin "20"
-		)
-		(pin "2"
-		)
-		(pin "1"
-		)
-		(pin "22"
-		)
-		(pin "12"
-		)
-		(pin "15"
-		)
-		(pin "24"
-		)
-		(pin "17"
-		)
-		(pin "6"
-		)
-		(pin "10"
-		)
-		(pin "7"
-		)
-		(pin "11"
-		)
-		(pin "8"
-		)
-		(pin "3"
-		)
-		(pin "16"
-		)
-		(instances
-			(project ""
-				(path "/23bf5400-d19c-445b-8744-b63ebcca303d/9cdecd3d-2b1f-4dfc-b0b2-cc7367cb6c39"
-					(reference "CN1")
-					(unit 1)
-				)

Commit message: dotting the i's , list checks before V2 order.
Parts:
- FPC1: LCSC (none) -> C22380687
Changed lines of the file:
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@@
 			)
 		)
-		(property "Datasheet" ""
+		(property "Datasheet" "https://www.lcsc.com/product-detail/C22380687.html"
 			(at 175.26 86.36 0)
 			(effects
@@
 			(effects
 				(font
+					(size 1.27 1.27)
+				)
+				(hide yes)
+			)
+		)
+		(property "LCSC" "C22380687"
+			(at 175.26 86.36 0)
+			(effects
+				(font
