File: display.kicad_sch (KiCad schematic)
At the start: 19 parts, among them Q2 AP2302B

Commit message: Changes for the SSD1681
Parts:
- removed FPC1: GT-F0501SR10-24S1101, lcsc:FPC-SMD_24P-P0.50_GT-F0501SR10-24S1101, symbol lcsc:GT-F0501SR10-24S1101
- added FPC2: 0.5-24P CTSJ-H2.0 119, lcsc:FPC-SMD_24P-P0.50_SHOU-HAN_CTSJ-H2.0, symbol lcsc:0.5-24PCTSJ-H2.0119
Connections:
- net 3V3: now also FPC2.10, FPC2.9
- net BUSY: now also FPC2.16
- net CS: now also FPC2.13
- net DC: now also FPC2.14
- net GDR: now also FPC2.23
- net GND: now also FPC2.17, FPC2.25, FPC2.26, FPC2.8
- net MOSI: now also FPC2.11
- net PREVGH: now also FPC2.4
- net PREVGL: now also FPC2.2
- net RESE: now also FPC2.22
- net RESETn: now also FPC2.15
- net SCK: now also FPC2.12
- net VCOM: now also FPC2.1
- net VGH: now also FPC2.20
- net VGL: now also FPC2.21
- net VSH: now also FPC2.5
- net VSL: now also FPC2.3
- net at C38.2, R13.2: now also FPC2.7
Changed lines of the file:
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@@
 			(justify left bottom)
 		)
-		(property "Net Class" "Power"
+		(property "Netclass" "Power"
 			(at 142.9385 97.79 0)
 			(show_name no)
@@
 			(justify left bottom)
 		)
-		(property "Net Class" "Power"
+		(property "Netclass" "Power"
 			(at 107.3785 105.41 0)
 			(show_name no)
@@
 			(justify left bottom)
 		)
-		(property "Net Class" "Power"
+		(property "Netclass" "Power"
 			(at 84.5185 50.8 0)
 			(show_name no)
@@
 	)
 	(symbol
-		(lib_id "lcsc:GT-F0501SR10-24S1101")
-		(at 175.26 86.36 0)
-		(mirror x)
-		(unit 1)
-		(body_style 1)
-		(exclude_from_sim no)
-		(in_bom yes)
-		(on_board yes)
-		(in_pos_files yes)
-		(dnp no)
-		(property "Reference" "FPC1"
-			(at 182.88 87.6301 0)
-			(show_name no)
-			(do_not_autoplace no)
-			(effects
-				(font
-					(size 1.27 1.27)
-				)
-				(justify left)
-			)
-		)
-		(property "Value" "GT-F0501SR10-24S1101"
-			(at 182.88 85.0901 0)
-			(show_name no)
-			(do_not_autoplace no)
-			(effects
-				(font
-					(size 1.27 1.27)
-				)
-				(justify left)
-			)
-		)
-		(property "Footprint" "lcsc:FPC-SMD_24P-P0.50_GT-F0501SR10-24S1101"
-			(at 175.26 44.45 0)
-			(hide yes)
-			(show_name no)
-			(do_not_autoplace no)
-			(effects
-				(font
-					(size 1.27 1.27)
-				)
-			)
-		)
-		(property "Datasheet" "https://www.lcsc.com/product-detail/C22380687.html"
-			(at 175.26 86.36 0)
-			(hide yes)
-			(show_name no)
-			(do_not_autoplace no)
-			(effects
-				(font
-					(size 1.27 1.27)
-				)
-			)
-		)
-		(property "Description" ""
-			(at 175.26 86.36 0)
-			(hide yes)
-			(show_name no)
-			(do_not_autoplace no)
-			(effects
-				(font
-					(size 1.27 1.27)
-				)
-			)
-		)
-		(property "LCSC Part" "C22380687"
-			(at 175.26 41.91 0)
-			(hide yes)
-			(show_name no)
-			(do_not_autoplace no)
-			(effects
-				(font
-					(size 1.27 1.27)
-				)
-			)
-		)
-		(property "LCSC" "C22380687"
-			(at 175.26 86.36 0)
-			(hide yes)
-			(show_name no)
-			(do_not_autoplace no)
-			(effects
-				(font
-					(size 1.27 1.27)
-				)
-			)
-		)
-		(pin "9"
-		)
-		(pin "12"
-		)
-		(pin "19"
-		)
-		(pin "22"
-		)
-		(pin "17"
-		)
-		(pin "4"
-		)
-		(pin "2"
-		)
-		(pin "14"
-		)
-		(pin "18"
-		)
-		(pin "21"
-		)
-		(pin "1"
-		)
-		(pin "3"
-		)
-		(pin "15"
-		)
-		(pin "8"
-		)
-		(pin "7"
-		)
-		(pin "24"
-		)
-		(pin "5"
-		)
-		(pin "25"
-		)
-		(pin "6"
-		)
-		(pin "13"
-		)
-		(pin "26"
-		)
-		(pin "11"
-		)
-		(pin "10"
-		)
-		(pin "23"
-		)
-		(pin "16"
-		)
-		(pin "20"
-		)
-		(instances
-			(project "bornhack2026-hardware"
-				(path "/23bf5400-d19c-445b-8744-b63ebcca303d/9cdecd3d-2b1f-4dfc-b0b2-cc7367cb6c39"
-					(reference "FPC1")
-					(unit 1)
-				)
-			)
-		)
-	)
-	(symbol
 		(lib_id "symbols:R")
 		(at 99.06 71.12 180)
@@
 					(unit 1)
 				)
+			)
+		)
+	)
+	(symbol
+		(lib_id "lcsc:0.5-24PCTSJ-H2.0119")
+		(at 175.26 86.36 0)
+		(mirror x)
+		(unit 1)
+		(body_style 1)
+		(exclude_from_sim no)
+		(in_bom yes)
+		(on_board yes)
+		(in_pos_files yes)
+		(dnp no)
+		(property "Reference" "FPC2"
+			(at 181.61 87.6301 0)
+			(show_name no)
+			(do_not_autoplace no)
+			(effects
+				(font
+					(size 1.27 1.27)
+				)
+				(justify left)
+			)
+		)
+		(property "Value" "0.5-24P CTSJ-H2.0 119"
+			(at 181.61 85.0901 0)
+			(show_name no)
+			(do_not_autoplace no)
+			(effects
+				(font
+					(size 1.27 1.27)
+				)
+				(justify left)
+			)
+		)
+		(property "Footprint" "lcsc:FPC-SMD_24P-P0.50_SHOU-HAN_CTSJ-H2.0"
+			(at 175.26 44.45 0)
+			(hide yes)
+			(show_name no)
+			(do_not_autoplace no)
+			(effects
+				(font
+					(size 1.27 1.27)
+				)
+			)
+		)
+		(property "Datasheet" ""
+			(at 175.26 86.36 0)
+			(hide yes)
+			(show_name no)
+			(do_not_autoplace no)
+			(effects
+				(font
+					(size 1.27 1.27)
+				)
+			)
+		)
+		(property "Description" ""
+			(at 175.26 86.36 0)
+			(hide yes)
+			(show_name no)
+			(do_not_autoplace no)
+			(effects
+				(font
+					(size 1.27 1.27)
+				)
+			)
+		)
+		(property "LCSC Part" "C2858299"
+			(at 175.26 41.91 0)
+			(hide yes)
+			(show_name no)
+			(do_not_autoplace no)
+			(effects
+				(font
+					(size 1.27 1.27)
+				)
+			)
+		)
+		(pin "8"
+		)
+		(pin "10"
+		)
+		(pin "16"
+		)
+		(pin "17"
+		)
+		(pin "19"
+		)
+		(pin "21"
+		)
+		(pin "23"
+		)
+		(pin "2"
+		)
+		(pin "12"
+		)
+		(pin "18"
+		)
+		(pin "20"
+		)
+		(pin "13"
+		)
+		(pin "15"
+		)
+		(pin "11"
+		)
+		(pin "14"
+		)
+		(pin "24"
+		)
+		(pin "22"
+		)
+		(pin "3"
+		)
+		(pin "6"
+		)
+		(pin "9"
+		)
+		(pin "1"
+		)
+		(pin "25"
+		)
+		(pin "26"
+		)
+		(pin "7"
+		)
+		(pin "5"
+		)
+		(pin "4"
+		)
+		(instances
+			(project "bornhack2026-hardware"
+				(path "/23bf5400-d19c-445b-8744-b63ebcca303d/9cdecd3d-2b1f-4dfc-b0b2-cc7367cb6c39"
+					(reference "FPC2")
+					(unit 1)
+				)
