File: nfc-antenna.kicad_sch (KiCad schematic)
At the start: 9 parts

Commit message: Replaced schottky diode with 1A version, fixed joystick footprint.
Changed lines of the file:
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@@
 		(pin "2"
+		)
+		(pin "0"
 		)
 		(instances
