File: nfc-antenna.kicad_sch (KiCad schematic)
At the start: 3 parts

Commit message: Progress, routed more stuff.
Parts:
- added C20, C59: ~, Capacitor_SMD:C_0402_1005Metric, symbol Device:C_Small
- AE1: footprint (none) -> lcsc:NFC_4uH_COIL; now left out of the parts list
- C42, C43: value C_Small -> 15pF; footprint (none) -> Capacitor_SMD:C_0402_1005Metric
Connections:
- net GND: now also C20.1, C59.1
- net NFC1: now also C20.2
- net NFC2: now also C59.2
Other:
- moved on the sheet: C42, C43

Commit message: Bluetooth antenna should work better, NFC has IPEX for tuning.
Parts:
- added R29, R30: 0, Resistor_SMD:R_0402_1005Metric, symbol Device:R_Small
- added RF2: A-IPEX1-1.25A, lcsc:IPEX-SMD_3P-L2.6-W2.6-LS3.0_RF1200001R, symbol lcsc:A-IPEX1-1.25A
- C42, C43: value 15pF -> 12pF; LCSC (none) -> C161304
Connections:
- net NFC1: now also R29.2; no longer AE1.2, C20.2, C43.2
- net NFC2: now also R30.2; no longer AE1.1, C42.1, C59.2
- new net: AE1.1, C42.1, C59.2, R30.1, RF2.2
- new net: AE1.2, C20.2, C43.2, R29.1, RF2.1
- no-connect marks 0 -> 1
Other:
- note added: "TODO: Tune on prototype current capacitance too low."

Commit message: Routed buttons to MCU.
Parts:
- added C65: ~, Capacitor_SMD:C_0402_1005Metric, symbol Device:C_Small
Connections:
- net at AE1.1, C42.1, C59.2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: now also C65.1
- net at AE1.2, C20.2, C43.2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: now also C65.2
Other:
- moved on the sheet: AE1
Changed lines of the file:
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@@
-	)
-	(junction
-		(at 138.43 96.52)
-		(diameter 0)
-		(color 0 0 0 0)
 	)
 	(junction
@@
 	)
 	(junction
-		(at 138.43 93.98)
+		(at 130.81 97.79)
+		(diameter 0)
+		(color 0 0 0 0)
+	)
+	(junction
+		(at 138.43 92.71)
 		(diameter 0)
 		(color 0 0 0 0)
@@
 	)
 	(junction
+		(at 138.43 97.79)
+		(diameter 0)
+		(color 0 0 0 0)
+	)
+	(junction
+		(at 130.81 92.71)
+		(diameter 0)
+		(color 0 0 0 0)
+	)
+	(junction
 		(at 148.59 83.82)
 		(diameter 0)
@@
 	(wire
 		(pts
+			(xy 125.73 96.52) (xy 125.73 97.79)
+		)
+		(stroke
+			(width 0)
+			(type default)
+		)
+	)
+	(wire
+		(pts
 			(xy 148.59 96.52) (xy 148.59 99.06)
 		)
@@
 	(wire
 		(pts
-			(xy 127 93.98) (xy 138.43 93.98)
-		)
-		(stroke
-			(width 0)
-			(type default)
-		)
-	)
-	(wire
-		(pts
-			(xy 138.43 91.44) (xy 138.43 93.98)
+			(xy 120.65 93.98) (xy 125.73 93.98)
+		)
+		(stroke
+			(width 0)
+			(type default)
+		)
+	)
+	(wire
+		(pts
+			(xy 130.81 92.71) (xy 138.43 92.71)
+		)
+		(stroke
+			(width 0)
+			(type default)
+		)
+	)
+	(wire
+		(pts
+			(xy 138.43 92.71) (xy 138.43 93.98)
+		)
+		(stroke
+			(width 0)
+			(type default)
+		)
+	)
+	(wire
+		(pts
+			(xy 138.43 91.44) (xy 138.43 92.71)
+		)
+		(stroke
+			(width 0)
+			(type default)
+		)
+	)
+	(wire
+		(pts
+			(xy 130.81 97.79) (xy 138.43 97.79)
 		)
 		(stroke
@@
 	(wire
 		(pts
+			(xy 125.73 92.71) (xy 130.81 92.71)
+		)
+		(stroke
+			(width 0)
+			(type default)
+		)
+	)
+	(wire
+		(pts
 			(xy 148.59 96.52) (xy 173.99 96.52)
 		)
@@
 	(wire
 		(pts
+			(xy 125.73 92.71) (xy 125.73 93.98)
+		)
+		(stroke
+			(width 0)
+			(type default)
+		)
+	)
+	(wire
+		(pts
+			(xy 125.73 97.79) (xy 130.81 97.79)
+		)
+		(stroke
+			(width 0)
+			(type default)
+		)
+	)
+	(wire
+		(pts
 			(xy 166.37 93.98) (xy 176.53 93.98)
 		)
@@
 	(wire
 		(pts
-			(xy 138.43 96.52) (xy 138.43 99.06)
+			(xy 138.43 96.52) (xy 138.43 97.79)
 		)
 		(stroke
@@
 	(wire
 		(pts
-			(xy 127 96.52) (xy 138.43 96.52)
+			(xy 120.65 96.52) (xy 125.73 96.52)
 		)
 		(stroke
@@
 		(pts
 			(xy 173.99 96.52) (xy 184.15 96.52)
+		)
+		(stroke
+			(width 0)
+			(type default)
+		)
+	)
+	(wire
+		(pts
+			(xy 138.43 97.79) (xy 138.43 99.06)
 		)
 		(stroke
@@
 	(symbol
 		(lib_id "Device:Antenna_Dipole")
-		(at 121.92 96.52 90)
+		(at 115.57 96.52 90)
 		(unit 1)
 		(exclude_from_sim no)
@@
 		(fields_autoplaced yes)
 		(property "Reference" "AE1"
-			(at 124.46 86.36 90)
+			(at 118.11 86.36 90)
 			(effects
 				(font
@@
 		)
 		(property "Value" "Antenna_Dipole"
-			(at 124.46 88.9 90)
+			(at 118.11 88.9 90)
 			(effects
 				(font
@@
 		)
 		(property "Footprint" "lcsc:NFC_4uH_COIL"
-			(at 121.92 96.52 0)
+			(at 115.57 96.52 0)
 			(effects
 				(font
@@
 		)
 		(property "Datasheet" "https://coil32.net/online-calculators/pcb-inductor-calculator.html"
-			(at 121.92 96.52 0)
+			(at 115.57 96.52 0)
 			(effects
 				(font
@@
 		)
 		(property "Description" "NFC coil antenna"
-			(at 121.92 96.52 0)
+			(at 115.57 96.52 0)
 			(effects
 				(font
@@
 					(unit 1)
 				)
+			)
+		)
+	)
+	(symbol
+		(lib_id "Device:C_Small")
+		(at 130.81 95.25 180)
+		(unit 1)
+		(exclude_from_sim no)
+		(in_bom no)
+		(on_board yes)
+		(dnp yes)
+		(fields_autoplaced yes)
+		(property "Reference" "C65"
+			(at 133.35 93.9735 0)
+			(effects
+				(font
+					(size 1.27 1.27)
+				)
+				(justify right)
+			)
+		)
+		(property "Value" "~"
+			(at 133.35 96.5135 0)
+			(effects
+				(font
+					(size 1.27 1.27)
+				)
+				(justify right)
+			)
+		)
+		(property "Footprint" "Capacitor_SMD:C_0402_1005Metric"
+			(at 130.81 95.25 0)
+			(effects
+				(font
+					(size 1.27 1.27)
+				)
+				(hide yes)
+			)
+		)
+		(property "Datasheet" "~"
+			(at 130.81 95.25 0)
+			(effects
+				(font
+					(size 1.27 1.27)
+				)
+				(hide yes)
+			)
+		)
+		(property "Description" "Unpolarized capacitor, small symbol"
+			(at 130.81 95.25 0)
+			(effects
+				(font
+					(size 1.27 1.27)
+				)
+				(hide yes)
+			)
+		)
+		(pin "1"
+		)
+		(pin "2"
+		)
+		(instances
+			(project "bornhack2026-hardware"
+				(path "/23bf5400-d19c-445b-8744-b63ebcca303d/90853474-a0e8-4c32-9bb2-223cb1f08aa7"
+					(reference "C65")
+					(unit 1)
+				)

Commit message: Checked PCBA for JLCPCB.
Parts:
- C43: LCSC C161304 -> C161304
Changed lines of the file:
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@@
 			)
 		)
-		(property "LCSC" "C161304 "
+		(property "LCSC" "C161304"
 			(at 148.59 88.9 0)
 			(effects

Commit message: Changed NFC coil + tune C's to match better with datasheet.
Parts:
- AE1: footprint lcsc:NFC_4uH_COIL -> lcsc:NFC_2.8uH_COIL
- C42, C43: value 12pF -> 75pF; LCSC C161304 -> C37809
Changed lines of the file:
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@@
 			)
 		)
-		(property "Value" "12pF"
+		(property "Value" "75pF"
 			(at 151.13 102.8762 0)
 			(effects
@@
 			)
 		)
-		(property "Datasheet" "https://jlcpcb.com/partdetail/172685-GJM1555C1H120FB01D/C161304"
+		(property "Datasheet" "https://jlcpcb.com/partdetail/38789-0402CG750J500NT/C37809"
 			(at 148.59 101.6 0)
 			(effects
@@
 			)
 		)
-		(property "LCSC" "C161304"
+		(property "LCSC" "C37809"
+			(at 148.59 101.6 0)
+			(effects
+				(font
+					(size 1.27 1.27)
+				)
+				(hide yes)
+			)
+		)
+		(property "Resource" ""
 			(at 148.59 101.6 0)
 			(effects
@@
 			)
 		)
+		(property "Resource" ""
+			(at 138.43 101.6 0)
+			(effects
+				(font
+					(size 1.27 1.27)
+				)
+				(hide yes)
+			)
+		)
 		(pin "1"
 		)
@@
 		)
 		(property "LCSC" "C17168"
+			(at 179.07 93.98 90)
+			(effects
+				(font
+					(size 1.27 1.27)
+				)
+				(hide yes)
+			)
+		)
+		(property "Resource" ""
 			(at 179.07 93.98 90)
 			(effects
@@
 			)
 		)
-		(property "Value" "12pF"
+		(property "Value" "75pF"
 			(at 151.13 90.1762 0)
 			(effects
@@
 			)
 		)
-		(property "Datasheet" "https://jlcpcb.com/partdetail/172685-GJM1555C1H120FB01D/C161304"
+		(property "Datasheet" "https://jlcpcb.com/partdetail/38789-0402CG750J500NT/C37809"
 			(at 148.59 88.9 0)
 			(effects
@@
 			)
 		)
-		(property "LCSC" "C161304"
+		(property "LCSC" "C37809"
+			(at 148.59 88.9 0)
+			(effects
+				(font
+					(size 1.27 1.27)
+				)
+				(hide yes)
+			)
+		)
+		(property "Resource" ""
 			(at 148.59 88.9 0)
 			(effects
@@
 			)
 		)
+		(property "Resource" ""
+			(at 138.43 88.9 0)
+			(effects
+				(font
+					(size 1.27 1.27)
+				)
+				(hide yes)
+			)
+		)
 		(pin "1"
 		)
@@
 			)
 		)
-		(property "Footprint" "lcsc:NFC_4uH_COIL"
+		(property "Footprint" "lcsc:NFC_2.8uH_COIL"
 			(at 115.57 96.52 0)
 			(effects
@@
 		(property "Description" "NFC coil antenna"
 			(at 115.57 96.52 0)
+			(effects
+				(font
+					(size 1.27 1.27)
+				)
+				(hide yes)
+			)
+		)
+		(property "Resource" ""
+			(at 115.57 96.52 90)
 			(effects
 				(font
@@
 			)
 		)
+		(property "Resource" ""
+			(at 186.69 96.52 90)
+			(effects
+				(font
+					(size 1.27 1.27)
+				)
+				(hide yes)
+			)
+		)
 		(pin "1"
 		)
@@
 					(size 1.27 1.27)
 				)
+			)
+		)
+		(property "Resource" ""
+			(at 166.37 88.9 0)
+			(effects
+				(font
+					(size 1.27 1.27)
+				)
+				(hide yes)
 			)
 		)
@@
 			(at 130.81 95.25 0)
 			(effects
+				(font
+					(size 1.27 1.27)
+				)
+				(hide yes)
+			)
+		)
+		(property "Resource" ""
+			(at 130.81 95.25 0)
+			(effects

Commit message: Fixed PCBA rotations in using component property.
Parts:
- AE1: now not fitted
Changed lines of the file:
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@@
 		(in_bom no)
 		(on_board yes)
-		(dnp no)
+		(dnp yes)
 		(fields_autoplaced yes)
 		(property "Reference" "AE1"

Commit message: Tuning capacitors NRF 22pF 13.5MHz
Parts:
- C42, C43: value 75pF -> 22pF; LCSC C37809 -> C1555
Changed lines of the file:
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@@
 			)
 		)
-		(property "Value" "75pF"
+		(property "Value" "22pF"
 			(at 151.13 102.8762 0)
 			(effects
@@
 			)
 		)
-		(property "Datasheet" "https://jlcpcb.com/partdetail/38789-0402CG750J500NT/C37809"
+		(property "Datasheet" "https://jlcpcb.com/partdetail/1907-0402CG220J500NT/C1555"
 			(at 148.59 101.6 0)
 			(effects
@@
 			)
 		)
-		(property "LCSC" "C37809"
+		(property "LCSC" "C1555"
 			(at 148.59 101.6 0)
 			(effects
@@
 			)
 		)
-		(property "Value" "75pF"
+		(property "Value" "22pF"
 			(at 151.13 90.1762 0)
 			(effects
@@
 			)
 		)
-		(property "Datasheet" "https://jlcpcb.com/partdetail/38789-0402CG750J500NT/C37809"
+		(property "Datasheet" "https://jlcpcb.com/partdetail/1907-0402CG220J500NT/C1555"
 			(at 148.59 88.9 0)
 			(effects
@@
 			)
 		)
-		(property "LCSC" "C37809"
+		(property "LCSC" "C1555"
 			(at 148.59 88.9 0)
 			(effects
