File: nfc-antenna.kicad_sch (KiCad schematic)
At the start: 9 parts

Commit message: On to proto v2.
Parts:
- removed RF2: A-IPEX1-1.25A, lcsc:IPEX-SMD_3P-L2.6-W2.6-LS3.0_RF1200001R, symbol lcsc:A-IPEX1-1.25A
- C42, C43: value 75pF -> 22pF; LCSC C37809 -> C1555
Connections:
- no-connect marks 1 -> 0
Other:
- moved on the sheet: R29

Commit message: Add ESD protoction to USB-C, small fixes
Parts:
- C42, C43: value 22pF -> 68pF; LCSC C1555 -> C389103
Other:
- moved on the sheet: R29, R30
Changed lines of the file:
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@@
-	)
-	(junction
-		(at 148.59 93.98)
-		(diameter 0)
-		(color 0 0 0 0)
-	)
-	(junction
-		(at 148.59 96.52)
-		(diameter 0)
-		(color 0 0 0 0)
 	)
 	(junction
@@
 	)
 	(junction
+		(at 148.59 92.71)
+		(diameter 0)
+		(color 0 0 0 0)
+	)
+	(junction
 		(at 138.43 92.71)
 		(diameter 0)
@@
 	)
 	(junction
+		(at 148.59 97.79)
+		(diameter 0)
+		(color 0 0 0 0)
+	)
+	(junction
 		(at 130.81 92.71)
 		(diameter 0)
@@
 	(wire
 		(pts
-			(xy 148.59 91.44) (xy 148.59 93.98)
+			(xy 148.59 91.44) (xy 148.59 92.71)
 		)
 		(stroke
@@
 	(wire
 		(pts
-			(xy 148.59 96.52) (xy 148.59 99.06)
-		)
-		(stroke
-			(width 0)
-			(type default)
-		)
-	)
-	(wire
-		(pts
-			(xy 189.23 96.52) (xy 191.77 96.52)
+			(xy 189.23 97.79) (xy 191.77 97.79)
 		)
 		(stroke
@@
 	(wire
 		(pts
-			(xy 138.43 92.71) (xy 138.43 93.98)
-		)
-		(stroke
-			(width 0)
-			(type default)
-		)
-	)
-	(wire
-		(pts
 			(xy 138.43 91.44) (xy 138.43 92.71)
 		)
@@
 	(wire
 		(pts
-			(xy 138.43 93.98) (xy 148.59 93.98)
+			(xy 138.43 92.71) (xy 148.59 92.71)
 		)
 		(stroke
@@
 	(wire
 		(pts
-			(xy 148.59 93.98) (xy 184.15 93.98)
-		)
-		(stroke
-			(width 0)
-			(type default)
-		)
-	)
-	(wire
-		(pts
-			(xy 138.43 96.52) (xy 138.43 97.79)
-		)
-		(stroke
-			(width 0)
-			(type default)
-		)
-	)
-	(wire
-		(pts
-			(xy 138.43 96.52) (xy 148.59 96.52)
+			(xy 148.59 92.71) (xy 184.15 92.71)
+		)
+		(stroke
+			(width 0)
+			(type default)
+		)
+	)
+	(wire
+		(pts
+			(xy 138.43 97.79) (xy 148.59 97.79)
 		)
 		(stroke
@@
 	(wire
 		(pts
-			(xy 148.59 96.52) (xy 184.15 96.52)
+			(xy 148.59 97.79) (xy 184.15 97.79)
 		)
 		(stroke
@@
 	(wire
 		(pts
-			(xy 189.23 93.98) (xy 191.77 93.98)
+			(xy 148.59 97.79) (xy 148.59 99.06)
+		)
+		(stroke
+			(width 0)
+			(type default)
+		)
+	)
+	(wire
+		(pts
+			(xy 189.23 92.71) (xy 191.77 92.71)
 		)
 		(stroke
@@
 	(hierarchical_label "NFC1"
 		(shape input)
-		(at 191.77 93.98 0)
+		(at 191.77 92.71 0)
 		(effects
 			(font
@@
 	(hierarchical_label "NFC2"
 		(shape input)
-		(at 191.77 96.52 0)
+		(at 191.77 97.79 0)
 		(effects
 			(font
@@
 			)
 		)
-		(property "Value" "22pF"
+		(property "Value" "68pF"
 			(at 151.13 102.8762 0)
 			(effects
@@
 			)
 		)
-		(property "Datasheet" "https://jlcpcb.com/partdetail/1907-0402CG220J500NT/C1555"
+		(property "Datasheet" "https://jlcpcb.com/partdetail/YAGEO-CC0402FRNPO9BN680/C389103"
 			(at 148.59 101.6 0)
 			(effects
@@
 			)
 		)
-		(property "LCSC" "C1555"
+		(property "LCSC" "C389103"
 			(at 148.59 101.6 0)
 			(effects
@@
 	(symbol
 		(lib_id "Device:R_Small")
-		(at 186.69 93.98 90)
+		(at 186.69 92.71 90)
 		(unit 1)
 		(exclude_from_sim no)
@@
 		(dnp no)
 		(property "Reference" "R29"
-			(at 186.69 89.662 90)
+			(at 186.69 88.392 90)
 			(effects
 				(font
@@
 		)
 		(property "Value" "0"
-			(at 186.69 91.44 90)
+			(at 186.69 90.17 90)
 			(effects
 				(font
@@
 		)
 		(property "Footprint" "Resistor_SMD:R_0402_1005Metric"
-			(at 186.69 93.98 0)
+			(at 186.69 92.71 0)
 			(effects
 				(font
@@
 		)
 		(property "Datasheet" "https://jlcpcb.com/partdetail/17853-0402WGF0000TCE/C17168"
-			(at 186.69 93.98 0)
+			(at 186.69 92.71 0)
 			(effects
 				(font
@@
 		)
 		(property "Description" "Resistor, small symbol"
-			(at 186.69 93.98 0)
+			(at 186.69 92.71 0)
 			(effects
 				(font
@@
 		)
 		(property "LCSC" "C17168"
-			(at 186.69 93.98 90)
+			(at 186.69 92.71 90)
 			(effects
 				(font
@@
 		)
 		(property "Resource" ""
-			(at 186.69 93.98 90)
+			(at 186.69 92.71 90)
 			(effects
 				(font
@@
 		)
 		(property "pin1" ""
-			(at 186.69 93.98 90)
+			(at 186.69 92.71 90)
 			(effects
 				(font
@@
 		)
 		(property "pin2" ""
-			(at 186.69 93.98 90)
+			(at 186.69 92.71 90)
 			(effects
 				(font
@@
 		)
 		(property "pin3" ""
-			(at 186.69 93.98 90)
+			(at 186.69 92.71 90)
 			(effects
 				(font
@@
 		)
 		(property "pin4" ""
-			(at 186.69 93.98 90)
+			(at 186.69 92.71 90)
 			(effects
 				(font
@@
 		)
 		(property "pin5" ""
-			(at 186.69 93.98 90)
+			(at 186.69 92.71 90)
 			(effects
 				(font
@@
 		)
 		(property "Sim.Device" ""
-			(at 186.69 93.98 90)
+			(at 186.69 92.71 90)
 			(effects
 				(font
@@
 		)
 		(property "Sim.Pins" ""
-			(at 186.69 93.98 90)
+			(at 186.69 92.71 90)
 			(effects
 				(font
@@
 			)
 		)
-		(property "Value" "22pF"
+		(property "Value" "68pF"
 			(at 151.13 90.1762 0)
 			(effects
@@
 			)
 		)
-		(property "Datasheet" "https://jlcpcb.com/partdetail/1907-0402CG220J500NT/C1555"
+		(property "Datasheet" "https://jlcpcb.com/partdetail/YAGEO-CC0402FRNPO9BN680/C389103"
 			(at 148.59 88.9 0)
 			(effects
@@
 			)
 		)
-		(property "LCSC" "C1555"
+		(property "LCSC" "C389103"
 			(at 148.59 88.9 0)
 			(effects
@@
 	(symbol
 		(lib_id "Device:R_Small")
-		(at 186.69 96.52 90)
+		(at 186.69 97.79 90)
 		(unit 1)
 		(exclude_from_sim no)
@@
 		(dnp no)
 		(property "Reference" "R30"
-			(at 186.69 100.076 90)
+			(at 186.69 101.346 90)
 			(effects
 				(font
@@
 		)
 		(property "Value" "0"
-			(at 186.69 98.298 90)
+			(at 186.69 99.568 90)
 			(effects
 				(font
@@
 		)
 		(property "Footprint" "Resistor_SMD:R_0402_1005Metric"
-			(at 186.69 96.52 0)
+			(at 186.69 97.79 0)
 			(effects
 				(font
@@
 		)
 		(property "Datasheet" "https://jlcpcb.com/partdetail/17853-0402WGF0000TCE/C17168"
-			(at 186.69 96.52 0)
+			(at 186.69 97.79 0)
 			(effects
 				(font
@@
 		)
 		(property "Description" "Resistor, small symbol"
-			(at 186.69 96.52 0)
+			(at 186.69 97.79 0)
 			(effects
 				(font
@@
 		)
 		(property "LCSC" "C17168"
-			(at 186.69 96.52 90)
+			(at 186.69 97.79 90)
 			(effects
 				(font
@@
 		)
 		(property "Resource" ""
-			(at 186.69 96.52 90)
+			(at 186.69 97.79 90)
 			(effects
 				(font
@@
 		)
 		(property "pin1" ""
-			(at 186.69 96.52 90)
+			(at 186.69 97.79 90)
 			(effects
 				(font
@@
 		)
 		(property "pin2" ""
-			(at 186.69 96.52 90)
+			(at 186.69 97.79 90)
 			(effects
 				(font
@@
 		)
 		(property "pin3" ""
-			(at 186.69 96.52 90)
+			(at 186.69 97.79 90)
 			(effects
 				(font
@@
 		)
 		(property "pin4" ""
-			(at 186.69 96.52 90)
+			(at 186.69 97.79 90)
 			(effects
 				(font
@@
 		)
 		(property "pin5" ""
-			(at 186.69 96.52 90)
+			(at 186.69 97.79 90)
 			(effects
 				(font
@@
 		)
 		(property "Sim.Device" ""
-			(at 186.69 96.52 90)
+			(at 186.69 97.79 90)
 			(effects
 				(font
@@
 		)
 		(property "Sim.Pins" ""
-			(at 186.69 96.52 90)
-			(effects
-				(font
+			(at 186.69 97.79 90)
+			(effects
+				(font

Commit message: Prototype V3, speaker resistor 50 ohm, 500ohm on to second pad epd
Parts:
- C20, C59, C65: value ~ -> (none)
