File: gen_button.kicad_sch (KiCad schematic)
At the start: 2 parts, among them SW2 TS3425PA 160GF 098

Commit message: Switched the LC filters from ceramic LoRa filter.
Parts:
- R15: LCSC (none) -> C25744
Changed lines of the file:
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@@
 			)
 		)
-		(property "Datasheet" "~"
+		(property "Datasheet" "https://jlcpcb.com/partdetail/26487-0402WGF1002TCE/C25744"
 			(at 78.74 55.88 0)
 			(effects
@@
 			(at 78.74 55.88 0)
 			(effects
+				(font
+					(size 1.27 1.27)
+				)
+				(hide yes)
+			)
+		)
+		(property "LCSC" "C25744"
+			(at 78.74 55.88 0)
+			(effects

Commit message: Progress, routed more stuff.
Parts:
- SW6: renamed from SW2; footprint lcsc:SW-SMD_4P-L4.2-W3.4-P2.15-LS5.2 -> lcsc:KEY-SMD_2P-L6.0-W6.0-P6.00; symbol lcsc:TS3425PA160GF098 -> lcsc:SKPMAME010; LCSC (none) -> C5363473; LCSC Part C5363473 -> C115348
- renumbered R15 to R19
Connections:
- net GND: now also SW6.1; no longer SW6.3
- no-connect marks 2 -> 0
Other:
- moved on the sheet: R19
Changed lines of the file:
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@@
 		(color 0 0 0 0)
 	)
-	(no_connect
-		(at 52.07 58.42)
-	)
-	(no_connect
-		(at 72.39 68.58)
+	(wire
+		(pts
+			(xy 52.07 58.42) (xy 57.15 58.42)
+		)
+		(stroke
+			(width 0)
+			(type default)
+		)
 	)
 	(wire
@@
 		(pts
 			(xy 72.39 58.42) (xy 78.74 58.42)
+		)
+		(stroke
+			(width 0)
+			(type default)
+		)
+	)
+	(wire
+		(pts
+			(xy 78.74 55.88) (xy 78.74 58.42)
+		)
+		(stroke
+			(width 0)
+			(type default)
+		)
+	)
+	(wire
+		(pts
+			(xy 52.07 58.42) (xy 52.07 68.58)
 		)
 		(stroke
@@
 	(hierarchical_label "3V3"
 		(shape input)
-		(at 78.74 53.34 90)
+		(at 78.74 50.8 90)
 		(effects
 			(font
@@
 	(symbol
 		(lib_id "Device:R_Small")
-		(at 78.74 55.88 0)
+		(at 78.74 53.34 0)
 		(unit 1)
 		(exclude_from_sim no)
@@
 		(dnp no)
 		(fields_autoplaced yes)
-		(property "Reference" "R15"
+		(property "Reference" "R19"
+			(at 81.28 52.0699 0)
+			(effects
+				(font
+					(size 1.016 1.016)
+				)
+				(justify left)
+			)
+		)
+		(property "Value" "10k"
 			(at 81.28 54.6099 0)
 			(effects
 				(font
-					(size 1.016 1.016)
+					(size 1.27 1.27)
 				)
 				(justify left)
 			)
 		)
-		(property "Value" "10k"
-			(at 81.28 57.1499 0)
-			(effects
-				(font
-					(size 1.27 1.27)
-				)
-				(justify left)
-			)
-		)
 		(property "Footprint" "Resistor_SMD:R_0402_1005Metric"
-			(at 78.74 55.88 0)
+			(at 78.74 53.34 0)
 			(effects
 				(font
@@
 		)
 		(property "Datasheet" "https://jlcpcb.com/partdetail/26487-0402WGF1002TCE/C25744"
-			(at 78.74 55.88 0)
+			(at 78.74 53.34 0)
 			(effects
 				(font
@@
 		)
 		(property "Description" "Resistor, small symbol"
-			(at 78.74 55.88 0)
+			(at 78.74 53.34 0)
 			(effects
 				(font
@@
 		)
 		(property "LCSC" "C25744"
-			(at 78.74 55.88 0)
+			(at 78.74 53.34 0)
 			(effects
 				(font
@@
 					(unit 1)
 				)
-				(path "/23bf5400-d19c-445b-8744-b63ebcca303d/1f4fc1c2-c6dd-4c37-a48b-5ed4d54351cc/226789dd-c696-45c4-96c5-c7a5d92148eb"
-					(reference "R14")
-					(unit 1)
-				)
 				(path "/23bf5400-d19c-445b-8744-b63ebcca303d/1f4fc1c2-c6dd-4c37-a48b-5ed4d54351cc/388f31d4-eb5f-444f-b721-36e3eb3ac7fd"
 					(reference "R20")
 					(unit 1)
 				)
-				(path "/23bf5400-d19c-445b-8744-b63ebcca303d/1f4fc1c2-c6dd-4c37-a48b-5ed4d54351cc/62b8fb51-fa99-487d-8ffd-9acc3ff5ffd7"
-					(reference "R23")
-					(unit 1)
-				)
-				(path "/23bf5400-d19c-445b-8744-b63ebcca303d/1f4fc1c2-c6dd-4c37-a48b-5ed4d54351cc/76feefb0-eecb-4e68-be3f-437d9c0218bd"
-					(reference "R18")
-					(unit 1)
-				)
-				(path "/23bf5400-d19c-445b-8744-b63ebcca303d/1f4fc1c2-c6dd-4c37-a48b-5ed4d54351cc/a0d8777c-f640-40a2-81c9-41b0bad380fd"
-					(reference "R16")
-					(unit 1)
-				)
-				(path "/23bf5400-d19c-445b-8744-b63ebcca303d/1f4fc1c2-c6dd-4c37-a48b-5ed4d54351cc/b546cf1c-99f0-406e-b30e-bca34362d495"
-					(reference "R22")
-					(unit 1)
-				)
 				(path "/23bf5400-d19c-445b-8744-b63ebcca303d/1f4fc1c2-c6dd-4c37-a48b-5ed4d54351cc/db62785b-07c7-49c0-8737-437f813264da"
 					(reference "R19")
 					(unit 1)
 				)
-				(path "/23bf5400-d19c-445b-8744-b63ebcca303d/1f4fc1c2-c6dd-4c37-a48b-5ed4d54351cc/e9b7ca2d-62c6-49f0-9abe-89336bb8d577"
-					(reference "R15")
-					(unit 1)
-				)
 			)
 		)
 	)
 	(symbol
-		(lib_id "lcsc:TS3425PA160GF098")
-		(at 62.23 63.5 0)
+		(lib_id "lcsc:SKPMAME010")
+		(at 64.77 55.88 0)
 		(unit 1)
 		(exclude_from_sim no)
@@
 		(dnp no)
 		(fields_autoplaced yes)
-		(property "Reference" "SW2"
-			(at 62.23 53.34 0)
+		(property "Reference" "SW6"
+			(at 64.77 48.26 0)
 			(effects
 				(font
@@
 		)
 		(property "Value" "TS3425PA 160GF 098"
-			(at 62.23 55.88 0)
-			(effects
-				(font
-					(size 1.27 1.27)
-				)
-			)
-		)
-		(property "Footprint" "lcsc:SW-SMD_4P-L4.2-W3.4-P2.15-LS5.2"
-			(at 62.23 76.2 0)
-			(effects
-				(font
-					(size 1.27 1.27)
-				)
-				(hide yes)
-			)
-		)
-		(property "Datasheet" ""
-			(at 62.23 63.5 0)
+			(at 64.77 50.8 0)
+			(effects
+				(font
+					(size 1.27 1.27)
+				)
+			)
+		)
+		(property "Footprint" "lcsc:KEY-SMD_2P-L6.0-W6.0-P6.00"
+			(at 64.77 66.04 0)
+			(effects
+				(font
+					(size 1.27 1.27)
+				)
+				(hide yes)
+			)
+		)
+		(property "Datasheet" "https://lcsc.com/product-detail/Tactile-Switches_ALPS_SKPMAME010_6-6-5-1-57N_C115348.html"
+			(at 64.77 68.58 0)
 			(effects
 				(font
@@
 		)
 		(property "Description" ""
-			(at 62.23 63.5 0)
-			(effects
-				(font
-					(size 1.27 1.27)
-				)
-				(hide yes)
-			)
-		)
-		(property "LCSC Part" "C5363473"
-			(at 62.23 78.74 0)
-			(effects
-				(font
-					(size 1.27 1.27)
-				)
-				(hide yes)
-			)
-		)
-		(pin "4"
+			(at 64.77 55.88 0)
+			(effects
+				(font
+					(size 1.27 1.27)
+				)
+				(hide yes)
+			)
+		)
+		(property "LCSC Part" "C115348"
+			(at 64.77 71.12 0)
+			(effects
+				(font
+					(size 1.27 1.27)
+				)
+				(hide yes)
+			)
+		)
+		(property "LCSC" "C5363473"
+			(at 64.77 55.88 0)
+			(effects
+				(font
+					(size 1.27 1.27)
+				)
+				(hide yes)
+			)
 		)
 		(pin "1"
 		)
 		(pin "2"
-		)
-		(pin "3"
 		)
 		(instances
@@
 					(unit 1)
 				)
-				(path "/23bf5400-d19c-445b-8744-b63ebcca303d/1f4fc1c2-c6dd-4c37-a48b-5ed4d54351cc/226789dd-c696-45c4-96c5-c7a5d92148eb"
-					(reference "SW1")
-					(unit 1)
-				)
 				(path "/23bf5400-d19c-445b-8744-b63ebcca303d/1f4fc1c2-c6dd-4c37-a48b-5ed4d54351cc/388f31d4-eb5f-444f-b721-36e3eb3ac7fd"
 					(reference "SW7")
 					(unit 1)
 				)
-				(path "/23bf5400-d19c-445b-8744-b63ebcca303d/1f4fc1c2-c6dd-4c37-a48b-5ed4d54351cc/62b8fb51-fa99-487d-8ffd-9acc3ff5ffd7"
-					(reference "SW10")
-					(unit 1)
-				)
-				(path "/23bf5400-d19c-445b-8744-b63ebcca303d/1f4fc1c2-c6dd-4c37-a48b-5ed4d54351cc/76feefb0-eecb-4e68-be3f-437d9c0218bd"
-					(reference "SW5")
-					(unit 1)
-				)
-				(path "/23bf5400-d19c-445b-8744-b63ebcca303d/1f4fc1c2-c6dd-4c37-a48b-5ed4d54351cc/a0d8777c-f640-40a2-81c9-41b0bad380fd"
-					(reference "SW3")
-					(unit 1)
-				)
-				(path "/23bf5400-d19c-445b-8744-b63ebcca303d/1f4fc1c2-c6dd-4c37-a48b-5ed4d54351cc/b546cf1c-99f0-406e-b30e-bca34362d495"
-					(reference "SW9")
-					(unit 1)
-				)
 				(path "/23bf5400-d19c-445b-8744-b63ebcca303d/1f4fc1c2-c6dd-4c37-a48b-5ed4d54351cc/db62785b-07c7-49c0-8737-437f813264da"
 					(reference "SW6")
-					(unit 1)
-				)
-				(path "/23bf5400-d19c-445b-8744-b63ebcca303d/1f4fc1c2-c6dd-4c37-a48b-5ed4d54351cc/e9b7ca2d-62c6-49f0-9abe-89336bb8d577"
-					(reference "SW2")
 					(unit 1)
 				)
@@
 		(dnp no)
 		(fields_autoplaced yes)
-		(property "Reference" "#PWR072"
+		(property "Reference" "#PWR076"
 			(at 52.07 74.93 0)
 			(effects
@@
 					(unit 1)
 				)
-				(path "/23bf5400-d19c-445b-8744-b63ebcca303d/1f4fc1c2-c6dd-4c37-a48b-5ed4d54351cc/226789dd-c696-45c4-96c5-c7a5d92148eb"
-					(reference "#PWR071")
-					(unit 1)
-				)
 				(path "/23bf5400-d19c-445b-8744-b63ebcca303d/1f4fc1c2-c6dd-4c37-a48b-5ed4d54351cc/388f31d4-eb5f-444f-b721-36e3eb3ac7fd"
 					(reference "#PWR077")
 					(unit 1)
 				)
-				(path "/23bf5400-d19c-445b-8744-b63ebcca303d/1f4fc1c2-c6dd-4c37-a48b-5ed4d54351cc/62b8fb51-fa99-487d-8ffd-9acc3ff5ffd7"
-					(reference "#PWR080")
-					(unit 1)
-				)
-				(path "/23bf5400-d19c-445b-8744-b63ebcca303d/1f4fc1c2-c6dd-4c37-a48b-5ed4d54351cc/76feefb0-eecb-4e68-be3f-437d9c0218bd"
-					(reference "#PWR075")
-					(unit 1)
-				)
-				(path "/23bf5400-d19c-445b-8744-b63ebcca303d/1f4fc1c2-c6dd-4c37-a48b-5ed4d54351cc/a0d8777c-f640-40a2-81c9-41b0bad380fd"
-					(reference "#PWR073")
-					(unit 1)
-				)
-				(path "/23bf5400-d19c-445b-8744-b63ebcca303d/1f4fc1c2-c6dd-4c37-a48b-5ed4d54351cc/b546cf1c-99f0-406e-b30e-bca34362d495"
-					(reference "#PWR079")
-					(unit 1)
-				)
 				(path "/23bf5400-d19c-445b-8744-b63ebcca303d/1f4fc1c2-c6dd-4c37-a48b-5ed4d54351cc/db62785b-07c7-49c0-8737-437f813264da"
 					(reference "#PWR076")
 					(unit 1)
 				)
-				(path "/23bf5400-d19c-445b-8744-b63ebcca303d/1f4fc1c2-c6dd-4c37-a48b-5ed4d54351cc/e9b7ca2d-62c6-49f0-9abe-89336bb8d577"
-					(reference "#PWR072")
-					(unit 1)
-				)

Commit message: Add capacitors, add DC pin to epaper-display.
Parts:
- added C60: 100nF, Capacitor_SMD:C_0402_1005Metric, symbol symbols:C
Connections:
- net BTN_OUT: now also C60.2
- net GND: now also C60.1
Changed lines of the file:
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@@
 		(color 0 0 0 0)
 	)
+	(junction
+		(at 52.07 67.31)
+		(diameter 0)
+		(color 0 0 0 0)
+	)
 	(wire
 		(pts
@@
 	(wire
 		(pts
+			(xy 52.07 67.31) (xy 52.07 68.58)
+		)
+		(stroke
+			(width 0)
+			(type default)
+		)
+	)
+	(wire
+		(pts
 			(xy 78.74 58.42) (xy 95.25 58.42)
 		)
@@
 	(wire
 		(pts
+			(xy 78.74 66.04) (xy 78.74 67.31)
+		)
+		(stroke
+			(width 0)
+			(type default)
+		)
+	)
+	(wire
+		(pts
 			(xy 72.39 58.42) (xy 78.74 58.42)
 		)
@@
 	(wire
 		(pts
+			(xy 52.07 67.31) (xy 78.74 67.31)
+		)
+		(stroke
+			(width 0)
+			(type default)
+		)
+	)
+	(wire
+		(pts
 			(xy 78.74 55.88) (xy 78.74 58.42)
 		)
@@
 	(wire
 		(pts
-			(xy 52.07 58.42) (xy 52.07 68.58)
+			(xy 52.07 58.42) (xy 52.07 67.31)
 		)
 		(stroke
@@
 					(unit 1)
 				)
+			)
+		)
+	)
+	(symbol
+		(lib_id "symbols:C")
+		(at 78.74 62.23 180)
+		(unit 1)
+		(exclude_from_sim no)
+		(in_bom yes)
+		(on_board yes)
+		(dnp no)
+		(property "Reference" "C60"
+			(at 83.82 60.96 0)
+			(effects
+				(font
+					(size 1.27 1.27)
+				)
+				(justify left)
+			)
+		)
+		(property "Value" "100nF"
+			(at 86.36 63.5 0)
+			(effects
+				(font
+					(size 1.27 1.27)
+				)
+				(justify left)
+			)
+		)
+		(property "Footprint" "Capacitor_SMD:C_0402_1005Metric"
+			(at 77.7748 58.42 0)
+			(effects
+				(font
+					(size 1.27 1.27)
+				)
+				(hide yes)
+			)
+		)
+		(property "Datasheet" "https://jlcpcb.com/partdetail/1877-CL05B104KO5NNNC/C1525"
+			(at 78.74 62.23 0)
+			(effects
+				(font
+					(size 1.27 1.27)
+				)
+				(hide yes)
+			)
+		)
+		(property "Description" ""
+			(at 78.74 62.23 0)
+			(effects
+				(font
+					(size 1.27 1.27)
+				)
+				(hide yes)
+			)
+		)
+		(property "LCSC" "C1525"
+			(at 78.74 62.23 0)
+			(effects
+				(font
+					(size 1.27 1.27)
+				)
+				(hide yes)
+			)
+		)
+		(property "Resource" ""
+			(at 78.74 62.23 0)
+			(effects
+				(font
+					(size 1.27 1.27)
+				)
+				(hide yes)
+			)
+		)
+		(property "pin1" ""
+			(at 78.74 62.23 0)
+			(effects
+				(font
+					(size 1.27 1.27)
+				)
+				(hide yes)
+			)
+		)
+		(property "pin2" ""
+			(at 78.74 62.23 0)
+			(effects
+				(font
+					(size 1.27 1.27)
+				)
+				(hide yes)
+			)
+		)
+		(property "pin3" ""
+			(at 78.74 62.23 0)
+			(effects
+				(font
+					(size 1.27 1.27)
+				)
+				(hide yes)
+			)
+		)
+		(property "pin4" ""
+			(at 78.74 62.23 0)
+			(effects
+				(font
+					(size 1.27 1.27)
+				)
+				(hide yes)
+			)
+		)
+		(property "pin5" ""
+			(at 78.74 62.23 0)
+			(effects
+				(font
+					(size 1.27 1.27)
+				)
+				(hide yes)
+			)
+		)
+		(property "Sim.Device" ""
+			(at 78.74 62.23 0)
+			(effects
+				(font
+					(size 1.27 1.27)
+				)
+				(hide yes)
+			)
+		)
+		(property "Sim.Pins" ""
+			(at 78.74 62.23 0)
+			(effects
+				(font
+					(size 1.27 1.27)
+				)
+				(hide yes)
+			)
+		)
+		(pin "1"
+		)
+		(pin "2"
+		)
+		(instances
+			(project "bornhack2026-hardware"
+				(path "/23bf5400-d19c-445b-8744-b63ebcca303d/1f4fc1c2-c6dd-4c37-a48b-5ed4d54351cc/1c8ff3e2-2f4f-4cda-9ba0-6180b9389fcf"
+					(reference "C61")
+					(unit 1)
+				)
+				(path "/23bf5400-d19c-445b-8744-b63ebcca303d/1f4fc1c2-c6dd-4c37-a48b-5ed4d54351cc/db62785b-07c7-49c0-8737-437f813264da"
+					(reference "C60")
+					(unit 1)
+				)
