File: qwiic.kicad_sch (KiCad schematic)
At the start: 4 parts, among them U8 HCZZ0032-4, U9 USBLC6-2P6

Commit message: Fix QWIIC connector polarity, update flatflex connector.
Connections:
- net +3V3: now also U8.2; no longer U8.1
- net GND: now also U8.1; no longer U8.2
Changed lines of the file:
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@@
+	)
+	(junction
+		(at 104.14 87.63)
+		(diameter 0)
+		(color 0 0 0 0)
 	)
 	(junction
@@
 	)
 	(junction
-		(at 104.14 87.63)
-		(diameter 0)
-		(color 0 0 0 0)
-	)
-	(junction
 		(at 96.52 87.63)
 		(diameter 0)
@@
 	(wire
 		(pts
-			(xy 104.14 66.04) (xy 104.14 73.66)
+			(xy 109.22 66.04) (xy 109.22 76.2)
 		)
 		(stroke
@@
 	(wire
 		(pts
-			(xy 104.14 76.2) (xy 104.14 87.63)
-		)
-		(stroke
-			(width 0)
-			(type default)
-		)
-	)
-	(wire
-		(pts
 			(xy 147.32 66.04) (xy 151.13 66.04)
 		)
@@
 	(wire
 		(pts
-			(xy 101.6 76.2) (xy 104.14 76.2)
+			(xy 104.14 87.63) (xy 119.38 87.63)
 		)
 		(stroke
@@
 	(wire
 		(pts
-			(xy 104.14 87.63) (xy 119.38 87.63)
+			(xy 143.51 66.04) (xy 143.51 67.31)
+		)
+		(stroke
+			(width 0)
+			(type default)
+		)
+	)
+	(wire
+		(pts
+			(xy 151.13 66.04) (xy 151.13 67.31)
+		)
+		(stroke
+			(width 0)
+			(type default)
+		)
+	)
+	(wire
+		(pts
+			(xy 101.6 76.2) (xy 109.22 76.2)
+		)
+		(stroke
+			(width 0)
+			(type default)
+		)
+	)
+	(wire
+		(pts
+			(xy 77.47 66.04) (xy 77.47 87.63)
+		)
+		(stroke
+			(width 0)
+			(type default)
+		)
+	)
+	(wire
+		(pts
+			(xy 124.46 78.74) (xy 143.51 78.74)
+		)
+		(stroke
+			(width 0)
+			(type default)
+		)
+	)
+	(wire
+		(pts
+			(xy 151.13 74.93) (xy 151.13 81.28)
 		)
 		(stroke
@@
 	(wire
 		(pts
-			(xy 143.51 66.04) (xy 143.51 67.31)
-		)
-		(stroke
-			(width 0)
-			(type default)
-		)
-	)
-	(wire
-		(pts
-			(xy 151.13 66.04) (xy 151.13 67.31)
-		)
-		(stroke
-			(width 0)
-			(type default)
-		)
-	)
-	(wire
-		(pts
-			(xy 77.47 66.04) (xy 77.47 87.63)
-		)
-		(stroke
-			(width 0)
-			(type default)
-		)
-	)
-	(wire
-		(pts
-			(xy 124.46 78.74) (xy 143.51 78.74)
-		)
-		(stroke
-			(width 0)
-			(type default)
-		)
-	)
-	(wire
-		(pts
-			(xy 151.13 74.93) (xy 151.13 81.28)
-		)
-		(stroke
-			(width 0)
-			(type default)
-		)
-	)
-	(wire
-		(pts
 			(xy 151.13 81.28) (xy 156.21 81.28)
 		)
@@
 		(pts
 			(xy 101.6 78.74) (xy 114.3 78.74)
+		)
+		(stroke
+			(width 0)
+			(type default)
+		)
+	)
+	(wire
+		(pts
+			(xy 104.14 73.66) (xy 104.14 87.63)
 		)
 		(stroke
@@
 	(symbol
 		(lib_id "power:+3V3")
-		(at 104.14 66.04 0)
+		(at 109.22 66.04 0)
 		(unit 1)
 		(body_style 1)
@@
 		(fields_autoplaced yes)
 		(property "Reference" "#PWR024"
-			(at 104.14 69.85 0)
+			(at 109.22 69.85 0)
 			(hide yes)
 			(show_name no)
@@
 		)
 		(property "Value" "+3V3"
-			(at 104.14 60.96 0)
+			(at 109.22 60.96 0)
 			(show_name no)
 			(do_not_autoplace no)
@@
 		)
 		(property "Footprint" ""
-			(at 104.14 66.04 0)
+			(at 109.22 66.04 0)
 			(hide yes)
 			(show_name no)
@@
 		)
 		(property "Datasheet" ""
-			(at 104.14 66.04 0)
+			(at 109.22 66.04 0)
 			(hide yes)
 			(show_name no)
@@
 		)
 		(property "Description" "Power symbol creates a global label with name \"+3V3\""
-			(at 104.14 66.04 0)
-			(hide yes)
-			(show_name no)
+			(at 109.22 66.04 0)
+			(hide yes)
+			(show_name no)
