File: rgb-led.kicad_sch (KiCad schematic)
At the start: 4 parts

Commit message: Fixed mistake in NRF52 footprint, add NAND FLASH, add NFC antenna schematic.
Parts:
- renumbered R5 to R6, R6 to R7, R7 to R8
Other:
- company: (none) -> Badge.Team
- title: (none) -> Bornhack 2026
Changed lines of the file:
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@@
 	(generator_version "9.0")
 	(paper "A4")
+	(title_block
+		(title "Bornhack 2026")
+		(rev "0.1")
+		(company "Badge.Team")
+	)
 	(wire
 		(pts
@@
 		(dnp no)
 		(fields_autoplaced yes)
-		(property "Reference" "R5"
+		(property "Reference" "R6"
 			(at 55.88 53.34 90)
 			(effects
@@
 			(project ""
 				(path "/23bf5400-d19c-445b-8744-b63ebcca303d/6b9e027f-7f51-40c0-a70e-149da1361e88"
-					(reference "R5")
+					(reference "R6")
 					(unit 1)
 				)
@@
 		(dnp no)
 		(fields_autoplaced yes)
-		(property "Reference" "R6"
+		(property "Reference" "R7"
 			(at 97.79 53.34 90)
 			(effects
@@
 			(project "bornhack2026-hardware"
 				(path "/23bf5400-d19c-445b-8744-b63ebcca303d/6b9e027f-7f51-40c0-a70e-149da1361e88"
-					(reference "R6")
+					(reference "R7")
 					(unit 1)
 				)
@@
 		(dnp no)
 		(fields_autoplaced yes)
-		(property "Reference" "R7"
+		(property "Reference" "R8"
 			(at 97.79 60.96 90)
 			(effects
@@
 			(project "bornhack2026-hardware"
 				(path "/23bf5400-d19c-445b-8744-b63ebcca303d/6b9e027f-7f51-40c0-a70e-149da1361e88"
-					(reference "R7")
+					(reference "R8")
 					(unit 1)
 				)

Commit message: Switched the LC filters from ceramic LoRa filter.
Parts:
- LED1: LCSC (none) -> C965840
Changed lines of the file:
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@@
 			)
 		)
-		(property "Datasheet" ""
+		(property "Datasheet" "https://jlcpcb.com/partdetail/XINGLIGHT-XL_1615RGBCRF/C965840"
 			(at 77.47 60.96 0)
 			(effects
@@
 			(effects
 				(font
+					(size 1.27 1.27)
+				)
+				(hide yes)
+			)
+		)
+		(property "LCSC" "C965840"
+			(at 77.47 60.96 0)
+			(effects
+				(font

Commit message: Routed buttons to MCU.
Parts:
- R6, R8: value 1k -> 2k; LCSC C11702 -> C4109
- R7: value 1k -> 10k; LCSC C11702 -> C25744
Changed lines of the file:
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@@
 			)
 		)
-		(property "Value" "1k"
+		(property "Value" "2k"
 			(at 55.88 55.88 90)
 			(effects
@@
 			)
 		)
-		(property "Datasheet" "https://jlcpcb.com/partdetail/12256-0402WGF1001TCE/C11702"
+		(property "Datasheet" "https://www.lcsc.com/product-detail/Chip-Resistor-Surface-Mount_UNI-ROYAL-Uniroyal-Elec-0402WGF2001TCE_C4109.html"
 			(at 55.88 58.42 0)
 			(effects
@@
 			)
 		)
-		(property "LCSC" "C11702"
+		(property "LCSC" "C4109"
 			(at 55.88 58.42 90)
 			(effects
@@
 			)
 		)
-		(property "Value" "1k"
+		(property "Value" "10k"
 			(at 97.79 55.88 90)
 			(effects
@@
 			)
 		)
-		(property "Datasheet" "https://jlcpcb.com/partdetail/12256-0402WGF1001TCE/C11702"
+		(property "Datasheet" "https://www.lcsc.com/product-detail/Chip-Resistor-Surface-Mount_UNI-ROYAL-Uniroyal-Elec-0402WGF1002TCE_C25744.html"
 			(at 97.79 58.42 0)
 			(effects
@@
 			)
 		)
-		(property "LCSC" "C11702"
+		(property "LCSC" "C25744"
 			(at 97.79 58.42 90)
 			(effects
@@
 			)
 		)
-		(property "Value" "1k"
+		(property "Value" "2k"
 			(at 97.79 63.5 90)
 			(effects
@@
 			)
 		)
-		(property "Datasheet" "https://jlcpcb.com/partdetail/12256-0402WGF1001TCE/C11702"
+		(property "Datasheet" "https://www.lcsc.com/product-detail/Chip-Resistor-Surface-Mount_UNI-ROYAL-Uniroyal-Elec-0402WGF2001TCE_C4109.html"
 			(at 97.79 66.04 0)
 			(effects
@@
 			)
 		)
-		(property "LCSC" "C11702"
+		(property "LCSC" "C4109"
 			(at 97.79 66.04 90)
 			(effects
